File: vme1.sch (EAGLE design)
At the start: 9 parts, among them IC1 PCM1865DBT, U1 RASPBERRY_PI_4B_4GB

Commit message: update
Parts:
- added C10, C11, C12, C13, C14, C15, C16, C17, C18, C19, C20, C21, C22, C23, C24, C8, C9: 0.047uF, rcl:C-US025-024X044
- added C25, C43, C44, C45, C46: (no value), rcl:C-US025-024X044
- added C26, C27, C28, C29, C30, C31, C32, C33, C34, C35, C36, C37, C38, C39, C40, C41, C42: 10uF, rcl:C-US025-024X044
- added R1, R2, R3, R4, R5, R6, R7: (no value), rcl:R-US_0204/2V
- added U$1: LC75281E, LC75281E:LC75281E
Connections:
- new net +8V: U$1.V_DD
- new net EQ1_CE: U$1.CE, U1.GPIO20
- new net EQ1_CL: U$1.CL, U1.GPIO26
- new net EQ1_DI: U$1.DI, U1.GPIO21
- new net N$12: C24.1, C9.1, U$1.LLC4
- new net N$13: C10.1, U$1.LLMC1
- new net N$14: C11.1, U$1.LLMC4
- new net N$15: C12.1, U$1.LHMC1
- new net N$16: C13.1, U$1.LHMC4
- new net N$17: C14.1, U$1.LHC1
- new net N$18: C15.1, U$1.LHC4
- new net N$19: C16.1, U$1.RHC4
- new net N$20: C17.1, U$1.RHC1
- new net N$21: C18.1, U$1.RHMC4
- new net N$22: C19.1, U$1.RHMC1
- new net N$23: C20.1, U$1.RLMC4
- new net N$24: C21.1, U$1.RLMC1
- new net N$25: C22.1, U$1.RLC4
- new net N$26: C23.1, U$1.RLC1
- new net N$27: C8.2, U$1.LLC2
- new net N$28: C24.2, C26.2, C9.2, U$1.LLC3
- new net N$29: C26.1, U$1.LLC5
- new net N$30: C27.1, U$1.LLMC5
- new net N$31: C28.1, U$1.LHMC5
- new net N$32: C29.1, U$1.LHC5
- new net N$33: C30.1, U$1.V_REF
- new net N$34: C31.1, U$1.RHC5
- new net N$35: C32.1, U$1.RHMC5
- new net N$36: C33.1, U$1.RLMC5
- new net N$37: C34.1, U$1.RLC5
- new net N$38: C35.1, U$1.ROUT
- new net N$39: C36.1, U$1.RBOOS2
- new net N$40: C37.1, U$1.RIN
- new net N$41: C38.1, U$1.RCUT2
- new net N$42: C39.1, U$1.LCUT1
- new net N$43: C40.1, U$1.LIN
- new net N$44: C41.1, U$1.LBOOS1
- new net N$45: C42.1, U$1.LOUT
- new net N$46: C10.2, U$1.LLMC2
- new net N$47: C11.2, C27.2, U$1.LLMC3
- new net N$48: C12.2, U$1.LHMC2
- new net N$49: C13.2, C28.2, U$1.LHMC3
- new net N$50: C14.2, U$1.LHC2
- new net N$51: C15.2, C29.2, U$1.LHC3
- new net N$59: C16.2, C31.2, U$1.RHC3
- new net N$60: C17.2, U$1.RHC2
- new net N$61: C18.2, C32.2, U$1.RHMC3
- new net N$62: C19.2, U$1.RHMC2
- new net N$63: C20.2, C33.2, U$1.RLMC3
- new net N$64: C21.2, U$1.RLMC2
- new net N$65: C22.2, C34.2, U$1.RLC3
- new net N$66: C23.2, U$1.RLC2
- new net N$67: C36.2, U$1.RBOOS1
- new net N$68: C37.2
- new net N$69: C38.2, U$1.RCUT1
- new net N$70: C39.2, U$1.LCUT2
- new net N$71: C40.2
- new net N$72: C41.2, U$1.LBOOS2
- new net N$73: C42.2
- new net N$74: C35.2
- new net N$9: C8.1, U$1.LLC1
- net AGND: now also C25.1, C30.2, C44.1, R1.1, U$1.TEST, U$1.V_SS

Commit message: update compressor with digital pots Added to man schem with muxes
Parts:
- added C47: 0.1, rcl:C-US025-024X044
- added C48, C49: 1.5u, rcl:C-US025-024X044
- added D1, D10, D11, D12, D13, D14, D15, D16, D17, D18, D19, D2, D20, D21, D22, D3, D4, D5, D6, D7, D8, D9: 1N4148DO35-7, diode:1N4148DO35-7
- added R10, R12, R13, R15, R16, R18, R21, R22, R23, R27, R28, R29, R31, R32, R33, R35, R36, R40, R41, R42, R44, R9: 100k, rcl:R-US_0204/7
- added R11, R14, R24, R26, R34, R37, R43: 10k, rcl:R-US_0204/7
- added R17, R20, R8: 470k, rcl:R-US_0204/7
- added R19: 1k, rcl:R-US_0204/7
- added R25, R38: 20k, rcl:R-US_0204/7
- added R30, R39: 1M, rcl:R-US_0204/7
- added U$2, U$5: MCP42100-I/P, MCP42100-I_P:MCP42100-I/P
- added U$3, U$4, U$6, U$7: MCP4131-503E/SN, MCP4131-503E_SN:MCP4131-503E/SN
- added U2, U3, U4, U5: MAX5419LETA+, MAX5419LETA_:MAX5419LETA+
- added U6, U7, U8: TMUX1204DGSR, TMUX1204DGSR:TMUX1204DGSR
- added U9: TCA9546ADR, TCA9546ADR:TCA9546ADR
- added X1, X10, X11, X12, X13, X14, X15, X16, X17, X18, X2, X3, X4, X5, X6, X7, X8, X9: OPAMP, ngspice-simulation:OPAMP
- C25, C46: value (none) -> 680p
- C43: value (none) -> 0.1
- C44, C45: value (none) -> 1.5u
- R1, R2, R3, R5: value (none) -> 100k; device rcl:R-US_0204/2V -> rcl:R-US_0204/7
- R4: value (none) -> 10k; device rcl:R-US_0204/2V -> rcl:R-US_0204/7
- R6: value (none) -> 470k; device rcl:R-US_0204/2V -> rcl:R-US_0204/7
- R7: value (none) -> 1k; device rcl:R-US_0204/2V -> rcl:R-US_0204/7
Connections:
- net N$73 renamed EOUT_1
- net N$74 renamed EOUT_0
- new net 0: R1.1, R30.2, R39.2, R5.1, U$2.VSS, U$3.VSS, U$4.VSS, U$5.VSS, U$6.VSS, U$7.VSS, U2.A0, U2.GND, U3.GND, U4.A0, U4.GND, U5.GND, X1.VSS, X10.VSS, X11.VSS, X12.VDD, X13.VDD, X14.VDD, X15.VDD, X16.VSS, X17.VSS, X18.VSS, X2.VSS, X3.VDD, X4.VSS, X5.VDD, X6.VDD, X7.VDD, X8.VSS, X9.VSS
- new net AIN_0: C43.2
- new net AIN_1: C47.2
- new net AOUT_0: C44.1, R30.1
- new net AOUT_1: C48.1, R39.1
- new net CS0: U1.GPIO12, U6.D
- new net CS0_0: U$2.~CS, U6.S1
- new net CS0_1: U$5.~CS, U6.S2
- new net CS1: U1.GPIO13, U8.D
- new net CS1_0: U$3.!CS, U8.S1
- new net CS1_1: U$6.!CS, U8.S2
- new net CS2: U1.GPIO16, U7.D
- new net CS2_0: U$4.!CS, U7.S1
- new net CS2_1: U$7.!CS, U7.S2
- new net H_0_0: C45.1, R8.1, U2.H, U3.H, X7.N
- new net H_0_1: C49.1, R20.1, U4.H, U5.H, X15.N
- new net L_0_0: R15.1, U2.L
- new net L_0_1: R27.1, U4.L
- new net L_1_0: D4.C, U3.L
- new net L_1_1: D15.C, U5.L
- new net MUX0: U1.GPIO5, U6.A0, U7.A0, U8.A0
- new net MUX1: U1.GPIO6, U6.A1, U7.A1, U8.A1
- new net N$100: D22.C, R29.2, X15.P
- new net N$101: R29.1, R33.2, X16.N
- new net N$102: R36.1, X13.VOUT, X14.P
- new net N$103: R36.2, R37.2, X13.N
- new net N$104: D13.C, D6.A
- new net N$105: C46.1, D13.A, D14.C, D21.A, R19.1, R40.2
- new net N$106: D15.A, X15.VOUT
- new net N$107: R40.1, R41.2, X17.P
- new net N$108: D16.C, R41.1, X17.VOUT
- new net N$109: D17.A, D18.C
- new net N$110: D16.A, D17.C
- new net N$111: D18.A, D19.C, R33.1, R44.1, X13.P
- new net N$112: R44.2, X18.P, X18.VOUT
- new net N$113: C47.1, R42.2
- new net N$114: D20.A, D21.C
- new net N$115: D19.A, D20.C
- new net N$116: D22.A, X16.VOUT
- new net N$118: R26.2
- new net N$119: C49.2
- new net N$123: U6.S3
- new net N$124: U6.S4
- new net N$125: U9.SC2
- new net N$126: U9.SC3
- new net N$127: U9.SD2
- new net N$128: U7.S3
- new net N$129: U7.S4
- new net N$130: U9.SD3
- new net N$133: U8.S3
- new net N$134: U8.S4
- new net N$52: R7.2, X1.VOUT
- new net N$53: C25.2, D1.C, D3.A, R3.2, X1.P
- new net N$54: R1.2, R2.1, X2.N
- new net N$55: X2.P, X2.VOUT
- new net N$56: R6.2, R8.2, X3.P
- new net N$57: R10.1, R9.2, X3.N
- new net N$58: D5.C, R16.2, X7.P
- new net N$75: R16.1, R18.2, X8.N
- new net N$76: R21.1, X5.VOUT, X6.P
- new net N$77: R21.2, R24.2, X5.N
- new net N$78: D1.A, D2.C
- new net N$79: C25.1, D12.A, D2.A, D3.C, R28.2, R7.1
- new net N$80: D4.A, X7.VOUT
- new net N$81: R28.1, R31.2, X9.P
- new net N$82: D7.C, R31.1, X9.VOUT
- new net N$83: D8.A, D9.C
- new net N$84: D7.A, D8.C
- new net N$85: D10.C, D9.A, R18.1, R35.1, X5.P
- new net N$86: R35.2, X10.P, X10.VOUT
- new net N$87: C43.1, R32.2
- new net N$88: D11.A, D12.C
- new net N$89: D10.A, D11.C
- new net N$90: D5.A, X8.VOUT
- new net N$92: R11.2
- new net N$93: C45.2
- new net N$94: R19.2, X4.VOUT
- new net N$95: C46.2, D14.A, D6.C, R13.2, X4.P
- new net N$96: R12.1, R5.2, X11.N
- new net N$97: X11.P, X11.VOUT
- new net N$98: R17.2, R20.2, X12.P
- new net N$99: R22.2, R23.1, X12.N
- new net P0A_0_0: U$3.P0A
- new net P0A_0_1: U$6.P0A
- new net P0A_1_0: R34.1, U$4.P0A
- new net P0A_1_1: R43.1, U$7.P0A
- new net P0B_0_0: U$3.P0B
- new net P0B_0_1: U$6.P0B
- new net P0B_1_0: R32.1, U$4.P0B, X10.N
- new net P0B_1_1: R42.1, U$7.P0B, X18.N
- new net P0W_0_0: U$3.P0W
- new net P0W_0_1: U$6.P0W
- new net PA0_0_0: R10.2, U$2.PA0, X3.VOUT
- new net PA0_1: R23.2, U$5.PA0, X12.VOUT
- new net PA1_0: R25.2, U$2.PA1, X6.N
- new net PA1_1: R38.2, U$5.PA1, X14.N
- new net PB0_0: R4.2, U$2.PB0, X1.N
- new net PB0_1: R14.2, U$5.PB0, X4.N
- new net PB1_0_0: C44.2, U$2.PB1, X6.VOUT
- new net PB1_1: C48.2, U$5.PB1, X14.VOUT
- new net SCK: U$2.SCK, U$3.SCK, U$4.SCK, U$5.SCK, U$6.SCK, U$7.SCK, U1.GPIO11/SPI_SCLK
- new net SCL: U1.GPIO14/TXD0, U9.SCL
- new net SCL_0: U2.SCL, U3.SCL, U9.SC0
- new net SCL_1: U4.SCL, U5.SCL, U9.SD0
- new net SDA: U1.GPIO15/RXD0, U9.SDA
- new net SDA_0: U2.SDA, U3.SDA, U9.SC1
- new net SDA_1: U4.SDA, U5.SDA, U9.SD1
- new net SDI/O: U$2.SI, U$3.SDI/SDO, U$4.SDI/SDO, U$5.SI, U$6.SDI/SDO, U$7.SDI/SDO, U1.GPIO10/SPI_MOSI
- new net SO_0: U$2.SO
- new net SO_1: U$5.SO
- new net VDD: R11.1, R12.2, R2.2, R26.1, U$2.VDD, U$3.VDD, U$4.VDD, U$5.VDD, U$6.VDD, U$7.VDD, U2.VDD, U3.A0, U3.VDD, U4.VDD, U5.A0, U5.VDD, X1.VDD, X10.VDD, X11.VDD, X12.VSS, X13.VSS, X14.VSS, X15.VSS, X16.VDD, X17.VDD, X18.VDD, X2.VDD, X3.VSS, X4.VDD, X5.VSS, X6.VSS, X7.VSS, X8.VDD, X9.VDD
- new net VREF: R14.1, R4.1
- net +3V3: now also U6.EN, U6.VDD, U7.EN, U7.VDD, U8.EN, U8.VDD, U9.VCC
- net AGND: no longer C25.1, C44.1, R1.1
- net DGND: now also U6.GND, U7.GND, U8.GND, U9.A0, U9.A1, U9.A2, U9.GND, U9.RESET
- net N$38: now also U$2.~RS, U$5.~RS
- net N$39: now also U$2.~SHDN, U$5.~SHDN
Other:
- moved on the sheet: C25, C43, C44, C45, C46, R1, R2, R3, R4, R5, R6, R7

Commit message: add other 2 comps and 1 other eq
Parts:
- added C50, C54: 680p, rcl:C-US025-024X044
- added C51, C55: 0.1, rcl:C-US025-024X044
- added C52, C53, C56, C57: 1.5u, rcl:C-US025-024X044
- added C58, C59, C60, C61, C62, C63, C64, C65, C66, C67, C68, C69, C70, C71, C72, C73, C74: 0.047uF, rcl:C-US025-024X044
- added C75, C76, C77, C78, C79, C80, C81, C82, C83, C84, C85, C86, C87, C88, C89, C90, C91: 10uF, rcl:C-US025-024X044
- added D23, D24, D25, D26, D27, D28, D29, D30, D31, D32, D33, D34, D35, D36, D37, D38, D39, D40, D41, D42, D43, D44: 1N4148DO35-7, diode:1N4148DO35-7
- added R45, R46, R47, R52, R53, R55, R56, R57, R58, R62, R63, R64, R66, R67, R68, R69, R74, R75, R77, R78, R79, R80, R84, R85, R86, R88: 100k, rcl:R-US_0204/7
- added R48, R54, R59, R65, R70, R76, R81, R87: 10k, rcl:R-US_0204/7
- added R49, R51, R71, R73: 470k, rcl:R-US_0204/7
- added R50, R72: 1k, rcl:R-US_0204/7
- added R60, R82: 20k, rcl:R-US_0204/7
- added R61, R83: 1M, rcl:R-US_0204/7
- added U$10, U$12, U$13, U$9: MCP4131-503E/SN, MCP4131-503E_SN:MCP4131-503E/SN
- added U$11, U$8: MCP42100-I/P, MCP42100-I_P:MCP42100-I/P
- added U$14: LC75281E, LC75281E:LC75281E
- added U10, U11, U12, U13: MAX5419LETA+, MAX5419LETA_:MAX5419LETA+
- added X19, X20, X21, X22, X23, X24, X25, X26, X27, X28, X29, X30, X31, X32, X33, X34, X35, X36: OPAMP, ngspice-simulation:OPAMP
Connections:
- net N$128 renamed CS2_2
- removed net CS0: U1.GPIO12, U6.D
- removed net CS1: U1.GPIO13, U8.D
- removed net N$1: IC1.VINL2/VIN1M
- removed net N$2: IC1.VINR2/VIN2M
- removed net N$3: IC1.VINL1/VIN1P
- removed net N$4: IC1.VINR1/VIN2P
- removed net N$5: IC1.VINR3/VIN3P
- removed net N$6: IC1.VINL3/VIN4P
- removed net N$7: IC1.VINR4/VIN3M
- removed net N$8: IC1.VINL4/VIN4M
- removed net SCL1: IC1.MC/SCL, U1.GPIO3/SCL1
- removed net SDA1: IC1.MOSI/SDA, U1.GPIO2/SDA1
- new net AIN_2: C51.2
- new net AIN_3: C55.2
- new net AOUT_2: C52.1, R61.1
- new net AOUT_3: C56.1, R83.1
- new net CS0_2: U$8.~CS, U1.GPIO12, U6.D, U6.S3
- new net CS0_3: U$11.~CS, U6.S4
- new net CS1_2: U$9.!CS, U1.GPIO13, U8.D, U8.S3
- new net CS1_3: U$12.!CS, U8.S4
- new net CS2_3: U$13.!CS, U7.S4
- new net EOUT_2: C84.2, IC1.VINR3/VIN3P
- new net EOUT_3: C91.2, IC1.VINR4/VIN3M
- new net EQ0_CE: U$1.CE, U1.GPIO23/GPIO_GEN4
- new net EQ0_CL: U$1.CL, U1.GPIO25/GPIO_GEN6
- new net EQ0_DI: U$1.DI, U1.GPIO24/GPIO_GEN5
- new net H_0_2: C53.1, R51.1, U10.H, U11.H, X24.N
- new net H_0_3: C57.1, R73.1, U12.H, U13.H, X33.N
- new net L_0_2: R55.1, U10.L
- new net L_0_3: R77.1, U12.L
- new net L_1_2: D26.C, U11.L
- new net L_1_3: D37.C, U13.L
- new net N$120: R45.2, R46.1, X20.N
- new net N$121: X20.P, X20.VOUT
- new net N$122: R49.2, R51.2, X21.P
- new net N$128: C63.1, U$14.LHMC4
- new net N$131: R52.2, R53.1, X21.N
- new net N$132: D33.C, R56.2, X24.P
- new net N$135: R56.1, R57.2, X25.N
- new net N$136: R58.1, X22.VOUT, X23.P
- new net N$137: R58.2, R59.2, X22.N
- new net N$138: D23.A, D24.C
- new net N$139: C50.1, D24.A, D25.C, D32.A, R50.1, R62.2
- new net N$140: D26.A, X24.VOUT
- new net N$141: R62.1, R63.2, X26.P
- new net N$142: D27.C, R63.1, X26.VOUT
- new net N$143: D28.A, D29.C
- new net N$144: D27.A, D28.C
- new net N$145: D29.A, D30.C, R57.1, R66.1, X22.P
- new net N$146: R66.2, X27.P, X27.VOUT
- new net N$147: C51.1, R64.2
- new net N$148: D31.A, D32.C
- new net N$149: D30.A, D31.C
- new net N$150: D33.A, X25.VOUT
- new net N$152: R54.2
- new net N$153: C53.2
- new net N$154: R72.2, X28.VOUT
- new net N$155: C54.2, D34.C, D36.A, R69.2, X28.P
- new net N$156: R67.2, R68.1, X29.N
- new net N$157: X29.P, X29.VOUT
- new net N$158: R71.2, R73.2, X30.P
- new net N$159: R74.2, R75.1, X30.N
- new net N$160: D44.C, R78.2, X33.P
- new net N$161: R78.1, R79.2, X34.N
- new net N$162: R80.1, X31.VOUT, X32.P
- new net N$163: R80.2, R81.2, X31.N
- new net N$164: D34.A, D35.C
- new net N$165: C54.1, D35.A, D36.C, D43.A, R72.1, R84.2
- new net N$166: D37.A, X33.VOUT
- new net N$167: R84.1, R85.2, X35.P
- new net N$168: D38.C, R85.1, X35.VOUT
- new net N$169: D39.A, D40.C
- new net N$170: D38.A, D39.C
- new net N$171: D40.A, D41.C, R79.1, R88.1, X31.P
- new net N$172: R88.2, X36.P, X36.VOUT
- new net N$173: C55.1, R86.2
- new net N$174: D42.A, D43.C
- new net N$175: D41.A, D42.C
- new net N$176: D44.A, X34.VOUT
- new net N$178: R76.2
- new net N$179: C57.2
- new net N$180: C68.1, U$14.RHMC4
- new net N$181: C69.1, U$14.RHMC1
- new net N$182: C70.1, U$14.RLMC4
- new net N$183: C71.1, U$14.RLMC1
- new net N$184: C72.1, U$14.RLC4
- new net N$185: C73.1, U$14.RLC1
- new net N$186: C58.2, U$14.LLC2
- new net N$187: C59.2, C74.2, C75.2, U$14.LLC3
- new net N$188: C75.1, U$14.LLC5
- new net N$189: C76.1, U$14.LLMC5
- new net N$190: C77.1, U$14.LHMC5
- new net N$191: C78.1, U$14.LHC5
- new net N$192: C79.1, U$14.V_REF
- new net N$193: C80.1, U$14.RHC5
- new net N$194: C81.1, U$14.RHMC5
- new net N$195: C82.1, U$14.RLMC5
- new net N$196: C83.1, U$14.RLC5
- new net N$197: C84.1, U$14.ROUT
- new net N$198: C85.1, U$14.RBOOS2
- new net N$199: C86.1, U$14.RIN
- new net N$200: C87.1, U$14.RCUT2
- new net N$201: C88.1, U$14.LCUT1
- new net N$202: C89.1, U$14.LIN
- new net N$203: C90.1, U$14.LBOOS1
- new net N$204: C91.1, U$14.LOUT
- new net N$205: C60.2, U$14.LLMC2
- new net N$206: C61.2, C76.2, U$14.LLMC3
- new net N$207: C62.2, U$14.LHMC2
- new net N$208: C63.2, C77.2, U$14.LHMC3
- new net N$209: C64.2, U$14.LHC2
- new net N$210: C65.2, C78.2, U$14.LHC3
- new net N$211: C66.2, C80.2, U$14.RHC3
- new net N$212: C67.2, U$14.RHC2
- new net N$213: C68.2, C81.2, U$14.RHMC3
- new net N$214: C69.2, U$14.RHMC2
- new net N$215: C70.2, C82.2, U$14.RLMC3
- new net N$216: C71.2, U$14.RLMC2
- new net N$217: C72.2, C83.2, U$14.RLC3
- new net N$218: C73.2, U$14.RLC2
- new net N$219: C85.2, U$14.RBOOS1
- new net N$220: C86.2
- new net N$221: C87.2, U$14.RCUT1
- new net N$222: C88.2, U$14.LCUT2
- new net N$223: C89.2
- new net N$224: C90.2, U$14.LBOOS2
- new net N$73: R50.2, X19.VOUT
- new net N$74: C50.2, D23.C, D25.A, R47.2, X19.P
- new net P0A_0_2: U$9.P0A
- new net P0A_0_3: U$12.P0A
- new net P0A_1_2: R65.1, U$10.P0A
- new net P0A_1_3: R87.1, U$13.P0A
- new net P0B_0_2: U$9.P0B
- new net P0B_0_3: U$12.P0B
- new net P0B_1_2: R64.1, U$10.P0B, X27.N
- new net P0B_1_3: R86.1, U$13.P0B, X36.N
- new net P0W_0_2: U$9.P0W
- new net P0W_0_3: U$12.P0W
- new net PA0_2: R53.2, U$8.PA0, X21.VOUT
- new net PA0_3: R75.2, U$11.PA0, X30.VOUT
- new net PA1_2: R60.2, U$8.PA1, X23.N
- new net PA1_3: R82.2, U$11.PA1, X32.N
- new net PB0_2: R48.2, U$8.PB0, X19.N
- new net PB0_3: R70.2, U$11.PB0, X28.N
- new net PB1_2: C52.2, U$8.PB1, X23.VOUT
- new net PB1_3: C56.2, U$11.PB1, X32.VOUT
- new net SCL_2: U10.SCL, U11.SCL, U9.SC2
- new net SCL_3: U12.SCL, U13.SCL, U9.SD2
- new net SDA_2: U10.SDA, U11.SDA, U9.SC3
- new net SDA_3: U12.SDA, U13.SDA, U9.SD3
- new net SO_2: U$8.SO
- new net SO_3: U$11.SO
- net +8V: now also U$14.V_DD
- net 0: now also R45.1, R61.2, R67.1, R83.2, U$10.VSS, U$11.VSS, U$12.VSS, U$13.VSS, U$8.VSS, U$9.VSS, U10.A0, U10.GND, U11.GND, U12.A0, U12.GND, U13.GND, X19.VSS, X20.VSS, X21.VDD, X22.VDD, X23.VDD, X24.VDD, X25.VSS, X26.VSS, X27.VSS, X28.VSS, X29.VSS, X30.VDD, X31.VDD, X32.VDD, X33.VDD, X34.VSS, X35.VSS, X36.VSS
- net AGND: now also C79.2, U$14.TEST, U$14.V_SS
- net CS2: now also U$10.!CS
- net EOUT_0: now also IC1.VINL2/VIN1M
- net EOUT_1: now also IC1.VINL1/VIN1P
- net EQ1_CE: now also U$14.CE; no longer U$1.CE
- net EQ1_CL: now also U$14.CL; no longer U$1.CL
- net EQ1_DI: now also U$14.DI; no longer U$1.DI
- net N$123: now also C58.1, U$14.LLC1; no longer U6.S3
- net N$124: now also C59.1, C74.1, U$14.LLC4; no longer U6.S4
- net N$125: now also C60.1, U$14.LLMC1; no longer U9.SC2
- net N$126: now also C61.1, U$14.LLMC4; no longer U9.SC3
- net N$127: now also C62.1, U$14.LHMC1; no longer U9.SD2
- net N$129: now also C64.1, U$14.LHC1; no longer U7.S4
- net N$130: now also C65.1, U$14.LHC4; no longer U9.SD3
- net N$133: now also C66.1, U$14.RHC4; no longer U8.S3
- net N$134: now also C67.1, U$14.RHC1; no longer U8.S4
- net N$38: now also U$11.~RS, U$8.~RS
- net N$39: now also U$11.~SHDN, U$8.~SHDN
- net SCK: now also U$10.SCK, U$11.SCK, U$12.SCK, U$13.SCK, U$8.SCK, U$9.SCK
- net SCL: now also IC1.MC/SCL, U1.GPIO3/SCL1; no longer U1.GPIO14/TXD0
- net SDA: now also IC1.MOSI/SDA, U1.GPIO2/SDA1; no longer U1.GPIO15/RXD0
- net SDI/O: now also U$10.SDI/SDO, U$11.SI, U$12.SDI/SDO, U$13.SDI/SDO, U$8.SI, U$9.SDI/SDO
- net VDD: now also R46.2, R54.1, R68.2, R76.1, U$10.VDD, U$11.VDD, U$12.VDD, U$13.VDD, U$8.VDD, U$9.VDD, U10.VDD, U11.A0, U11.VDD, U12.VDD, U13.A0, U13.VDD, X19.VDD, X20.VDD, X21.VSS, X22.VSS, X23.VSS, X24.VSS, X25.VDD, X26.VDD, X27.VDD, X28.VDD, X29.VDD, X30.VSS, X31.VSS, X32.VSS, X33.VSS, X34.VDD, X35.VDD, X36.VDD
- net VREF: now also R48.1, R70.1

Commit message: update, split out into schematics for each component
Parts:
- removed C10, C11, C12, C13, C14, C15, C16, C17, C18, C19, C20, C21, C22, C23, C24, C58, C59, C60, C61, C62, C63, C64, C65, C66, C67, C68, C69, C70, C71, C72, C73, C74, C8, C9: 0.047uF, rcl:C-US025-024X044
- removed C25, C46, C50, C54: 680p, rcl:C-US025-024X044
- removed C26, C27, C28, C29, C30, C31, C32, C33, C34, C35, C36, C37, C38, C39, C40, C41, C42, C75, C76, C77, C78, C79, C80, C81, C82, C83, C84, C85, C86, C87, C88, C89, C90, C91: 10uF, rcl:C-US025-024X044
- removed C43, C47, C51, C55: 0.1, rcl:C-US025-024X044
- removed C44, C45, C48, C49, C52, C53, C56, C57: 1.5u, rcl:C-US025-024X044
- removed C5, C7: 1μF, rcl:C-US025-024X044
- removed C6: 0.1μF, rcl:C-US025-024X044
- removed D13, D14, D15, D16, D17, D18, D19, D20, D21, D22, D23, D24, D25, D26, D27, D28, D29, D30, D31, D32, D33, D34, D35, D36, D37, D38, D39, D40, D41, D42, D43, D44, D6: 1N4148DO35-7, diode:1N4148DO35-7
- removed IC1: PCM1865DBT, PCM1865DBT:PCM1865DBT
- removed R12, R13, R2, R22, R23, R27, R29, R33, R36, R40, R41, R42, R44, R45, R46, R47, R5, R52, R53, R55, R56, R57, R58, R62, R63, R64, R66, R67, R68, R69, R74, R75, R77, R78, R79, R80, R84, R85, R86, R88: 100k, rcl:R-US_0204/7
- removed R14, R26, R37, R43, R48, R54, R59, R65, R70, R76, R81, R87: 10k, rcl:R-US_0204/7
- removed R17, R20, R49, R51, R71, R73: 470k, rcl:R-US_0204/7
- removed R19, R50, R72: 1k, rcl:R-US_0204/7
- removed R38, R60, R82: 20k, rcl:R-US_0204/7
- removed R39, R61, R83: 1M, rcl:R-US_0204/7
- removed U$10, U$12, U$13, U$4, U$6, U$7, U$9: MCP4131-503E/SN, MCP4131-503E_SN:MCP4131-503E/SN
- removed U$11, U$5, U$8: MCP42100-I/P, MCP42100-I_P:MCP42100-I/P
- removed U$14: LC75281E, LC75281E:LC75281E
- removed U10, U11, U12, U13, U3, U4, U5: MAX5419LETA+, MAX5419LETA_:MAX5419LETA+
- removed U6, U7, U8: TMUX1204DGSR, TMUX1204DGSR:TMUX1204DGSR
- removed U9: TCA9546ADR, TCA9546ADR:TCA9546ADR
- removed X11, X12, X13, X14, X15, X16, X17, X18, X19, X2, X20, X21, X22, X23, X24, X25, X26, X27, X28, X29, X30, X31, X32, X33, X34, X35, X36: OPAMP, ngspice-simulation:OPAMP
- C1: value 0.1μF -> 680p
- C2: value 10μF -> 0.1
- C3: value 0.1μF -> 1.5u
- C4: value 10μF -> 1.5u
- R1: value 100k -> 0
- U$1: value LC75281E -> MCP42100-I/P; device LC75281E:LC75281E -> MCP42100-I_P:MCP42100-I/P
- U$2: value MCP42100-I/P -> MCP4131-503E/SN; device MCP42100-I_P:MCP42100-I/P -> MCP4131-503E_SN:MCP4131-503E/SN
- U1: value RASPBERRY_PI_4B_4GB -> MAX5419LETA+; device RASPBERRY_PI_4B_4GB:RASPBERRY_PI_4B_4GB -> MAX5419LETA_:MAX5419LETA+
- X4: value OPAMP -> NCJ10FI-H; device ngspice-simulation:OPAMP -> con-neutrik_ag:NCJ10FI-H
Connections:
- removed net +3V3: C1.1, C2.1, C3.1, C4.1, IC1.AVDD, IC1.DVDD, IC1.IOVDD, U1.3V3, U6.EN, U6.VDD, U7.EN, U7.VDD, U8.EN, U8.VDD, U9.VCC
- removed net +5V: U1.5V
- removed net +8V: U$1.V_DD, U$14.V_DD
- removed net 0: R1.1, R30.2, R39.2, R45.1, R5.1, R61.2, R67.1, R83.2, U$10.VSS, U$11.VSS, U$12.VSS, U$13.VSS, U$2.VSS, U$3.VSS, U$4.VSS, U$5.VSS, U$6.VSS, U$7.VSS, U$8.VSS, U$9.VSS, U10.A0, U10.GND, U11.GND, U12.A0, U12.GND, U13.GND, U2.A0, U2.GND, U3.GND, U4.A0, U4.GND, U5.GND, X1.VSS, X10.VSS, X11.VSS, X12.VDD, X13.VDD, X14.VDD, X15.VDD, X16.VSS, X17.VSS, X18.VSS, X19.VSS, X2.VSS, X20.VSS, X21.VDD, X22.VDD, X23.VDD, X24.VDD, X25.VSS, X26.VSS, X27.VSS, X28.VSS, X29.VSS, X3.VDD, X30.VDD, X31.VDD, X32.VDD, X33.VDD, X34.VSS, X35.VSS, X36.VSS, X4.VSS, X5.VDD, X6.VDD, X7.VDD, X8.VSS, X9.VSS
- removed net AGND: C3.2, C30.2, C4.2, C5.2, C6.2, C7.2, C79.2, IC1.AGND, IC1.DGND, U$1.TEST, U$1.V_SS, U$14.TEST, U$14.V_SS
- removed net AIN_0: C43.2
- removed net AIN_1: C47.2
- removed net AIN_2: C51.2
- removed net AIN_3: C55.2
- removed net AOUT_0: C44.1, R30.1
- removed net AOUT_1: C48.1, R39.1
- removed net AOUT_2: C52.1, R61.1
- removed net AOUT_3: C56.1, R83.1
- removed net BCK_ADC: IC1.BCK, U1.GPIO27/GPIO_GEN2
- removed net CLK_ADC: IC1.SCKI, U1.GPIO4/GPIO_GCKL
- removed net CS0_0: U$2.~CS, U6.S1
- removed net CS0_1: U$5.~CS, U6.S2
- removed net CS0_2: U$8.~CS, U1.GPIO12, U6.D, U6.S3
- removed net CS0_3: U$11.~CS, U6.S4
- removed net CS1_0: U$3.!CS, U8.S1
- removed net CS1_1: U$6.!CS, U8.S2
- removed net CS1_2: U$9.!CS, U1.GPIO13, U8.D, U8.S3
- removed net CS1_3: U$12.!CS, U8.S4
- removed net CS2_0: U$4.!CS, U7.S1
- removed net CS2_1: U$7.!CS, U7.S2
- removed net CS2_2: U7.S3
- removed net CS2_3: U$13.!CS, U7.S4
- removed net DGND: C1.2, C2.2, U1.GND, U1.SHIELD, U6.GND, U7.GND, U8.GND, U9.A0, U9.A1, U9.A2, U9.GND, U9.RESET
- removed net DOUT_ADC: IC1.DOUT, U1.GPIO17/GPIO_GEN0
- removed net EOUT_0: C35.2, IC1.VINL2/VIN1M
- removed net EOUT_1: C42.2, IC1.VINL1/VIN1P
- removed net EOUT_2: C84.2, IC1.VINR3/VIN3P
- removed net EOUT_3: C91.2, IC1.VINR4/VIN3M
- removed net EQ0_CE: U$1.CE, U1.GPIO23/GPIO_GEN4
- removed net EQ0_CL: U$1.CL, U1.GPIO25/GPIO_GEN6
- removed net EQ0_DI: U$1.DI, U1.GPIO24/GPIO_GEN5
- removed net EQ1_CE: U$14.CE, U1.GPIO20
- removed net EQ1_CL: U$14.CL, U1.GPIO26
- removed net EQ1_DI: U$14.DI, U1.GPIO21
- removed net H_0_0: C45.1, R8.1, U2.H, U3.H, X7.N
- removed net H_0_1: C49.1, R20.1, U4.H, U5.H, X15.N
- removed net H_0_2: C53.1, R51.1, U10.H, U11.H, X24.N
- removed net H_0_3: C57.1, R73.1, U12.H, U13.H, X33.N
- removed net LRCK_ADC: IC1.LRCK, U1.GPIO18/GPIO_GEN1
- removed net L_0_0: R15.1, U2.L
- removed net L_0_1: R27.1, U4.L
- removed net L_0_2: R55.1, U10.L
- removed net L_0_3: R77.1, U12.L
- removed net L_1_0: D4.C, U3.L
- removed net L_1_1: D15.C, U5.L
- removed net L_1_2: D26.C, U11.L
- removed net L_1_3: D37.C, U13.L
- removed net MUX0: U1.GPIO5, U6.A0, U7.A0, U8.A0
- removed net MUX1: U1.GPIO6, U6.A1, U7.A1, U8.A1
- removed net N$10: C5.1, IC1.VREF
- removed net N$100: D22.C, R29.2, X15.P
- removed net N$101: R29.1, R33.2, X16.N
- removed net N$102: R36.1, X13.VOUT, X14.P
- removed net N$103: R36.2, R37.2, X13.N
- removed net N$104: D13.C, D6.A
- removed net N$105: C46.1, D13.A, D14.C, D21.A, R19.1, R40.2
- removed net N$106: D15.A, X15.VOUT
- removed net N$107: R40.1, R41.2, X17.P
- removed net N$108: D16.C, R41.1, X17.VOUT
- removed net N$109: D17.A, D18.C
- removed net N$11: C6.1, C7.1, IC1.LDO
- removed net N$110: D16.A, D17.C
- removed net N$111: D18.A, D19.C, R33.1, R44.1, X13.P
- removed net N$112: R44.2, X18.P, X18.VOUT
- removed net N$113: C47.1, R42.2
- removed net N$114: D20.A, D21.C
- removed net N$115: D19.A, D20.C
- removed net N$116: D22.A, X16.VOUT
- removed net N$118: R26.2
- removed net N$119: C49.2
- removed net N$12: C24.1, C9.1, U$1.LLC4
- removed net N$120: R45.2, R46.1, X20.N
- removed net N$121: X20.P, X20.VOUT
- removed net N$122: R49.2, R51.2, X21.P
- removed net N$123: C58.1, U$14.LLC1
- removed net N$124: C59.1, C74.1, U$14.LLC4
- removed net N$125: C60.1, U$14.LLMC1
- removed net N$126: C61.1, U$14.LLMC4
- removed net N$127: C62.1, U$14.LHMC1
- removed net N$128: C63.1, U$14.LHMC4
- removed net N$129: C64.1, U$14.LHC1
- removed net N$13: C10.1, U$1.LLMC1
- removed net N$130: C65.1, U$14.LHC4
- removed net N$131: R52.2, R53.1, X21.N
- removed net N$132: D33.C, R56.2, X24.P
- removed net N$133: C66.1, U$14.RHC4
- removed net N$134: C67.1, U$14.RHC1
- removed net N$135: R56.1, R57.2, X25.N
- removed net N$136: R58.1, X22.VOUT, X23.P
- removed net N$137: R58.2, R59.2, X22.N
- removed net N$138: D23.A, D24.C
- removed net N$139: C50.1, D24.A, D25.C, D32.A, R50.1, R62.2
- removed net N$14 (its old number): C11.1, U$1.LLMC4
- removed net N$140: D26.A, X24.VOUT
- removed net N$141: R62.1, R63.2, X26.P
- removed net N$142: D27.C, R63.1, X26.VOUT
- removed net N$143: D28.A, D29.C
- removed net N$144: D27.A, D28.C
- removed net N$145: D29.A, D30.C, R57.1, R66.1, X22.P
- removed net N$146: R66.2, X27.P, X27.VOUT
- removed net N$147: C51.1, R64.2
- removed net N$148: D31.A, D32.C
- removed net N$149: D30.A, D31.C
- removed net N$15 (its old number): C12.1, U$1.LHMC1
- removed net N$150: D33.A, X25.VOUT
- removed net N$152: R54.2
- removed net N$153: C53.2
- removed net N$154: R72.2, X28.VOUT
- removed net N$155: C54.2, D34.C, D36.A, R69.2, X28.P
- removed net N$156: R67.2, R68.1, X29.N
- removed net N$157: X29.P, X29.VOUT
- removed net N$158: R71.2, R73.2, X30.P
- removed net N$159: R74.2, R75.1, X30.N
- removed net N$16 (its old number): C13.1, U$1.LHMC4
- removed net N$160: D44.C, R78.2, X33.P
- removed net N$161: R78.1, R79.2, X34.N
- removed net N$162: R80.1, X31.VOUT, X32.P
- removed net N$163: R80.2, R81.2, X31.N
- removed net N$164: D34.A, D35.C
- removed net N$165: C54.1, D35.A, D36.C, D43.A, R72.1, R84.2
- removed net N$166: D37.A, X33.VOUT
- removed net N$167: R84.1, R85.2, X35.P
- removed net N$168: D38.C, R85.1, X35.VOUT
- removed net N$169: D39.A, D40.C
- removed net N$17: C14.1, U$1.LHC1
- removed net N$170: D38.A, D39.C
- removed net N$171: D40.A, D41.C, R79.1, R88.1, X31.P
- removed net N$172: R88.2, X36.P, X36.VOUT
- removed net N$173: C55.1, R86.2
- removed net N$174: D42.A, D43.C
- removed net N$175: D41.A, D42.C
- removed net N$176: D44.A, X34.VOUT
- removed net N$178: R76.2
- removed net N$179: C57.2
- removed net N$18 (its old number): C15.1, U$1.LHC4
- removed net N$180: C68.1, U$14.RHMC4
- removed net N$181: C69.1, U$14.RHMC1
- removed net N$182: C70.1, U$14.RLMC4
- removed net N$183: C71.1, U$14.RLMC1
- removed net N$184: C72.1, U$14.RLC4
- removed net N$185: C73.1, U$14.RLC1
- removed net N$186: C58.2, U$14.LLC2
- removed net N$187: C59.2, C74.2, C75.2, U$14.LLC3
- removed net N$188: C75.1, U$14.LLC5
- removed net N$189: C76.1, U$14.LLMC5
- removed net N$19 (its old number): C16.1, U$1.RHC4
- removed net N$190: C77.1, U$14.LHMC5
- removed net N$191: C78.1, U$14.LHC5
- removed net N$192: C79.1, U$14.V_REF
- removed net N$193: C80.1, U$14.RHC5
- removed net N$194: C81.1, U$14.RHMC5
- removed net N$195: C82.1, U$14.RLMC5
- removed net N$196: C83.1, U$14.RLC5
- removed net N$197: C84.1, U$14.ROUT
- removed net N$198: C85.1, U$14.RBOOS2
- removed net N$199: C86.1, U$14.RIN
- removed net N$20 (its old number): C17.1, U$1.RHC1
- removed net N$200: C87.1, U$14.RCUT2
- removed net N$201: C88.1, U$14.LCUT1
- removed net N$202: C89.1, U$14.LIN
- removed net N$203: C90.1, U$14.LBOOS1
- removed net N$204: C91.1, U$14.LOUT
- removed net N$205: C60.2, U$14.LLMC2
- removed net N$206: C61.2, C76.2, U$14.LLMC3
- removed net N$207: C62.2, U$14.LHMC2
- removed net N$208: C63.2, C77.2, U$14.LHMC3
- removed net N$209: C64.2, U$14.LHC2
- removed net N$210: C65.2, C78.2, U$14.LHC3
- removed net N$211: C66.2, C80.2, U$14.RHC3
- removed net N$212: C67.2, U$14.RHC2
- removed net N$213: C68.2, C81.2, U$14.RHMC3
- removed net N$214: C69.2, U$14.RHMC2
- removed net N$215: C70.2, C82.2, U$14.RLMC3
- removed net N$216: C71.2, U$14.RLMC2
- removed net N$217: C72.2, C83.2, U$14.RLC3
- removed net N$218: C73.2, U$14.RLC2
- removed net N$219: C85.2, U$14.RBOOS1
- removed net N$22 (its old number): C19.1, U$1.RHMC1
- removed net N$220: C86.2
- removed net N$221: C87.2, U$14.RCUT1
- removed net N$222: C88.2, U$14.LCUT2
- removed net N$223: C89.2
- removed net N$224: C90.2, U$14.LBOOS2
- removed net N$23 (its old number): C20.1, U$1.RLMC4
- removed net N$24 (its old number): C21.1, U$1.RLMC1
- removed net N$25 (its old number): C22.1, U$1.RLC4
- removed net N$26 (its old number): C23.1, U$1.RLC1
- removed net N$27 (its old number): C8.2, U$1.LLC2
- removed net N$28: C24.2, C26.2, C9.2, U$1.LLC3
- removed net N$29: C26.1, U$1.LLC5
- removed net N$31 (its old number): C28.1, U$1.LHMC5
- removed net N$32 (its old number): C29.1, U$1.LHC5
- removed net N$33 (its old number): C30.1, U$1.V_REF
- removed net N$34: C31.1, U$1.RHC5
- removed net N$35: C32.1, U$1.RHMC5
- removed net N$36: C33.1, U$1.RLMC5
- removed net N$37: C34.1, U$1.RLC5
- removed net N$38: C35.1, U$1.ROUT, U$11.~RS, U$2.~RS, U$5.~RS, U$8.~RS
- removed net N$39: C36.1, U$1.RBOOS2, U$11.~SHDN, U$2.~SHDN, U$5.~SHDN, U$8.~SHDN
- removed net N$40: C37.1, U$1.RIN
- removed net N$41: C38.1, U$1.RCUT2
- removed net N$42: C39.1, U$1.LCUT1
- removed net N$43: C40.1, U$1.LIN
- removed net N$44: C41.1, U$1.LBOOS1
- removed net N$45: C42.1, U$1.LOUT
- removed net N$46: C10.2, U$1.LLMC2
- removed net N$47: C11.2, C27.2, U$1.LLMC3
- removed net N$48: C12.2, U$1.LHMC2
- removed net N$49: C13.2, C28.2, U$1.LHMC3
- removed net N$50: C14.2, U$1.LHC2
- removed net N$51: C15.2, C29.2, U$1.LHC3
- removed net N$53: C25.2, D1.C, D3.A, R3.2, X1.P
- removed net N$54: R1.2, R2.1, X2.N
- removed net N$55: X2.P, X2.VOUT
- removed net N$59: C16.2, C31.2, U$1.RHC3
- removed net N$60: C17.2, U$1.RHC2
- removed net N$61: C18.2, C32.2, U$1.RHMC3
- removed net N$62: C19.2, U$1.RHMC2
- removed net N$63: C20.2, C33.2, U$1.RLMC3
- removed net N$64: C21.2, U$1.RLMC2
- removed net N$65: C22.2, C34.2, U$1.RLC3
- removed net N$66: C23.2, U$1.RLC2
- removed net N$67: C36.2, U$1.RBOOS1
- removed net N$68: C37.2
- removed net N$69: C38.2, U$1.RCUT1
- removed net N$70: C39.2, U$1.LCUT2
- removed net N$71: C40.2
- removed net N$72: C41.2, U$1.LBOOS2
- removed net N$73: R50.2, X19.VOUT
- removed net N$74: C50.2, D23.C, D25.A, R47.2, X19.P
- removed net N$79: C25.1, D12.A, D2.A, D3.C, R28.2, R7.1
- removed net N$87: C43.1, R32.2
- removed net N$9: C8.1, U$1.LLC1
- removed net N$92: R11.2
- removed net N$93: C45.2
- removed net N$94: R19.2, X4.VOUT
- removed net N$95: C46.2, D14.A, D6.C, R13.2, X4.P
- removed net N$96: R12.1, R5.2, X11.N
- removed net N$97: X11.P, X11.VOUT
- removed net N$98: R17.2, R20.2, X12.P
- removed net N$99: R22.2, R23.1, X12.N
- removed net P0A_0_0: U$3.P0A
- removed net P0A_0_1: U$6.P0A
- removed net P0A_0_2: U$9.P0A
- removed net P0A_0_3: U$12.P0A
- removed net P0A_1_0: R34.1, U$4.P0A
- removed net P0A_1_1: R43.1, U$7.P0A
- removed net P0A_1_2: R65.1, U$10.P0A
- removed net P0A_1_3: R87.1, U$13.P0A
- removed net P0B_0_0: U$3.P0B
- removed net P0B_0_1: U$6.P0B
- removed net P0B_0_2: U$9.P0B
- removed net P0B_0_3: U$12.P0B
- removed net P0B_1_0: R32.1, U$4.P0B, X10.N
- removed net P0B_1_1: R42.1, U$7.P0B, X18.N
- removed net P0B_1_2: R64.1, U$10.P0B, X27.N
- removed net P0B_1_3: R86.1, U$13.P0B, X36.N
- removed net P0W_0_0: U$3.P0W
- removed net P0W_0_1: U$6.P0W
- removed net P0W_0_2: U$9.P0W
- removed net P0W_0_3: U$12.P0W
- removed net PA0_0_0: R10.2, U$2.PA0, X3.VOUT
- removed net PA0_1: R23.2, U$5.PA0, X12.VOUT
- removed net PA0_2: R53.2, U$8.PA0, X21.VOUT
- removed net PA0_3: R75.2, U$11.PA0, X30.VOUT
- removed net PA1_0: R25.2, U$2.PA1, X6.N
- removed net PA1_1: R38.2, U$5.PA1, X14.N
- removed net PA1_2: R60.2, U$8.PA1, X23.N
- removed net PA1_3: R82.2, U$11.PA1, X32.N
- removed net PB0_0: R4.2, U$2.PB0, X1.N
- removed net PB0_1: R14.2, U$5.PB0, X4.N
- removed net PB0_2: R48.2, U$8.PB0, X19.N
- removed net PB0_3: R70.2, U$11.PB0, X28.N
- removed net PB1_0_0: C44.2, U$2.PB1, X6.VOUT
- removed net PB1_1: C48.2, U$5.PB1, X14.VOUT
- removed net PB1_2: C52.2, U$8.PB1, X23.VOUT
- removed net PB1_3: C56.2, U$11.PB1, X32.VOUT
- removed net SCL_0: U2.SCL, U3.SCL, U9.SC0
- removed net SCL_1: U4.SCL, U5.SCL, U9.SD0
- removed net SCL_2: U10.SCL, U11.SCL, U9.SC2
- removed net SCL_3: U12.SCL, U13.SCL, U9.SD2
- removed net SDA_0: U2.SDA, U3.SDA, U9.SC1
- removed net SDA_1: U4.SDA, U5.SDA, U9.SD1
- removed net SDA_2: U10.SDA, U11.SDA, U9.SC3
- removed net SDA_3: U12.SDA, U13.SDA, U9.SD3
- removed net SO_0: U$2.SO
- removed net SO_1: U$5.SO
- removed net SO_2: U$8.SO
- removed net SO_3: U$11.SO
- new net AIN: C2.2
- new net AOUT: C3.1, R30.1
- new net AOUT1+: X4.2, X4.T
- new net AOUT1-: X4.3, X4.R
- new net CS0: U$1.~CS
- new net CS1: U$2.!CS
- new net GND: X4.1, X4.G, X4.S
- new net H_0: C4.1, R8.1, U1.H, U2.H, X7.N
- new net L_0: R15.1, U1.L
- new net L_1: D4.C, U2.L
- new net N$3: C1.2, D1.C, D3.A, R3.2, X1.P
- new net P0A_0: R11.2, U$2.P0A
- new net P0A_1: R34.1, U$3.P0A
- new net P0B_0: R1.2, U$2.P0B
- new net P0B_1: R32.1, U$3.P0B, X10.N
- new net P0W_0: R9.1, U$2.P0W
- new net PA0: R10.2, U$1.PA0, X3.VOUT
- new net PA1: R25.2, U$1.PA1, X6.N
- new net PB0: R4.2, U$1.PB0, X1.N
- new net PB1: C3.2, U$1.PB1, X6.VOUT
- new net RS: U$1.~RS
- new net SHDN: U$1.~SHDN
- new net VSS: R30.2, U$1.VSS, U$2.VSS, U$3.VSS, U1.A0, U1.EPAD, U1.GND, U2.EPAD, U2.GND, X1.VSS, X10.VSS, X3.VSS, X5.VSS, X6.VSS, X7.VSS, X8.VSS, X9.VSS
- net CS2: now also U$3.!CS; no longer U$10.!CS, U1.GPIO16, U7.D
- net N$21: now also C1.1, D12.A, D2.A, D3.C, R28.2, R7.1; no longer C18.1, U$1.RHMC4
- net N$30: now also C2.1, R32.2; no longer C27.1, U$1.LLMC5
- net SCK: now also U$1.SCK; no longer U$10.SCK, U$11.SCK, U$12.SCK, U$13.SCK, U$4.SCK, U$5.SCK, U$6.SCK, U$7.SCK, U$8.SCK, U$9.SCK, U1.GPIO11/SPI_SCLK
- net SCL: now also U1.SCL, U2.SCL; no longer IC1.MC/SCL, U1.GPIO3/SCL1, U9.SCL
- net SDA: now also U1.SDA, U2.SDA; no longer IC1.MOSI/SDA, U1.GPIO2/SDA1, U9.SDA
- net SDI/O: now also U$1.SI, U$2.SDI/SDO; no longer U$10.SDI/SDO, U$11.SI, U$12.SDI/SDO, U$13.SDI/SDO, U$2.SI, U$4.SDI/SDO, U$5.SI, U$6.SDI/SDO, U$7.SDI/SDO, U$8.SI, U$9.SDI/SDO, U1.GPIO10/SPI_MOSI
- net VDD: now also U$1.VDD, U1.VDD, U2.A0, X3.VDD, X5.VDD, X6.VDD, X7.VDD; no longer R12.2, R2.2, R26.1, R46.2, R54.1, R68.2, R76.1, U$10.VDD, U$11.VDD, U$12.VDD, U$13.VDD, U$4.VDD, U$5.VDD, U$6.VDD, U$7.VDD, U$8.VDD, U$9.VDD, U10.VDD, U11.A0, U11.VDD, U12.VDD, U13.A0, U13.VDD, U3.A0, U3.VDD, U4.VDD, U5.A0, U5.VDD, X11.VDD, X12.VSS, X13.VSS, X14.VSS, X15.VSS, X16.VDD, X17.VDD, X18.VDD, X19.VDD, X2.VDD, X20.VDD, X21.VSS, X22.VSS, X23.VSS, X24.VSS, X25.VDD, X26.VDD, X27.VDD, X28.VDD, X29.VDD, X3.VSS, X30.VSS, X31.VSS, X32.VSS, X33.VSS, X34.VDD, X35.VDD, X36.VDD, X4.VDD, X5.VSS, X6.VSS, X7.VSS
- net VREF: now also C4.2, R1.1, R15.2, R24.1, R25.1, R3.1, R34.2, R6.1, X9.N; no longer R14.1, R48.1, R70.1
Other:
- moved on the sheet: C1, C2, C3, C4, D1, D10, D11, D12, D2, D3, D4, D5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
