File: combined.sch (EAGLE design)
At the start: 46 parts, among them U1 MAX5419LETA+, U2 MAX5419LETA+, U3 LM4562MAX/NOPB, U4 LM4562MAX/NOPB, U5 LM4562MAX/NOPB, U6 LM4562MAX/NOPB

Commit message: finish compressor routing, and sloppy combined routing
Parts:
- removed AIN, GND: (no value), wirepad:SMD5
- removed D1, D10, D11, D12, D2, D3, D4, D5, D7, D8, D9: 1N4148W-TP, 1N4148W-TP:1N4148W-TP
- removed R34: 10k, rcl:R-US_R0402
- removed R35: 100k, rcl:R-US_R0402
- removed U$2, U$3: MCP4131-503E/SN, MCP4131-503E_SN:MCP4131-503E/SN
- removed U4, U5, U6: LM4562MAX/NOPB, LM4562MAX_NOPB:LM4562MAX/NOPB
- added C58, C59, C60, C61, C62, C63, C64, C65, C66, C67, C68, C69, C70, C71, C72, C73: 0.047uF, rcl:C-USC0402
- added C75, C76, C77, C78, C79, C80, C81, C82, C83, C84, C85, C86, C87, C88, C89, C90, C91: 10uF, rcl:C-USC0402
- added R1, R2, R20: 1k, rcl:R-US_R0402
- added R12, R13, R14, R5: 5k, rcl:R-US_R0402
- added R17, R19, R26: 20k, rcl:R-US_R0402
- added R22, R23: 10k, rcl:R-US_R0402
- added R27: 6k, rcl:R-US_R0402
- added R29: 4k, rcl:R-US_R0402
- added U$14: LC75281E, LC75281E:LC75281E
- C1: value 680p -> 0.1u
- C2: value 0.1 -> 0.1u
- C3, C4: value 1.5u -> 0.1u
- R10, R9: value 100k -> 5k
- R11: value 10k -> 5k
- R15, R16, R18: value 100k -> 20k
- R21, R31, R32: value 100k -> 1.5M
- R25: value 20k -> 4k
- R28: value 100k -> 6k
- R3: value 100k -> 1k
- R30: value 1M -> 20k
- R4: value 10k -> 1.7k
- R6, R8: value 470k -> 20k
- R7: value 1k -> 5k
- U$1: value MCP42100-I/P -> MCP4131-503E/SN; device MCP42100-I_P:MCP42100-I/P -> MCP4131-503E_SN:MCP4131-503E/SN; SPICEPREFIX (none) -> X
- U1, U2: value MAX5419LETA+ -> LM4562MAX/NOPB; device MAX5419LETA_:MAX5419LETA+ -> LM4562MAX_NOPB:LM4562MAX/NOPB
Connections:
- removed net CS0: U$1.~CS
- removed net CS1: U$2.!CS
- removed net CS2: U$3.!CS
- removed net H_0: C4.1, R8.1, U1.H, U2.H, U3.NEG_B
- removed net L_0: R15.1, U1.L
- removed net L_1: D4.C, U2.L
- removed net N$18: R21.1, U6.OUT_A, U6.POS_B
- removed net N$19: R21.2, R24.2, U6.NEG_A
- removed net N$21: C1.1, D12.A, D2.A, D3.C, R28.2, R7.1
- removed net N$24: D8.A, D9.C
- removed net N$25: D7.A, D8.C
- removed net N$26: D10.C, D9.A, R18.1, R35.1, U6.POS_A
- removed net N$27: R35.2, U4.OUT_B, U4.POS_B
- removed net N$31: D11.A, D12.C
- removed net N$32: D10.A, D11.C
- removed net P0A_0: R11.2, U$2.P0A
- removed net P0A_1: R34.1, U$3.P0A
- removed net P0B_1: R32.1, U$3.P0B, U4.NEG_B
- removed net P0W_0: R9.1, U$2.P0W
- removed net PA0: R10.2, U$1.PA0, U4.OUT_A
- removed net PA1: R25.2, U$1.PA1, U6.NEG_B
- removed net PB0: R4.2, U$1.PB0, U3.POS_A
- removed net PB1: C3.2, U$1.PB1, U6.OUT_B
- removed net RS: U$1.~RS
- removed net SCL: U1.SCL, U2.SCL
- removed net SDA: U1.SDA, U2.SDA
- removed net SHDN: U$1.~SHDN
- new net 3V3A: U1.NEG_A, U1.OUT_A
- new net AIN0: R13.1
- new net AIN1: R14.1
- new net AIN2: R7.1
- new net AIN3: R5.1
- new net AOUTL: C3.2, R31.2
- new net AOUTR: C2.2, R32.2
- new net CS: U$1.!CS
- new net EIN0: C86.2
- new net EIN1: C89.2
- new net EOUT0: C84.2
- new net EOUT1: C91.2
- new net EQ1_CE: U$14.CE
- new net EQ1_CL: U$14.CL
- new net EQ1_DI: U$14.DI
- new net GND: C79.2, R1.1, R3.1, U$14.TEST, U$14.V_SS, U1.V-
- new net N$123: C58.1, U$14.LLC1
- new net N$125: C60.1, U$14.LLMC1
- new net N$126: C61.1, U$14.LLMC4
- new net N$127: C62.1, U$14.LHMC1
- new net N$128: C63.1, U$14.LHMC4
- new net N$129: C64.1, U$14.LHC1
- new net N$13: R13.2, R6.1, R9.2
- new net N$130: C65.1, U$14.LHC4
- new net N$133: C66.1, U$14.RHC4
- new net N$134: C67.1, U$14.RHC1
- new net N$17: R10.1, R14.2, R8.1
- new net N$180: C68.1, U$14.RHMC4
- new net N$181: C69.1, U$14.RHMC1
- new net N$182: C70.1, U$14.RLMC4
- new net N$183: C71.1, U$14.RLMC1
- new net N$184: C72.1, U$14.RLC4
- new net N$185: C73.1, U$14.RLC1
- new net N$186: C58.2, U$14.LLC2
- new net N$187: C59.2, C75.2, U$14.LLC3
- new net N$188: C75.1, U$14.LLC5
- new net N$189: C76.1, U$14.LLMC5
- new net N$190: C77.1, U$14.LHMC5
- new net N$191: C78.1, U$14.LHC5
- new net N$192: C79.1, U$14.V_REF
- new net N$193: C80.1, U$14.RHC5
- new net N$194: C81.1, U$14.RHMC5
- new net N$195: C82.1, U$14.RLMC5
- new net N$196: C83.1, U$14.RLC5
- new net N$197: C84.1, U$14.ROUT
- new net N$198: C85.1, U$14.RBOOS2
- new net N$199: C86.1, U$14.RIN
- new net N$200: C87.1, U$14.RCUT2
- new net N$201: C88.1, U$14.LCUT1
- new net N$202: C89.1, U$14.LIN
- new net N$203: C90.1, U$14.LBOOS1
- new net N$204: C91.1, U$14.LOUT
- new net N$205: C60.2, U$14.LLMC2
- new net N$206: C61.2, C76.2, U$14.LLMC3
- new net N$207: C62.2, U$14.LHMC2
- new net N$208: C63.2, C77.2, U$14.LHMC3
- new net N$209: C64.2, U$14.LHC2
- new net N$210: C65.2, C78.2, U$14.LHC3
- new net N$211: C66.2, C80.2, U$14.RHC3
- new net N$212: C67.2, U$14.RHC2
- new net N$213: C68.2, C81.2, U$14.RHMC3
- new net N$214: C69.2, U$14.RHMC2
- new net N$215: C70.2, C82.2, U$14.RLMC3
- new net N$216: C71.2, U$14.RLMC2
- new net N$217: C72.2, C83.2, U$14.RLC3
- new net N$218: C73.2, U$14.RLC2
- new net N$219: C85.2, U$14.RBOOS1
- new net N$221: C87.2, U$14.RCUT1
- new net N$222: C88.2, U$14.LCUT2
- new net N$224: C90.2, U$14.LBOOS2
- new net N$5: R18.1, R19.2, U2.NEG_A
- new net N$50: C4.2, R22.2, R23.2, R24.2
- new net N$51: R25.1, U3.POS_A
- new net N$9: C3.1, R30.2, U3.OUT_A
- new net P0A: R24.1, R25.2, U$1.P0A
- new net P0B: R23.1, R29.1, U$1.P0B
- new net P0W: R27.2, R28.1, R30.1, U$1.P0W
- net AIN: now also C4.1; no longer AIN.P, C2.2
- net AOUT: now also C1.2, R21.2; no longer C3.1, R30.1
- net N$1: now also R3.2, R4.2, U1.POS_A; no longer R7.2, U3.OUT_A
- net N$14: now also R15.2, R16.2, R17.1, R6.2, R8.2, U2.NEG_B; no longer D4.A, U3.OUT_B
- net N$15: now also R12.1, R16.1, R5.2; no longer D5.C, R16.2, U3.POS_B
- net N$16: now also R11.1, R15.1, R7.2; no longer R16.1, R18.2, U5.NEG_A
- net N$2: now also R1.2, R2.2, U1.POS_B; no longer D7.C, R31.1, U5.OUT_B
- net N$20: now also R18.2, R20.1, U2.OUT_A; no longer D1.A, D2.C
- net N$3: now also C59.1, U$14.LLC4; no longer C1.2, D1.C, D3.A, R3.2, U3.NEG_A
- net N$30: now also R29.2, U3.POS_B; no longer C2.1, R32.2
- net N$4: now also C1.1, R17.2, R19.1, R20.2, U2.OUT_B; no longer D5.A, U5.OUT_A
- net N$6: now also R27.1, U3.NEG_A; no longer R6.2, R8.2, U4.POS_A
- net N$7: now also R26.2, R28.2, U3.NEG_B; no longer R10.1, R9.2, U4.NEG_A
- net N$8: now also C2.1, R26.1, U3.OUT_B; no longer R28.1, R31.2, U5.POS_B
- net SCK: no longer U$2.SCK, U$3.SCK
- net SDI/O: now also U$1.SDI/SDO; no longer U$1.SI, U$2.SDI/SDO, U$3.SDI/SDO
- net VDD: now also R2.1, R4.1, U$14.V_DD, U1.V+, U2.V+; no longer R11.1, U$1.VDD, U$2.VDD, U$3.VDD, U1.VDD, U2.A0, U2.VDD, U4.V+, U5.V+, U6.V+
- net VREF: now also R10.2, R11.2, R12.2, R22.1, R9.1, U$1.VDD, U1.NEG_B, U1.OUT_B, U2.POS_A, U2.POS_B; no longer C4.2, R15.2, R24.1, R25.1, R3.1, R34.2, R4.1, R6.1, U$2.P0B, U5.NEG_B, U5.POS_A
- net VSS: now also R21.1, R31.1, R32.1, U2.V-; no longer GND.P, R30.2, U$2.VSS, U$3.VSS, U1.A0, U1.EPAD, U1.GND, U2.EPAD, U2.GND, U4.V-, U5.V-, U6.V-
Other:
- moved on the sheet: C1, C2, C3, R10, R11, R15, R16, R18, R21, R24, R25, R28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

Commit message: corrections
Parts:
- removed C1, C2, C3: 0.1u, rcl:C-USC0402
- removed C59, C60, C72, C73: 0.047uF, rcl:C-USC0402
- removed C75, C76, C77, C78, C79, C80, C81, C82, C83, C84, C85, C86, C87, C88, C89, C90, C91: 10uF, rcl:C-USC0402
- removed R10, R11, R7, R9: 5k, rcl:R-US_R0402
- removed R15, R16, R18, R6, R8: 20k, rcl:R-US_R0402
- removed R3: 1k, rcl:R-US_R0402
- removed R4: 1.7k, rcl:R-US_R0402
- removed U$1: MCP4131-503E/SN, MCP4131-503E_SN:MCP4131-503E/SN
- removed U1: LM4562MAX/NOPB, LM4562MAX_NOPB:LM4562MAX/NOPB
- added 3V3_D1, 9VDD1, BCK_ADC1, CE_EQ1, CE_EQ2, CLK_ADC1, CL_EQ1, CL_EQ2, CS3, CS4, CS5, DI_EQ1, DI_EQ2, DOUT_ADC1, GND5, GND7, LRCK_ADC1, MUX2, MUX3, SCK1, SCL1, SDA1, SDI/O1: (no value), wirepad:SMD2
- added AIN1, AIN2, AIN3, AIN5, AOUT1, AOUT2, GND1, GND2, GND3, GND4, GND6, GND8: (no value), wirepad:SMD5
- added C10, C11, C139, C140, C141, C143, C51, C52, C53, C55, C57, C9: 0.1u, rcl:C-USC0402
- added C103, C104, C105, C106, C107, C108, C109, C110, C111, C112, C113, C114, C115, C116, C117, C118, C17, C18, C19, C20, C21, C22, C23, C24, C25, C26, C27, C28, C29, C30, C31, C32: 0.047uF, rcl:C-USC0402
- added C119, C120, C121, C122, C123, C124, C125, C126, C127, C128, C129, C130, C131, C132, C133, C134, C135, C33, C34, C35, C36, C37, C38, C39, C40, C41, C42, C43, C44, C45, C46, C47, C48, C49: 10uF, rcl:C-USC0402
- added C12, C13, C5: 680p, rcl:C-USC0402
- added C14, C50, C6: 0.1, rcl:C-USC0402
- added C15, C16, C54, C56, C7, C8: 1.5u, rcl:C-USC0402
- added D13, D14, D15, D16, D17, D18, D19, D20, D21, D22, D23, D24, D25, D26, D27, D28, D29, D30, D31, D32, D33, D34, D35, D36, D37, D38, D39, D40, D41, D42, D43, D44, D56, D57, D58, D59, D6, D60, D61, D62, D63, D64, D65, D66: 1N4148W-TP, 1N4148W-TP:1N4148W-TP
- added IC2: PCM1865DBT, PCM1865DBT:PCM1865DBT
- added R100, R119, R144, R149, R150, R152, R153, R154, R155, R159, R160, R161, R163, R36, R37, R38, R40, R52, R61, R66, R67, R69, R70, R71, R72, R76, R77, R78, R80, R88, R89, R91, R92, R93, R94, R98, R99: 100k, rcl:R-US_R0402
- added R101, R137, R138, R139, R145, R151, R156, R162, R39, R43, R44, R45, R53, R54, R55, R56, R62, R68, R73, R79, R90, R95: 10k, rcl:R-US_R0402
- added R102, R104, R106, R107, R108, R109, R110, R111, R185, R187, R189, R190, R191, R192, R193, R194: 5k, rcl:R-US_R0402
- added R103, R105, R112, R113, R114, R115, R116, R141, R157, R165, R186, R188, R195, R196, R197, R198, R199, R35, R47, R51, R58, R74, R82, R96: 20k, rcl:R-US_R0402
- added R117, R123, R124, R125, R147, R200, R64, R86: 1k, rcl:R-US_R0402
- added R118, R120, R121, R166, R167, R201, R41, R42, R83, R84: 1.5M, rcl:R-US_R0402
- added R126: 1.7k, rcl:R-US_R0402
- added R140, R164, R34, R46, R50, R57, R81: 4k, rcl:R-US_R0402
- added R142, R143, R48, R49, R59, R60: 6k, rcl:R-US_R0402
- added R146, R148, R63, R65, R85, R87: 470k, rcl:R-US_R0402
- added R158, R33, R75, R97: 1M, rcl:R-US_R0402
- added U$10, U$19, U$4, U$9: MCP42100-I/P, MCP42100-I_P:MCP42100-I/P
- added U$11, U$12, U$15, U$18, U$2, U$20, U$21, U$3, U$5, U$6, U$7: MCP4131-503E/SN, MCP4131-503E_SN:MCP4131-503E/SN
- added U$13, U$16: LC75281E, LC75281E:LC75281E
- added U10, U11, U12, U13, U15, U21, U22, U23, U24, U28, U29, U30, U31, U32, U4, U41, U42, U43, U44, U6, U9: LM4562MAX/NOPB, LM4562MAX_NOPB:LM4562MAX/NOPB
- added U16, U19, U20, U27, U39, U40, U7, U8: MAX5419LETA+, MAX5419LETA_:MAX5419LETA+
- added U17, U18, U25: TMUX1204DGSR, TMUX1204DGSR:TMUX1204DGSR
- added U26: TCA9546ADR, TCA9546ADR:TCA9546ADR
- C58: value 0.047uF -> 0.1u
- C61: value 0.047uF -> 680p
- C62: value 0.047uF -> 0.1
- C63, C65, C68: value 0.047uF -> 0.1μF
- C64, C66: value 0.047uF -> 10μF
- C67, C69: value 0.047uF -> 1μF
- C70, C71: value 0.047uF -> 1.5u
- R1, R20: value 1k -> 100k
- R12: value 5k -> 1k
- R13, R5: value 5k -> 470k
- R14: value 5k -> 100k
- R17, R26: value 20k -> 100k
- R19: value 20k -> 10k
- R2: value 1k -> 10k
- R21: value 1.5M -> 10k
- R22, R23: value 10k -> 100k
- R25: value 4k -> 10k
- R27: value 6k -> 10k
- R28: value 6k -> 4k
- R29: value 4k -> 20k
- R31, R32: value 1.5M -> 6k
- U$14: value LC75281E -> MCP4131-503E/SN; device LC75281E:LC75281E -> MCP4131-503E_SN:MCP4131-503E/SN
Connections:
- removed net EQ1_CE: U$14.CE
- removed net EQ1_CL: U$14.CL
- removed net EQ1_DI: U$14.DI
- removed net N$123: C58.1, U$14.LLC1
- removed net N$125: C60.1, U$14.LLMC1
- removed net N$126: C61.1, U$14.LLMC4
- removed net N$127: C62.1, U$14.LHMC1
- removed net N$128: C63.1, U$14.LHMC4
- removed net N$129: C64.1, U$14.LHC1
- removed net N$130: C65.1, U$14.LHC4
- removed net N$134: C67.1, U$14.RHC1
- removed net N$180: C68.1, U$14.RHMC4
- removed net N$183: C71.1, U$14.RLMC1
- removed net N$184: C72.1, U$14.RLC4
- removed net N$185: C73.1, U$14.RLC1
- removed net N$186: C58.2, U$14.LLC2
- removed net N$187: C59.2, C75.2, U$14.LLC3
- removed net N$188: C75.1, U$14.LLC5
- removed net N$189: C76.1, U$14.LLMC5
- removed net N$190: C77.1, U$14.LHMC5
- removed net N$192: C79.1, U$14.V_REF
- removed net N$193: C80.1, U$14.RHC5
- removed net N$194: C81.1, U$14.RHMC5
- removed net N$195: C82.1, U$14.RLMC5
- removed net N$196: C83.1, U$14.RLC5
- removed net N$197: C84.1, U$14.ROUT
- removed net N$198: C85.1, U$14.RBOOS2
- removed net N$199: C86.1, U$14.RIN
- removed net N$200: C87.1, U$14.RCUT2
- removed net N$201: C88.1, U$14.LCUT1
- removed net N$202: C89.1, U$14.LIN
- removed net N$203: C90.1, U$14.LBOOS1
- removed net N$204: C91.1, U$14.LOUT
- removed net N$205: C60.2, U$14.LLMC2
- removed net N$206: C61.2, C76.2, U$14.LLMC3
- removed net N$207: C62.2, U$14.LHMC2
- removed net N$208: C63.2, C77.2, U$14.LHMC3
- removed net N$209: C64.2, U$14.LHC2
- removed net N$210: C65.2, C78.2, U$14.LHC3
- removed net N$212: C67.2, U$14.RHC2
- removed net N$214: C69.2, U$14.RHMC2
- removed net N$215: C70.2, C82.2, U$14.RLMC3
- removed net N$216: C71.2, U$14.RLMC2
- removed net N$217: C72.2, C83.2, U$14.RLC3
- removed net N$218: C73.2, U$14.RLC2
- removed net N$219: C85.2, U$14.RBOOS1
- removed net N$222: C88.2, U$14.LCUT2
- removed net N$224: C90.2, U$14.LBOOS2
- new net +3V3: 3V3_D1.P, U17.EN, U17.VDD, U18.EN, U18.VDD, U25.EN, U25.VDD, U26.VCC
- new net 3V3D: C63.1, C64.1, IC2.DVDD, IC2.IOVDD
- new net AIN01: R110.1
- new net AIN02: R193.1
- new net AIN11: R111.1
- new net AIN12: C53.1
- new net AIN123: R194.1
- new net AIN223: R187.1
- new net AIN31: C141.1
- new net AIN323: R185.1
- new net AIN33: AIN2.P, C50.2
- new net AIN4: AIN5.P, C62.2
- new net AIN45: C58.1
- new net AOUT1: AOUT1.P, C55.2, R118.2
- new net AOUT2: C15.1, R75.1
- new net AOUT23: AOUT2.P, C143.2, R201.2
- new net AOUT3: C54.1, R97.1
- new net AOUT4: C70.1, R158.1
- new net AOUTL1: C52.2, R83.2
- new net AOUTL3: C140.2, R166.2
- new net AOUTL4: C57.2, R120.2
- new net AOUTR1: C51.2, R84.2
- new net AOUTR3: C139.2, R167.2
- new net AOUTR4: C11.2, R121.2
- new net BCK_ADC: BCK_ADC1.P, IC2.BCK
- new net CLK_ADC: CLK_ADC1.P, IC2.SCKI
- new net CS0: U$4.~CS
- new net CS01: U$10.~CS
- new net CS03: U$9.~CS
- new net CS04: U$19.~CS
- new net CS0D: CS3.P, U17.D
- new net CS0_0: U17.S1
- new net CS0_1: U17.S2
- new net CS0_2: U17.S3
- new net CS0_3: U17.S4
- new net CS1: U$5.!CS, U$7.!CS
- new net CS11: U$11.!CS
- new net CS13: U$14.!CS
- new net CS14: U$20.!CS
- new net CS1D: CS4.P, U25.D
- new net CS1_0: U25.S1
- new net CS1_1: U25.S2
- new net CS1_2: U25.S3
- new net CS1_3: U25.S4
- new net CS2: U$6.!CS
- new net CS21: U$12.!CS
- new net CS23: U$15.!CS
- new net CS24: U$21.!CS
- new net CS2D: CS5.P, U18.D
- new net CS2_0: U18.S1
- new net CS2_1: U18.S2
- new net CS2_2: U18.S3
- new net CS2_3: U18.S4
- new net CS3: U$18.!CS
- new net CS4: U$3.!CS
- new net DGND: GND5.P, U17.GND, U18.GND, U25.GND, U26.A0, U26.A1, U26.A2, U26.GND, U26.RESET
- new net DOUT_ADC: DOUT_ADC1.P, IC2.DOUT
- new net EIN01: C130.2
- new net EIN11: C133.2
- new net EOUT01: C128.2
- new net EOUT11: C135.2
- new net EQ1_CE1: CE_EQ1.P, U$13.CE
- new net EQ1_CE2: CE_EQ2.P, U$16.CE
- new net EQ1_CL1: CL_EQ1.P, U$13.CL
- new net EQ1_CL2: CL_EQ2.P, U$16.CL
- new net EQ1_DI1: DI_EQ1.P, U$13.DI
- new net EQ1_DI2: DI_EQ2.P, U$16.DI
- new net H_0: C8.1, R13.1, U7.H, U8.H, U9.NEG_B
- new net H_01: C16.1, R65.1, U19.H, U20.H, U21.NEG_B
- new net H_03: C56.1, R87.1, U16.H, U27.H, U29.NEG_B
- new net H_04: C71.1, R148.1, U39.H, U40.H, U41.NEG_B
- new net LRCK_ADC: IC2.LRCK, LRCK_ADC1.P
- new net L_0: R20.1, U7.L
- new net L_01: R69.1, U19.L
- new net L_03: R91.1, U16.L
- new net L_04: R152.1, U39.L
- new net L_1: D15.C, U8.L
- new net L_11: D37.C, U20.L
- new net L_13: D26.C, U27.L
- new net L_14: D59.C, U40.L
- new net MUX0: MUX2.P, U17.A0, U18.A0, U25.A0
- new net MUX1: MUX3.P, U17.A1, U18.A1, U25.A1
- new net N$10: C10.2, R21.2, R24.2, R25.2
- new net N$100: C105.1, U$16.LLMC1
- new net N$101: C106.1, U$16.LLMC4
- new net N$102: D56.A, D57.C
- new net N$103: D61.A, D62.C
- new net N$104: D60.A, D61.C
- new net N$105: C62.1, R161.2
- new net N$106: D64.A, D65.C
- new net N$107: D63.A, D64.C
- new net N$108: C107.1, U$16.LHMC1
- new net N$109: C108.1, U$16.LHMC4
- new net N$11: R64.2, U21.OUT_A
- new net N$110: C109.1, U$16.LHC1
- new net N$111: C110.1, U$16.LHC4
- new net N$112: C111.1, U$16.RHC4
- new net N$113: C112.1, U$16.RHC1
- new net N$114: C113.1, U$16.RHMC4
- new net N$115: C114.1, U$16.RHMC1
- new net N$116: C115.1, U$16.RLMC4
- new net N$117: C116.1, U$16.RLMC1
- new net N$118: C117.1, U$16.RLC4
- new net N$119: C118.1, U$16.RLC1
- new net N$120: C103.2, U$16.LLC2
- new net N$121: C104.2, C119.2, U$16.LLC3
- new net N$122: C119.1, U$16.LLC5
- new net N$124: C120.1, U$16.LLMC5
- new net N$131: C121.1, U$16.LHMC5
- new net N$132: C122.1, U$16.LHC5
- new net N$135: C123.1, U$16.V_REF
- new net N$136: C124.1, U$16.RHC5
- new net N$137: C125.1, U$16.RHMC5
- new net N$138: C126.1, U$16.RLMC5
- new net N$139: C127.1, U$16.RLC5
- new net N$140: C128.1, U$16.ROUT
- new net N$141: D37.A, U21.OUT_B
- new net N$1413: R103.2, R105.2, R112.2, R113.2, R114.1, U6.NEG_B
- new net N$142: D39.A, D40.C
- new net N$1421: R186.2, R188.2, R195.2, R196.2, R197.1, U15.NEG_B
- new net N$143: C129.1, U$16.RBOOS2
- new net N$1433: D26.A, U29.OUT_B
- new net N$144: R147.2, U41.OUT_A
- new net N$1444: D59.A, U41.OUT_B
- new net N$145: C130.1, U$16.RIN
- new net N$146: C131.1, U$16.RCUT2
- new net N$147: C132.1, U$16.LCUT1
- new net N$148: C133.1, U$16.LIN
- new net N$149: C134.1, U$16.LBOOS1
- new net N$150: C135.1, U$16.LOUT
- new net N$151: D44.C, R70.2, U21.POS_B
- new net N$152: D38.A, D39.C
- new net N$153: C105.2, U$16.LLMC2
- new net N$1533: D33.C, R92.2, U29.POS_B
- new net N$154: C106.2, C120.2, U$16.LLMC3
- new net N$1544: D66.C, R153.2, U41.POS_B
- new net N$155: C107.2, U$16.LHMC2
- new net N$156: C108.2, C121.2, U$16.LHMC3
- new net N$157: C109.2, U$16.LHC2
- new net N$158: C110.2, C122.2, U$16.LHC3
- new net N$159: C111.2, C124.2, U$16.RHC3
- new net N$160: C112.2, U$16.RHC2
- new net N$161: R70.1, R71.2, U23.NEG_A
- new net N$162: C14.1, R78.2
- new net N$163: C113.2, C125.2, U$16.RHMC3
- new net N$1633: R92.1, R93.2, U31.NEG_A
- new net N$164: C114.2, U$16.RHMC2
- new net N$1644: R153.1, R154.2, U43.NEG_A
- new net N$165: C115.2, C126.2, U$16.RLMC3
- new net N$166: C116.2, U$16.RLMC2
- new net N$167: C117.2, C127.2, U$16.RLC3
- new net N$168: C118.2, U$16.RLC2
- new net N$169: C129.2, U$16.RBOOS1
- new net N$170: C131.2, U$16.RCUT1
- new net N$171: C132.2, U$16.LCUT2
- new net N$172: C134.2, U$16.LBOOS2
- new net N$173: C104.1, U$16.LLC4
- new net N$175: C141.2, R137.2, R138.2, R139.2
- new net N$18: R26.1, U12.OUT_A, U12.POS_B
- new net N$1833: R94.1, U32.OUT_A, U32.POS_B
- new net N$1844: R155.1, U44.OUT_A, U44.POS_B
- new net N$19: R26.2, R27.2, U12.NEG_A
- new net N$1933: R94.2, R95.2, U32.NEG_A
- new net N$1944: R155.2, R156.2, U44.NEG_A
- new net N$2012: C53.2, R54.2, R55.2, R56.2
- new net N$21: C5.1, D13.A, D14.C, D21.A, R12.1, R36.2
- new net N$2111: C13.1, D35.A, D36.C, D43.A, R64.1, R76.2
- new net N$21111: C17.1, U$13.LLC1
- new net N$2133: C12.1, D24.A, D25.C, D32.A, R86.1, R98.2
- new net N$2144: C61.1, D57.A, D58.C, D65.A, R147.1, R159.2
- new net N$22: C19.1, U$13.LLMC1
- new net N$223: C143.1, R200.2
- new net N$225: R186.1, R189.2, R193.2
- new net N$226: R185.2, R192.1, R196.1
- new net N$227: R187.2, R191.1, R195.1
- new net N$228: R188.1, R190.1, R194.2
- new net N$23: C20.1, U$13.LLMC4
- new net N$233: D27.C, R99.1, U31.OUT_B
- new net N$244: D60.C, R160.1, U43.OUT_B
- new net N$246: D62.A, D63.C, R154.1, R163.1, U44.POS_A
- new net N$26: D18.A, D19.C, R23.1, R40.1, U12.POS_A
- new net N$261: D40.A, D41.C, R71.1, R80.1, U24.POS_A
- new net N$2611: C21.1, U$13.LHMC1
- new net N$2633: D29.A, D30.C, R119.1, R93.1, U32.POS_A
- new net N$27: R40.2, U10.OUT_B, U10.POS_B
- new net N$271: R80.2, U22.OUT_B, U22.POS_B
- new net N$2711: C22.1, U$13.LHMC4
- new net N$2733: R119.2, U30.OUT_B, U30.POS_B
- new net N$2744: R163.2, U42.OUT_B, U42.POS_B
- new net N$28: C23.1, U$13.LHC1
- new net N$29: C24.1, U$13.LHC4
- new net N$31: C13.2, D34.C, D36.A, R61.2, U21.NEG_A
- new net N$312: R81.2, U4.POS_B
- new net N$33: C25.1, U$13.RHC4
- new net N$331: R164.2, U13.POS_B
- new net N$333: C12.2, D23.C, D25.A, R52.2, U29.NEG_A
- new net N$34: C26.1, U$13.RHC1
- new net N$344: C61.2, D56.C, D58.A, R144.2, U41.NEG_A
- new net N$35: C27.1, U$13.RHMC4
- new net N$36: C28.1, U$13.RHMC1
- new net N$37: C29.1, U$13.RLMC4
- new net N$38: C30.1, U$13.RLMC1
- new net N$39: C31.1, U$13.RLC4
- new net N$40: C32.1, U$13.RLC1
- new net N$41: D44.A, U23.OUT_A
- new net N$411: C17.2, U$13.LLC2
- new net N$413: R114.2, R116.1, U6.OUT_B
- new net N$414: R50.2, U3.POS_B
- new net N$42: C18.2, C33.2, U$13.LLC3
- new net N$421: R197.2, R199.1, U15.OUT_B
- new net N$43: C33.1, U$13.LLC5
- new net N$433: D33.A, U31.OUT_A
- new net N$44: C34.1, U$13.LLMC5
- new net N$444: D66.A, U43.OUT_A
- new net N$45: C35.1, U$13.LHMC5
- new net N$46: C36.1, U$13.LHC5
- new net N$47: C37.1, U$13.V_REF
- new net N$48: C38.1, U$13.RHC5
- new net N$49: C39.1, U$13.RHMC5
- new net N$500: R28.1, U2.POS_A
- new net N$512: R57.1, U4.POS_A
- new net N$513: R115.1, R116.2, U6.NEG_A
- new net N$514: R46.1, U3.POS_A
- new net N$52: C42.1, U$13.ROUT
- new net N$521: R198.1, R199.2, U15.NEG_A
- new net N$53: C43.1, U$13.RBOOS2
- new net N$531: R140.1, U13.POS_A
- new net N$54: C44.1, U$13.RIN
- new net N$55: C45.1, U$13.RCUT2
- new net N$56: C46.1, U$13.LCUT1
- new net N$57: C47.1, U$13.LIN
- new net N$58: C48.1, U$13.LBOOS1
- new net N$59: C49.1, U$13.LOUT
- new net N$60: C19.2, U$13.LLMC2
- new net N$600: R31.1, U2.NEG_A
- new net N$61: R63.2, R65.2, U22.POS_A
- new net N$611: C20.2, C34.2, U$13.LLMC3
- new net N$612: R59.1, U4.NEG_A
- new net N$614: R48.1, U3.NEG_A
- new net N$62: C21.2, U$13.LHMC2
- new net N$63: C22.2, C35.2, U$13.LHMC3
- new net N$631: R142.1, U13.NEG_A
- new net N$633: R85.2, R87.2, U30.POS_A
- new net N$64: C23.2, U$13.LHC2
- new net N$644: R146.2, R148.2, U42.POS_A
- new net N$65: C24.2, C36.2, U$13.LHC3
- new net N$66: C25.2, C38.2, U$13.RHC3
- new net N$67: C26.2, U$13.RHC2
- new net N$68: C27.2, C39.2, U$13.RHMC3
- new net N$69: C28.2, U$13.RHMC2
- new net N$70: C29.2, C40.2, U$13.RLMC3
- new net N$700: R30.2, R32.2, U2.NEG_B
- new net N$71: R66.2, R67.1, U22.NEG_A
- new net N$711: C30.2, U$13.RLMC2
- new net N$712: R58.2, R60.2, U4.NEG_B
- new net N$714: R47.2, R49.2, U3.NEG_B
- new net N$72: C31.2, C41.2, U$13.RLC3
- new net N$73: C32.2, U$13.RLC2
- new net N$731: R141.2, R143.2, U13.NEG_B
- new net N$733: R88.2, R89.1, U30.NEG_A
- new net N$74: C43.2, U$13.RBOOS1
- new net N$744: R149.2, R150.1, U42.NEG_A
- new net N$75: C45.2, U$13.RCUT1
- new net N$76: C46.2, U$13.LCUT2
- new net N$77: C48.2, U$13.LBOOS2
- new net N$78: C18.1, U$13.LLC4
- new net N$80: C55.1, R117.2
- new net N$800: C4.1, R30.1, U2.OUT_B
- new net N$81: R76.1, R77.2, U23.POS_B
- new net N$812: C51.1, R58.1, U4.OUT_B
- new net N$814: C11.1, R47.1, U3.OUT_B
- new net N$82: R103.1, R106.2, R110.2
- new net N$83: R102.2, R109.1, R113.1
- new net N$831: C139.1, R141.1, U13.OUT_B
- new net N$833: R98.1, R99.2, U31.POS_B
- new net N$84: R104.2, R108.1, R112.1
- new net N$844: R159.1, R160.2, U43.POS_B
- new net N$85: R105.1, R107.1, R111.2
- new net N$86: D23.A, D24.C
- new net N$87: D28.A, D29.C
- new net N$88: C67.1, IC2.VREF
- new net N$89: C68.1, C69.1, IC2.LDO
- new net N$90: D27.A, D28.C
- new net N$91: C50.1, R100.2
- new net N$912: C52.1, R82.2, U4.OUT_A
- new net N$914: C57.1, R51.2, U3.OUT_A
- new net N$92: R125.2, R126.2, U28.POS_A
- new net N$93: R123.2, R124.2, U28.POS_B
- new net N$931: C140.1, R165.2, U13.OUT_A
- new net N$94: D31.A, D32.C
- new net N$95: D30.A, D31.C
- new net N$99: C103.1, U$16.LLC1
- new net P0A1: R56.1, R57.2, U$7.P0A
- new net P0A31: R139.1, R140.2, U$18.P0A
- new net P0A4: R45.1, R46.2, U$3.P0A
- new net P0A_0: R19.2, U$5.P0A
- new net P0A_01: R68.2, U$11.P0A
- new net P0A_03: R90.2, U$14.P0A
- new net P0A_04: R151.2, U$20.P0A
- new net P0A_1: R39.1, U$6.P0A
- new net P0A_11: R79.1, U$12.P0A
- new net P0A_13: R101.1, U$15.P0A
- new net P0A_14: R162.1, U$21.P0A
- new net P0B1: R55.1, R81.1, U$7.P0B
- new net P0B31: R138.1, R164.1, U$18.P0B
- new net P0B4: R44.1, R50.1, U$3.P0B
- new net P0B_1: R38.1, U$6.P0B, U10.NEG_B
- new net P0B_11: R78.1, U$12.P0B, U22.NEG_B
- new net P0B_13: R100.1, U$15.P0B, U30.NEG_B
- new net P0B_14: R161.1, U$21.P0B, U42.NEG_B
- new net P0W1: R59.2, R60.1, R82.1, U$7.P0W
- new net P0W31: R142.2, R143.1, R165.1, U$18.P0W
- new net P0W4: R48.2, R49.1, R51.1, U$3.P0W
- new net P0W_0: R14.1, U$5.P0W
- new net P0W_01: R66.1, U$11.P0W
- new net P0W_03: R88.1, U$14.P0W
- new net P0W_04: R149.1, U$20.P0W
- new net PA0: R17.2, U$4.PA0, U10.OUT_A
- new net PA01: R67.2, U$10.PA0, U22.OUT_A
- new net PA03: R89.2, U$9.PA0, U30.OUT_A
- new net PA04: R150.2, U$19.PA0, U42.OUT_A
- new net PA1: R29.2, U$4.PA1, U12.NEG_B
- new net PA11: R74.2, U$10.PA1, U24.NEG_B
- new net PA13: R96.2, U$9.PA1, U32.NEG_B
- new net PA14: R157.2, U$19.PA1, U44.NEG_B
- new net PB0: R2.2, U$4.PB0, U9.POS_A
- new net PB01: R62.2, U$10.PB0, U21.POS_A
- new net PB03: R53.2, U$9.PB0, U29.POS_A
- new net PB04: R145.2, U$19.PB0, U41.POS_A
- new net PB1: C7.2, U$4.PB1, U12.OUT_B
- new net PB11: C15.2, U$10.PB1, U24.OUT_B
- new net PB13: C54.2, U$9.PB1, U32.OUT_B
- new net PB14: C70.2, U$19.PB1, U44.OUT_B
- new net RS: U$4.~RS
- new net RS1: U$10.~RS
- new net RS3: U$9.~RS
- new net RS4: U$19.~RS
- new net SCL: IC2.MC/SCL, SCL1.P, U16.SCL, U19.SCL, U20.SCL, U26.SCL, U27.SCL, U39.SCL, U40.SCL, U7.SCL, U8.SCL
- new net SCL_0: U26.SC0
- new net SCL_1: U26.SD0
- new net SCL_2: U26.SC2
- new net SCL_3: U26.SD2
- new net SDA: IC2.MOSI/SDA, SDA1.P, U16.SDA, U19.SDA, U20.SDA, U26.SDA, U27.SDA, U39.SDA, U40.SDA, U7.SDA, U8.SDA
- new net SDA_0: U26.SC1
- new net SDA_1: U26.SD1
- new net SDA_2: U26.SC3
- new net SDA_3: U26.SD3
- new net SHDN: U$4.~SHDN
- new net SHDN1: U$10.~SHDN
- new net SHDN3: U$9.~SHDN
- new net SHDN4: U$19.~SHDN
- new net VIN1: IC2.VINL2/VIN1M
- new net VIN2: IC2.VINL1/VIN1P
- new net VIN3: IC2.VINR3/VIN3P
- new net VIN4: IC2.VINR4/VIN3M
- net 3V3A: now also C65.1, C66.1, IC2.AVDD, U28.NEG_A, U28.OUT_A; no longer U1.NEG_A, U1.OUT_A
- net AIN: now also AIN1.P, C6.2; no longer C4.1
- net AIN0: now also C10.1; no longer R13.1
- net AIN1: now also AIN3.P, C14.2; no longer R14.1
- net AIN2: now also R104.1; no longer R7.1
- net AIN3: now also R102.1; no longer R5.1
- net AOUT: now also C7.1, R33.1; no longer C1.2, R21.2
- net AOUTL: now also C9.2, R41.2; no longer C3.2, R31.2
- net AOUTR: now also C4.2, R42.2; no longer C2.2, R32.2
- net CS: now also U$2.!CS; no longer U$1.!CS
- net EIN0: now also C44.2; no longer C86.2
- net EIN1: now also C47.2; no longer C89.2
- net EOUT0: now also C42.2; no longer C84.2
- net EOUT1: now also C49.2; no longer C91.2
- net GND: now also C123.2, C37.2, C63.2, C64.2, C65.2, C66.2, C67.2, C68.2, C69.2, GND2.P, GND6.P, GND7.P, IC2.AGND, IC2.DGND, R118.1, R120.1, R121.1, R123.1, R125.1, R166.1, R167.1, R201.1, R41.1, R42.1, R83.1, R84.1, U$13.TEST, U$13.V_SS, U$16.TEST, U$16.V_SS, U$18.VSS, U$2.VSS, U$3.VSS, U$7.VSS, U13.V-, U15.V-, U2.V-, U28.V-, U3.V-, U4.V-, U6.V-; no longer C79.2, R1.1, R3.1, U$14.TEST, U$14.V_SS, U1.V-
- net N$1: now also D13.C, D6.A, R12.2, U9.OUT_A; no longer R3.2, R4.2, U1.POS_A
- net N$13: now also D34.A, D35.C; no longer R13.2, R6.1, R9.2
- net N$133: now also R86.2, U29.OUT_A; no longer C66.1, U$14.RHC4
- net N$14: now also D15.A, U9.OUT_B; no longer R15.2, R16.2, R17.1, R6.2, R8.2, U2.NEG_B
- net N$15: now also D22.C, R22.2, U9.POS_B; no longer R12.1, R16.1, R5.2
- net N$16: now also R22.1, R23.2, U11.NEG_A; no longer R11.1, R15.1, R7.2
- net N$17: now also D42.A, D43.C; no longer R10.1, R14.2, R8.1
- net N$181: now also R72.1, U24.OUT_A, U24.POS_B; no longer C69.1, U$14.RHMC1
- net N$182: now also D41.A, D42.C; no longer C70.1, U$14.RLMC4
- net N$191: now also R72.2, R73.2, U24.NEG_A; no longer C78.1, U$14.LHC5
- net N$2: now also D16.C, D17.A, D18.C, R37.1, U11.OUT_B; no longer R1.2, R2.2, U1.POS_B
- net N$20: now also C58.2, R43.2, R44.2, R45.2; no longer R18.2, R20.1, U2.OUT_A
- net N$211: now also D38.C, R77.1, U23.OUT_B; no longer C66.2, C80.2, U$14.RHC3
- net N$213: now also R115.2, R117.1, U6.OUT_A; no longer C68.2, C81.2, U$14.RHMC3
- net N$221: now also R198.2, R200.1, U15.OUT_A; no longer C87.2, U$14.RCUT1
- net N$3: now also C5.2, D14.A, D16.A, D17.C, D6.C, R1.2, U9.NEG_A; no longer C59.1, U$14.LLC4
- net N$30: now also R34.2, U2.POS_B; no longer R29.2, U3.POS_B
- net N$4: now also C6.1, D22.A, R38.2, U11.OUT_A; no longer C1.1, R17.2, R19.1, R20.2, U2.OUT_B
- net N$5: now also D20.A, D21.C; no longer R18.1, R19.2, U2.NEG_A
- net N$50: now also C40.1, U$13.RLMC5; no longer C4.2, R22.2, R23.2, R24.2
- net N$51: now also C41.1, U$13.RLC5; no longer R25.1, U3.POS_A
- net N$6: now also D19.A, D20.C, R13.2, R5.2, U10.POS_A; no longer R27.1, U3.NEG_A
- net N$7: now also R14.2, R17.1, U10.NEG_A; no longer R26.2, R28.2, U3.NEG_B
- net N$8: now also R36.1, R37.2, U11.POS_B; no longer C2.1, R26.1, U3.OUT_B
- net N$9: now also C9.1, R35.2, U2.OUT_A; no longer C3.1, R30.2, U3.OUT_A
- net P0A: now also R25.1, R28.2, U$2.P0A; no longer R24.1, R25.2, U$1.P0A
- net P0B: now also R24.1, R34.1, U$2.P0B; no longer R23.1, R29.1, U$1.P0B
- net P0W: now also R31.2, R32.1, R35.1, U$2.P0W; no longer R27.2, R28.1, R30.1, U$1.P0W
- net SCK: now also SCK1.P, U$10.SCK, U$11.SCK, U$12.SCK, U$14.SCK, U$15.SCK, U$18.SCK, U$19.SCK, U$2.SCK, U$20.SCK, U$21.SCK, U$3.SCK, U$4.SCK, U$5.SCK, U$6.SCK, U$7.SCK, U$9.SCK; no longer U$1.SCK
- net SDI/O: now also SDI/O1.P, U$10.SI, U$11.SDI/SDO, U$12.SDI/SDO, U$14.SDI/SDO, U$15.SDI/SDO, U$18.SDI/SDO, U$19.SI, U$2.SDI/SDO, U$20.SDI/SDO, U$21.SDI/SDO, U$3.SDI/SDO, U$4.SI, U$5.SDI/SDO, U$6.SDI/SDO, U$7.SDI/SDO, U$9.SI; no longer U$1.SDI/SDO
- net VDD: now also 9VDD1.P, R124.1, R126.1, R151.1, R19.1, R68.1, R90.1, U$10.VDD, U$11.VDD, U$12.VDD, U$13.V_DD, U$14.VDD, U$15.VDD, U$16.V_DD, U$19.VDD, U$20.VDD, U$21.VDD, U$4.VDD, U$5.VDD, U$6.VDD, U$9.VDD, U10.V+, U11.V+, U12.V+, U13.V+, U15.V+, U16.VDD, U19.VDD, U20.A0, U20.VDD, U21.V+, U22.V+, U23.V+, U24.V+, U27.A0, U27.VDD, U28.V+, U29.V+, U30.V+, U31.V+, U32.V+, U39.VDD, U4.V+, U40.A0, U40.VDD, U41.V+, U42.V+, U43.V+, U44.V+, U6.V+, U7.VDD, U8.A0, U8.VDD, U9.V+; no longer R2.1, R4.1, U$14.V_DD, U1.V+
- net VREF: now also C16.2, C56.2, C71.2, C8.2, R1.1, R101.2, R106.1, R107.2, R108.2, R109.2, R137.1, R144.1, R145.1, R146.1, R152.2, R156.1, R157.1, R162.2, R189.1, R190.2, R191.2, R192.2, R2.1, R20.2, R21.1, R27.1, R29.1, R39.2, R43.1, R5.1, R52.1, R53.1, R54.1, R61.1, R62.1, R63.1, R69.2, R73.1, R74.1, R79.2, R85.1, R91.2, R95.1, R96.1, U$11.P0B, U$14.P0B, U$18.VDD, U$2.VDD, U$20.P0B, U$3.VDD, U$5.P0B, U$7.VDD, U11.NEG_B, U11.POS_A, U15.POS_A, U15.POS_B, U23.NEG_B, U23.POS_A, U28.NEG_B, U28.OUT_B, U31.NEG_B, U31.POS_A, U43.NEG_B, U43.POS_A, U6.POS_A, U6.POS_B; no longer R10.2, R11.2, R12.2, R22.1, R9.1, U$1.VDD, U1.NEG_B, U1.OUT_B, U2.POS_A, U2.POS_B
- net VSS: now also GND1.P, GND3.P, GND4.P, GND8.P, R158.2, R33.2, R75.2, R97.2, U$10.VSS, U$11.VSS, U$12.VSS, U$14.VSS, U$15.VSS, U$19.VSS, U$20.VSS, U$21.VSS, U$4.VSS, U$5.VSS, U$6.VSS, U$9.VSS, U10.V-, U11.V-, U12.V-, U16.A0, U16.EPAD, U16.GND, U19.A0, U19.EPAD, U19.GND, U20.EPAD, U20.GND, U21.V-, U22.V-, U23.V-, U24.V-, U27.EPAD, U27.GND, U29.V-, U30.V-, U31.V-, U32.V-, U39.A0, U39.EPAD, U39.GND, U40.EPAD, U40.GND, U41.V-, U42.V-, U43.V-, U44.V-, U7.A0, U7.EPAD, U7.GND, U8.EPAD, U8.GND, U9.V-; no longer R21.1, R31.1, R32.1, U$1.VSS, U2.V-, U3.V-
Other:
- moved on the sheet: C61, C62, C63, C64, C65, C66, C67, C68, C69, C70, C71, R1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
