File: compressor.sch (EAGLE design)
At the start: 46 parts, among them U1 MAX5419LETA+, U2 MAX5419LETA+, U3 LM4562MAX/NOPB, U4 LM4562MAX/NOPB, U5 LM4562MAX/NOPB, U6 LM4562MAX/NOPB

Commit message: corrections
Parts:
- removed R30: 1M, rcl:R-US_R0402
- C2: value 0.1 -> 0.1u
Connections:
- net AOUT: no longer R30.1
- net VSS: no longer R30.2
Other:
- moved on the sheet: U$1, U$2, U$3, U1, U2, U3, U4, U5, U6

Commit message: updates
Parts:
- removed AIN: (no value), wirepad:SMD5
- removed C3: 1.5u, rcl:C-USC0402
- removed R15: 100k, rcl:R-US_R0402
- removed R4: 10k, rcl:R-US_R0402
- removed U$1: MCP42100-I/P, MCP42100-I_P:MCP42100-I/P
- removed U$2, U$3: MCP4131-503E/SN, MCP4131-503E_SN:MCP4131-503E/SN
- removed U3, U4, U5, U6: LM4562MAX/NOPB, LM4562MAX_NOPB:LM4562MAX/NOPB
- added 100POT1_COMP: MCP42100-I/P, MCP42100-I_P:MCP42100-I/P
- added 10POT1_COMP, 10POT2_COMP: MCP4131-503E/SN, MCP4131-503E_SN:MCP4131-503E/SN
- added IN_COMP: (no value), wirepad:SMD5
- added OPAMP1_COMP, OPAMP2_COMP, OPAMP3_COMP, OPAMP4_COMP: LM4562MAX/NOPB, LM4562MAX_NOPB:LM4562MAX/NOPB
- added R1: 100k, rcl:R-US_R0402
- C2: value 0.1u -> 10u
- renumbered U1 to 200POT2_COMP, U2 to 200POT1_COMP
Connections:
- net SCL renamed SCL_COMP
- net SDA renamed SDA_COMP
- removed net AIN: AIN.P, C2.2
- removed net AOUT: C3.1
- removed net CS0: U$1.~CS
- removed net CS1: U$2.!CS
- removed net CS2: U$3.!CS
- removed net H_0: 200POT1_COMP.H, 200POT2_COMP.H, C4.1, R8.1, U3.NEG_B
- removed net L_0: 200POT2_COMP.L, R15.1
- removed net L_1: 200POT1_COMP.L, D4.C
- removed net N$1: R7.2, U3.OUT_A
- removed net N$14: D4.A, U3.OUT_B
- removed net N$15: D5.C, R16.2, U3.POS_B
- removed net N$16: R16.1, R18.2, U5.NEG_A
- removed net N$18: R21.1, U6.OUT_A, U6.POS_B
- removed net N$19: R21.2, R24.2, U6.NEG_A
- removed net N$2: D7.C, R31.1, U5.OUT_B
- removed net N$26: D10.C, D9.A, R18.1, R35.1, U6.POS_A
- removed net N$27: R35.2, U4.OUT_B, U4.POS_B
- removed net N$3: C1.2, D1.C, D3.A, R3.2, U3.NEG_A
- removed net N$4: D5.A, U5.OUT_A
- removed net N$6: R6.2, R8.2, U4.POS_A
- removed net N$7: R10.1, R9.2, U4.NEG_A
- removed net N$8: R28.1, R31.2, U5.POS_B
- removed net P0A_0: R11.2, U$2.P0A
- removed net P0A_1: R34.1, U$3.P0A
- removed net P0B_1: R32.1, U$3.P0B, U4.NEG_B
- removed net P0W_0: R9.1, U$2.P0W
- removed net PA0: R10.2, U$1.PA0, U4.OUT_A
- removed net PA1: R25.2, U$1.PA1, U6.NEG_B
- removed net PB0: R4.2, U$1.PB0, U3.POS_A
- removed net PB1: C3.2, U$1.PB1, U6.OUT_B
- removed net RS: U$1.~RS
- removed net SHDN: U$1.~SHDN
- removed net VSS: 200POT1_COMP.EPAD, 200POT1_COMP.GND, 200POT2_COMP.A0, 200POT2_COMP.EPAD, 200POT2_COMP.GND, GND.P, U$1.VSS, U$2.VSS, U$3.VSS, U3.V-, U4.V-, U5.V-, U6.V-
- new net CS0_COMP: 100POT1_COMP.~CS
- new net CS1_COMP: 10POT1_COMP.!CS
- new net CS2_COMP: 10POT2_COMP.!CS
- new net GND: 100POT1_COMP.VSS, 10POT1_COMP.VSS, 10POT2_COMP.VSS, 200POT1_COMP.EPAD, 200POT1_COMP.GND, 200POT2_COMP.A0, 200POT2_COMP.EPAD, 200POT2_COMP.GND, GND.P, OPAMP1_COMP.V-, OPAMP2_COMP.V-, OPAMP3_COMP.V-, OPAMP4_COMP.V-
- new net H1_COMP: 200POT1_COMP.H, 200POT2_COMP.H, C4.1, OPAMP1_COMP.NEG_B, R8.1
- new net IN_COMP: C2.2, IN_COMP.P
- new net L1_COMP: 200POT1_COMP.L, 200POT1_COMP.W, D4.C
- new net L2_COMP: 200POT2_COMP.L, 200POT2_COMP.W, R1.2
- new net NEG_A1_COMP: C1.2, D1.C, D3.A, OPAMP1_COMP.NEG_A, R3.2
- new net NEG_A2_COMP: OPAMP2_COMP.NEG_A, R10.1, R9.2
- new net NEG_A3_COMP: OPAMP3_COMP.NEG_A, R16.1, R18.2
- new net NEG_A4_COMP: OPAMP4_COMP.NEG_A, R21.2, R24.2
- new net NEG_B2_COMP: OPAMP2_COMP.NEG_B, OPAMP2_COMP.OUT_B, R35.2
- new net NEG_B3_COMP: OPAMP3_COMP.NEG_B, R28.1, R31.2
- new net NEG_B4_COMP: 100POT1_COMP.PB1, OPAMP4_COMP.NEG_B, R25.2
- new net OUT_A1_COMP: OPAMP1_COMP.OUT_A, R7.2
- new net OUT_A2_COMP: 100POT1_COMP.PB0, OPAMP2_COMP.OUT_A, R10.2
- new net OUT_A3_COMP: D5.A, OPAMP3_COMP.OUT_A
- new net OUT_A4_COMP: OPAMP4_COMP.OUT_A, OPAMP4_COMP.POS_B, R18.1, R21.1
- new net OUT_B1_COMP: D4.A, OPAMP1_COMP.OUT_B
- new net OUT_B3_COMP: D7.C, OPAMP3_COMP.OUT_B, R31.1
- new net OUT_COMP: 100POT1_COMP.PA1, 100POT1_COMP.PW1, OPAMP4_COMP.OUT_B
- new net P0A1_COMP: 10POT1_COMP.P0A, R11.2
- new net P0A2_COMP: 10POT2_COMP.P0A, R34.1
- new net P0W1_COMP: 10POT1_COMP.P0W, R9.1
- new net POS_A1_COMP: 100POT1_COMP.PW0, OPAMP1_COMP.POS_A
- new net POS_A2_COMP: OPAMP2_COMP.POS_A, R6.2, R8.2
- new net POS_A4_COMP: D10.C, D9.A, OPAMP4_COMP.POS_A, R35.1
- new net POS_B1_COMP: D5.C, OPAMP1_COMP.POS_B, R16.2
- new net POS_B2_COMP: 10POT2_COMP.P0B, 10POT2_COMP.P0W, OPAMP2_COMP.POS_B, R32.1
- net SCK: now also 100POT1_COMP.SCK, 10POT1_COMP.SCK, 10POT2_COMP.SCK; no longer U$1.SCK, U$2.SCK, U$3.SCK
- net SDI/O: now also 100POT1_COMP.SI, 10POT1_COMP.SDI/SDO, 10POT2_COMP.SDI/SDO; no longer U$1.SI, U$2.SDI/SDO, U$3.SDI/SDO
- net VDD: now also OPAMP1_COMP.V+, OPAMP2_COMP.V+, OPAMP3_COMP.V+, OPAMP4_COMP.V+; no longer 200POT1_COMP.A0, 200POT1_COMP.VDD, 200POT2_COMP.VDD, U$1.VDD, U$2.VDD, U$3.VDD, U3.V+, U4.V+, U5.V+, U6.V+
- net VREF: now also 100POT1_COMP.PA0, 100POT1_COMP.VDD, 100POT1_COMP.~RS, 100POT1_COMP.~SHDN, 10POT1_COMP.P0B, 10POT1_COMP.VDD, 10POT2_COMP.VDD, 200POT1_COMP.A0, 200POT1_COMP.VDD, 200POT2_COMP.VDD, OPAMP3_COMP.POS_A, OPAMP3_COMP.POS_B, R1.1; no longer R15.2, R4.1, U$2.P0B, U5.NEG_B, U5.POS_A
Other:
- moved on the sheet: C4, D4, D5, GND, R16, R18, R31, R8
