File: mixer.sch (EAGLE design)
At the start: 20 parts, among them U1 LM4562MAX/NOPB

Commit message: updates
Parts:
- removed AOUT, GND: (no value), wirepad:SMD5
- removed U1: LM4562MAX/NOPB, LM4562MAX_NOPB:LM4562MAX/NOPB
- added C2: 0.1u, rcl:C-USC0402
- added GNDL, GNDR, OUTL_MIX, OUTR_MIX: (no value), wirepad:SMD5
- added OPAMP1_MIX: LM4562MAX/NOPB, LM4562MAX_NOPB:LM4562MAX/NOPB
- added R17, R19, R26, R27: 10k, rcl:R-US_R0402
- added R18, R20, R21, R22, R23, R24, R25, R28: 5k, rcl:R-US_R0402
- added R29: 50k, rcl:R-US_R0402
- added R30: 1k, rcl:R-US_R0402
- R11, R12, R2, R4: value 20k -> 10k
- R13, R14: value 20k -> 5k
- R15: value 20k -> 50k
Connections:
- net AIN0 renamed IN1L_MIX
- net AIN1 renamed IN2L_MIX
- net AIN2 renamed IN3L_MIX
- net AIN3 renamed IN4L_MIX
- removed net AOUT: AOUT.P, C1.2
- new net IN1R_MIX: R24.1
- new net IN2R_MIX: R25.1
- new net IN3R_MIX: R18.1
- new net IN4R_MIX: R14.1
- new net N$3: R17.1, R20.2, R24.2
- new net N$6: R18.2, R22.1, R26.1
- new net N$7: R19.1, R21.1, R25.2
- new net NEG_A_MIX: OPAMP1_MIX.NEG_A, R13.2, R15.1
- new net NEG_B_MIX: OPAMP1_MIX.NEG_B, R28.2, R29.1
- new net OUTL_MIX: C1.2, OUTL_MIX.P
- new net OUTR_MIX: C2.2, OUTR_MIX.P
- new net OUT_A_MIX: OPAMP1_MIX.OUT_A, R15.2, R16.1
- new net OUT_B_MIX: OPAMP1_MIX.OUT_B, R29.2, R30.1
- net GND: now also GNDL.P, GNDR.P, OPAMP1_MIX.V-; no longer GND.P, U1.V-
- net N$14: no longer U1.NEG_B
- net N$2: now also C2.1, R30.2; no longer R14.2, R16.1, U1.OUT_A
- net N$4: now also R17.2, R19.2, R26.2, R27.2, R28.1; no longer R13.2, R15.1, U1.OUT_B
- net N$5: now also R14.2, R23.1, R27.1; no longer R14.1, R15.2, U1.NEG_A
- net VDD: now also OPAMP1_MIX.V+; no longer U1.V+
- net VREF: now also OPAMP1_MIX.POS_A, OPAMP1_MIX.POS_B, R20.1, R21.2, R22.2, R23.2; no longer U1.POS_A, U1.POS_B
Other:
- moved on the sheet: C1, R1, R10, R11, R12, R13, R14, R15, R16, R2, R3, R4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
