File: nopi.sch (EAGLE design)
At the start: 5 parts, among them U1 RASPBERRY_PI_4B_4GB, U6 TMUX1204DGSR, U7 TMUX1204DGSR, U8 TMUX1204DGSR, U9 TCA9546ADR

Commit message: corrections
Parts:
- removed U1: RASPBERRY_PI_4B_4GB, RASPBERRY_PI_4B_4GB:RASPBERRY_PI_4B_4GB
- added 3V3_D, CS0, CS1, CS2, GND, MUX0, MUX1, SCK, SCL, SDA, SDI/O: (no value), wirepad:SMD2
Connections:
- removed net BCK_ADC: U1.GPIO27/GPIO_GEN2
- removed net CLK_ADC: U1.GPIO4/GPIO_GCKL
- removed net DOUT_ADC: U1.GPIO17/GPIO_GEN0
- removed net EQ0_CE: U1.GPIO23/GPIO_GEN4
- removed net EQ0_CL: U1.GPIO25/GPIO_GEN6
- removed net EQ0_DI: U1.GPIO24/GPIO_GEN5
- removed net EQ1_CE: U1.GPIO20
- removed net EQ1_CL: U1.GPIO26
- removed net EQ1_DI: U1.GPIO21
- removed net LRCK_ADC: U1.GPIO18/GPIO_GEN1
- net +3V3: now also 3V3_D.P; no longer U1.3V3
- net CS0: now also CS0.P; no longer U1.GPIO12
- net CS1: now also CS1.P; no longer U1.GPIO13
- net CS2: now also CS2.P; no longer U1.GPIO16
- net DGND: now also GND.P; no longer U1.GND, U1.SHIELD
- net MUX0: now also MUX0.P; no longer U1.GPIO5
- net MUX1: now also MUX1.P; no longer U1.GPIO6
- net SCK: now also SCK.P; no longer U1.GPIO11/SPI_SCLK
- net SCL: now also SCL.P; no longer U1.GPIO3/SCL1
- net SDA: now also SDA.P; no longer U1.GPIO2/SDA1
- net SDI/O: now also SDI/O.P; no longer U1.GPIO10/SPI_MOSI

Commit message: updates
Parts:
- added CS: (no value), wirepad:SMD2
- added U1: TMUX1204DGSR, TMUX1204DGSR:TMUX1204DGSR
Connections:
- net CS0_0 renamed CS0_COMP1
- net CS0_1 renamed CS0_COMP2
- net CS0_2 renamed CS0_COMP3
- net CS0_3 renamed CS0_COMP4
- net CS1_0 renamed CS1_COMP1
- net CS1_1 renamed CS1_COMP2
- net CS1_2 renamed CS1_COMP3
- net CS1_3 renamed CS1_COMP4
- net CS2_0 renamed CS2_COMP1
- net CS2_1 renamed CS2_COMP2
- net CS2_2 renamed CS2_COMP3
- net CS2_3 renamed CS2_COMP4
- new net CS: CS.P, U1.D
- new net CS0_PAN4: U1.S4
- new net CS_PAN1: U1.S1
- new net CS_PAN2: U1.S2
- new net CS_PAN3: U1.S3
- net +3V3: now also U1.EN, U1.VDD
- net DGND: now also U1.GND
- net MUX0: now also U1.A0
- net MUX1: now also U1.A1
Other:
- moved on the sheet: U7
