File: panner.brd (EAGLE design)
At the start: 26.6 x 31.4 mm, 16 parts, among them U1 LM4562MAX/NOPB

Commit message: corrections
Parts:
- removed C1, C2, C3: 0.1u, rcl:C0402
- removed R10, R11: 1.5M, rcl:R0402
- moved R6 0.46 mm to (17.8, 9.14)
Connections:
- removed net N$2: C3.2, R1.2, R2.2, R3.2
- removed net N$8: C1.1, R5.1, U1.7
- removed net N$9: C2.1, R9.2, U1.1
- removed net P0W: R6.2, R7.1, R9.1, U$1.6
- net AIN: now also R1.2, R2.2, R3.2; no longer C3.1
- net AOUTL: now also R9.2, U1.1; no longer C2.2, R10.2
- net AOUTR: now also R5.1, U1.7; no longer C1.2, R11.2
- net GND: no longer R10.1, R11.1
- net N$6: now also R9.1
- net VREF: now also R6.2, R7.1, U$1.6
Routing:
- net VREF: track 7.32 -> 31.7 mm, vias 1 -> 2
- net N$9: track 12.7 -> 0.00 mm
- net P0W: track 12.4 -> 0.00 mm
- net AOUTL: track 8.00 -> 15.8 mm
- net N$2: track 7.66 -> 0.00 mm
- net N$8: track 7.56 -> 0.00 mm
- net GND: track 15.3 -> 8.43 mm, vias 2 -> 1
- net AIN: track 1.53 -> 7.22 mm
- net AOUTR: track 7.89 -> 10.7 mm
- net N$6: track 2.49 -> 4.74 mm
- net SDI/O: track 3.04 -> 1.77 mm, vias 0 -> 1
- net SCK: vias 0 -> 1
- net CS: vias 0 -> 1
Other:
- board outline removed

Commit message: updates
Parts:
- removed R6, R7: 6k, rcl:R0402
- added C1: 10uF, rcl:C0402
- added D1: 1N4148W-TPSOD123-L, 1N4148W-TP:SOD123-L
- R1: value 10k -> 1M
- R2, R3: value 10k -> 5k
- R4, R8: value 4k -> 5k
- R5, R9: value 20k -> 10k
- moved R8 2.57 mm to (17.8, 11.2)
- renumbered U$1 to 10KPOT1_PAN, U1 to OPAMP1_PAN
Connections:
- net AOUTL renamed OUTL_PAN
- net AOUTR renamed OUTR_PAN
- net CS renamed CS_PAN
- net P0A renamed P0A_PAN
- net P0B renamed P0B_PAN
- removed net AIN: R1.2, R2.2, R3.2
- removed net N$3: OPAMP1_PAN.5, R8.2
- removed net N$5: OPAMP1_PAN.3, R4.1
- removed net N$6: OPAMP1_PAN.2, R6.1, R9.1
- removed net N$7: OPAMP1_PAN.6, R5.2, R7.2
- new net IN_PAN: C1.1
- new net N$1: C1.2, R1.2, R2.2, R3.2
- new net NEG_A_PAN: OPAMP1_PAN.2, R4.1, R9.1
- new net NEG_B_PAN: OPAMP1_PAN.6, R5.2, R8.2
- new net P0W_PAN: 10KPOT1_PAN.6, D1.1
- net VREF: now also D1.2, OPAMP1_PAN.3, OPAMP1_PAN.5; no longer 10KPOT1_PAN.6, R6.2, R7.1
Routing:
- net N$3: track 29.6 -> 0.00 mm
- net NEG_B_PAN: track 0.00 -> 22.2 mm
- net N$7: track 17.6 -> 0.00 mm
- net NEG_A_PAN: track 0.00 -> 9.22 mm
- net AIN: track 7.22 -> 0.00 mm
- net P0B_PAN: track 13.8 -> 19.6 mm
- net N$6: track 4.74 -> 0.00 mm
- net N$5: track 4.68 -> 0.00 mm
- net N$1: track 0.00 -> 4.60 mm
- net VREF: track 31.7 -> 35.0 mm, vias 2 -> 4
- net IN_PAN: track 0.00 -> 3.16 mm
- net P0W_PAN: track 0.00 -> 2.87 mm
- net OUTR_PAN: track 10.7 -> 13.3 mm
- net OUTL_PAN: track 15.8 -> 17.6 mm
