File: adc.sch (EAGLE design)
At the start: 83 parts, among them IC1 PCM1865DBT, U1 RASPBERRY_PI_4B_4GB, U6 TMUX1204DGSR, U7 TMUX1204DGSR, U8 TMUX1204DGSR, U9 TCA9546ADR

Commit message: update, split out into schematics for each component
Parts:
- removed C10, C11, C12, C13, C14, C15, C16, C17, C18, C19, C20, C21, C22, C23, C24, C58, C59, C60, C61, C62, C63, C64, C65, C66, C67, C68, C69, C70, C71, C72, C73, C74, C8, C9: 0.047uF, rcl:C-US025-024X044
- removed C26, C27, C28, C29, C30, C31, C32, C33, C34, C35, C36, C37, C38, C39, C40, C41, C42, C75, C76, C77, C78, C79, C80, C81, C82, C83, C84, C85, C86, C87, C88, C89, C90, C91: 10uF, rcl:C-US025-024X044
- removed U$1, U$14: LC75281E, LC75281E:LC75281E
- removed U1: RASPBERRY_PI_4B_4GB, RASPBERRY_PI_4B_4GB:RASPBERRY_PI_4B_4GB
- removed U6, U7, U8: TMUX1204DGSR, TMUX1204DGSR:TMUX1204DGSR
- removed U9: TCA9546ADR, TCA9546ADR:TCA9546ADR
Connections:
- removed net +3V3: C1.1, C2.1, C3.1, C4.1, IC1.AVDD, IC1.DVDD, IC1.IOVDD, U1.3V3, U6.EN, U6.VDD, U7.EN, U7.VDD, U8.EN, U8.VDD, U9.VCC
- removed net +5V: U1.5V
- removed net +8V: U$1.V_DD, U$14.V_DD
- removed net AGND: C3.2, C30.2, C4.2, C5.2, C6.2, C7.2, C79.2, IC1.AGND, IC1.DGND, U$1.TEST, U$1.V_SS, U$14.TEST, U$14.V_SS
- removed net CS0_0: U6.S1
- removed net CS0_1: U6.S2
- removed net CS0_2: U1.GPIO12, U6.D, U6.S3
- removed net CS0_3: U6.S4
- removed net CS1_0: U8.S1
- removed net CS1_1: U8.S2
- removed net CS1_2: U1.GPIO13, U8.D, U8.S3
- removed net CS1_3: U8.S4
- removed net CS2: U1.GPIO16, U7.D
- removed net CS2_0: U7.S1
- removed net CS2_1: U7.S2
- removed net CS2_2: U7.S3
- removed net CS2_3: U7.S4
- removed net DGND: C1.2, C2.2, U1.GND, U1.SHIELD, U6.GND, U7.GND, U8.GND, U9.A0, U9.A1, U9.A2, U9.GND, U9.RESET
- removed net EOUT_0: C35.2, IC1.VINL2/VIN1M
- removed net EOUT_1: C42.2, IC1.VINL1/VIN1P
- removed net EOUT_2: C84.2, IC1.VINR3/VIN3P
- removed net EOUT_3: C91.2, IC1.VINR4/VIN3M
- removed net EQ0_CE: U$1.CE, U1.GPIO23/GPIO_GEN4
- removed net EQ0_CL: U$1.CL, U1.GPIO25/GPIO_GEN6
- removed net EQ0_DI: U$1.DI, U1.GPIO24/GPIO_GEN5
- removed net EQ1_CE: U$14.CE, U1.GPIO20
- removed net EQ1_CL: U$14.CL, U1.GPIO26
- removed net EQ1_DI: U$14.DI, U1.GPIO21
- removed net MUX0: U1.GPIO5, U6.A0, U7.A0, U8.A0
- removed net MUX1: U1.GPIO6, U6.A1, U7.A1, U8.A1
- removed net N$12: C24.1, C9.1, U$1.LLC4
- removed net N$123: C58.1, U$14.LLC1
- removed net N$124: C59.1, C74.1, U$14.LLC4
- removed net N$125: C60.1, U$14.LLMC1
- removed net N$126: C61.1, U$14.LLMC4
- removed net N$127: C62.1, U$14.LHMC1
- removed net N$128: C63.1, U$14.LHMC4
- removed net N$129: C64.1, U$14.LHC1
- removed net N$13: C10.1, U$1.LLMC1
- removed net N$130: C65.1, U$14.LHC4
- removed net N$133: C66.1, U$14.RHC4
- removed net N$134: C67.1, U$14.RHC1
- removed net N$14: C11.1, U$1.LLMC4
- removed net N$15: C12.1, U$1.LHMC1
- removed net N$16: C13.1, U$1.LHMC4
- removed net N$17: C14.1, U$1.LHC1
- removed net N$18: C15.1, U$1.LHC4
- removed net N$180: C68.1, U$14.RHMC4
- removed net N$181: C69.1, U$14.RHMC1
- removed net N$182: C70.1, U$14.RLMC4
- removed net N$183: C71.1, U$14.RLMC1
- removed net N$184: C72.1, U$14.RLC4
- removed net N$185: C73.1, U$14.RLC1
- removed net N$186: C58.2, U$14.LLC2
- removed net N$187: C59.2, C74.2, C75.2, U$14.LLC3
- removed net N$188: C75.1, U$14.LLC5
- removed net N$189: C76.1, U$14.LLMC5
- removed net N$19: C16.1, U$1.RHC4
- removed net N$190: C77.1, U$14.LHMC5
- removed net N$191: C78.1, U$14.LHC5
- removed net N$192: C79.1, U$14.V_REF
- removed net N$193: C80.1, U$14.RHC5
- removed net N$194: C81.1, U$14.RHMC5
- removed net N$195: C82.1, U$14.RLMC5
- removed net N$196: C83.1, U$14.RLC5
- removed net N$197: C84.1, U$14.ROUT
- removed net N$198: C85.1, U$14.RBOOS2
- removed net N$199: C86.1, U$14.RIN
- removed net N$20: C17.1, U$1.RHC1
- removed net N$200: C87.1, U$14.RCUT2
- removed net N$201: C88.1, U$14.LCUT1
- removed net N$202: C89.1, U$14.LIN
- removed net N$203: C90.1, U$14.LBOOS1
- removed net N$204: C91.1, U$14.LOUT
- removed net N$205: C60.2, U$14.LLMC2
- removed net N$206: C61.2, C76.2, U$14.LLMC3
- removed net N$207: C62.2, U$14.LHMC2
- removed net N$208: C63.2, C77.2, U$14.LHMC3
- removed net N$209: C64.2, U$14.LHC2
- removed net N$21: C18.1, U$1.RHMC4
- removed net N$210: C65.2, C78.2, U$14.LHC3
- removed net N$211: C66.2, C80.2, U$14.RHC3
- removed net N$212: C67.2, U$14.RHC2
- removed net N$213: C68.2, C81.2, U$14.RHMC3
- removed net N$214: C69.2, U$14.RHMC2
- removed net N$215: C70.2, C82.2, U$14.RLMC3
- removed net N$216: C71.2, U$14.RLMC2
- removed net N$217: C72.2, C83.2, U$14.RLC3
- removed net N$218: C73.2, U$14.RLC2
- removed net N$219: C85.2, U$14.RBOOS1
- removed net N$22: C19.1, U$1.RHMC1
- removed net N$220: C86.2
- removed net N$221: C87.2, U$14.RCUT1
- removed net N$222: C88.2, U$14.LCUT2
- removed net N$223: C89.2
- removed net N$224: C90.2, U$14.LBOOS2
- removed net N$23: C20.1, U$1.RLMC4
- removed net N$24: C21.1, U$1.RLMC1
- removed net N$25: C22.1, U$1.RLC4
- removed net N$26: C23.1, U$1.RLC1
- removed net N$27: C8.2, U$1.LLC2
- removed net N$28: C24.2, C26.2, C9.2, U$1.LLC3
- removed net N$29: C26.1, U$1.LLC5
- removed net N$30: C27.1, U$1.LLMC5
- removed net N$31: C28.1, U$1.LHMC5
- removed net N$32: C29.1, U$1.LHC5
- removed net N$33: C30.1, U$1.V_REF
- removed net N$34: C31.1, U$1.RHC5
- removed net N$35: C32.1, U$1.RHMC5
- removed net N$36: C33.1, U$1.RLMC5
- removed net N$37: C34.1, U$1.RLC5
- removed net N$38: C35.1, U$1.ROUT
- removed net N$39: C36.1, U$1.RBOOS2
- removed net N$40: C37.1, U$1.RIN
- removed net N$41: C38.1, U$1.RCUT2
- removed net N$42: C39.1, U$1.LCUT1
- removed net N$43: C40.1, U$1.LIN
- removed net N$44: C41.1, U$1.LBOOS1
- removed net N$45: C42.1, U$1.LOUT
- removed net N$46: C10.2, U$1.LLMC2
- removed net N$47: C11.2, C27.2, U$1.LLMC3
- removed net N$48: C12.2, U$1.LHMC2
- removed net N$49: C13.2, C28.2, U$1.LHMC3
- removed net N$50: C14.2, U$1.LHC2
- removed net N$51: C15.2, C29.2, U$1.LHC3
- removed net N$59: C16.2, C31.2, U$1.RHC3
- removed net N$60: C17.2, U$1.RHC2
- removed net N$61: C18.2, C32.2, U$1.RHMC3
- removed net N$62: C19.2, U$1.RHMC2
- removed net N$63: C20.2, C33.2, U$1.RLMC3
- removed net N$64: C21.2, U$1.RLMC2
- removed net N$65: C22.2, C34.2, U$1.RLC3
- removed net N$66: C23.2, U$1.RLC2
- removed net N$67: C36.2, U$1.RBOOS1
- removed net N$68: C37.2
- removed net N$69: C38.2, U$1.RCUT1
- removed net N$70: C39.2, U$1.LCUT2
- removed net N$71: C40.2
- removed net N$72: C41.2, U$1.LBOOS2
- removed net N$9: C8.1, U$1.LLC1
- removed net SCK: U1.GPIO11/SPI_SCLK
- removed net SCL_0: U9.SC0
- removed net SCL_1: U9.SD0
- removed net SCL_2: U9.SC2
- removed net SCL_3: U9.SD2
- removed net SDA_0: U9.SC1
- removed net SDA_1: U9.SD1
- removed net SDA_2: U9.SC3
- removed net SDA_3: U9.SD3
- removed net SDI/O: U1.GPIO10/SPI_MOSI
- new net 3V3A: C3.1, C4.1, IC1.AVDD
- new net 3V3D: C1.1, C2.1, IC1.DVDD, IC1.IOVDD
- new net GND: C1.2, C2.2, C3.2, C4.2, C5.2, C6.2, C7.2, IC1.AGND, IC1.DGND
- new net VIN1: IC1.VINL2/VIN1M
- new net VIN2: IC1.VINL1/VIN1P
- new net VIN3: IC1.VINR3/VIN3P
- new net VIN4: IC1.VINR4/VIN3M
- net BCK_ADC: no longer U1.GPIO27/GPIO_GEN2
- net CLK_ADC: no longer U1.GPIO4/GPIO_GCKL
- net DOUT_ADC: no longer U1.GPIO17/GPIO_GEN0
- net LRCK_ADC: no longer U1.GPIO18/GPIO_GEN1
- net SCL: no longer U1.GPIO3/SCL1, U9.SCL
- net SDA: no longer U1.GPIO2/SDA1, U9.SDA
Other:
- moved on the sheet: C1, C2, C3, C4, C5, C6, C7, IC1

Commit message: corrections
Parts:
- added BCK_ADC, CLK_ADC, DOUT_ADC, LRCK_ADC: (no value), wirepad:SMD2
- C1, C2, C3, C4, C5, C6, C7: device rcl:C-US025-024X044 -> rcl:C-USC0402
Connections:
- net BCK_ADC: now also BCK_ADC.P
- net CLK_ADC: now also CLK_ADC.P
- net DOUT_ADC: now also DOUT_ADC.P
- net LRCK_ADC: now also LRCK_ADC.P
Changed lines of the file:
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@@
 <layers>
 <layer number="1" name="Top" color="4" fill="1" visible="no" active="no"/>
+<layer number="2" name="Route2" color="1" fill="3" visible="no" active="no"/>
+<layer number="3" name="Route3" color="4" fill="3" visible="no" active="no"/>
+<layer number="4" name="Route4" color="1" fill="4" visible="no" active="no"/>
+<layer number="5" name="Route5" color="4" fill="4" visible="no" active="no"/>
+<layer number="6" name="Route6" color="1" fill="8" visible="no" active="no"/>
+<layer number="7" name="Route7" color="4" fill="8" visible="no" active="no"/>
+<layer number="8" name="Route8" color="1" fill="2" visible="no" active="no"/>
+<layer number="9" name="Route9" color="4" fill="2" visible="no" active="no"/>
+<layer number="10" name="Route10" color="1" fill="7" visible="no" active="no"/>
+<layer number="11" name="Route11" color="4" fill="7" visible="no" active="no"/>
+<layer number="12" name="Route12" color="1" fill="5" visible="no" active="no"/>
+<layer number="13" name="Route13" color="4" fill="5" visible="no" active="no"/>
+<layer number="14" name="Route14" color="1" fill="6" visible="no" active="no"/>
+<layer number="15" name="Route15" color="4" fill="6" visible="no" active="no"/>
 <layer number="16" name="Bottom" color="1" fill="1" visible="no" active="no"/>
 <layer number="17" name="Pads" color="2" fill="1" visible="no" active="no"/>
@@
 <parts>
 <part name="IC1" library="PCM1865DBT" deviceset="PCM1865DBT" device=""/>
-<part name="C1" library="rcl" library_urn="urn:adsk.eagle:library:334" deviceset="C-US" device="025-024X044" package3d_urn="urn:adsk.eagle:package:23630/1" value="0.1μF"/>
-<part name="C2" library="rcl" library_urn="urn:adsk.eagle:library:334" deviceset="C-US" device="025-024X044" package3d_urn="urn:adsk.eagle:package:23630/1" value="10μF"/>
-<part name="C3" library="rcl" library_urn="urn:adsk.eagle:library:334" deviceset="C-US" device="025-024X044" package3d_urn="urn:adsk.eagle:package:23630/1" value="0.1μF"/>
-<part name="C4" library="rcl" library_urn="urn:adsk.eagle:library:334" deviceset="C-US" device="025-024X044" package3d_urn="urn:adsk.eagle:package:23630/1" value="10μF"/>
-<part name="C5" library="rcl" library_urn="urn:adsk.eagle:library:334" deviceset="C-US" device="025-024X044" package3d_urn="urn:adsk.eagle:package:23630/1" value="1μF"/>
-<part name="C6" library="rcl" library_urn="urn:adsk.eagle:library:334" deviceset="C-US" device="025-024X044" package3d_urn="urn:adsk.eagle:package:23630/1" value="0.1μF"/>
-<part name="C7" library="rcl" library_urn="urn:adsk.eagle:library:334" deviceset="C-US" device="025-024X044" package3d_urn="urn:adsk.eagle:package:23630/1" value="1μF"/>
+<part name="C1" library="rcl" library_urn="urn:adsk.eagle:library:334" deviceset="C-US" device="C0402" package3d_urn="urn:adsk.eagle:package:23626/2" value="0.1μF"/>
+<part name="C2" library="rcl" library_urn="urn:adsk.eagle:library:334" deviceset="C-US" device="C0402" package3d_urn="urn:adsk.eagle:package:23626/2" value="10μF"/>
+<part name="C3" library="rcl" library_urn="urn:adsk.eagle:library:334" deviceset="C-US" device="C0402" package3d_urn="urn:adsk.eagle:package:23626/2" value="0.1μF"/>
+<part name="C4" library="rcl" library_urn="urn:adsk.eagle:library:334" deviceset="C-US" device="C0402" package3d_urn="urn:adsk.eagle:package:23626/2" value="10μF"/>
+<part name="C5" library="rcl" library_urn="urn:adsk.eagle:library:334" deviceset="C-US" device="C0402" package3d_urn="urn:adsk.eagle:package:23626/2" value="1μF"/>
+<part name="C6" library="rcl" library_urn="urn:adsk.eagle:library:334" deviceset="C-US" device="C0402" package3d_urn="urn:adsk.eagle:package:23626/2" value="0.1μF"/>
+<part name="C7" library="rcl" library_urn="urn:adsk.eagle:library:334" deviceset="C-US" device="C0402" package3d_urn="urn:adsk.eagle:package:23626/2" value="1μF"/>
+<part name="CLK_ADC" library="wirepad" library_urn="urn:adsk.eagle:library:412" deviceset="SMD2" device="" package3d_urn="urn:adsk.eagle:package:30839/1"/>
+<part name="LRCK_ADC" library="wirepad" library_urn="urn:adsk.eagle:library:412" deviceset="SMD2" device="" package3d_urn="urn:adsk.eagle:package:30839/1"/>
+<part name="BCK_ADC" library="wirepad" library_urn="urn:adsk.eagle:library:412" deviceset="SMD2" device="" package3d_urn="urn:adsk.eagle:package:30839/1"/>
+<part name="DOUT_ADC" library="wirepad" library_urn="urn:adsk.eagle:library:412" deviceset="SMD2" device="" package3d_urn="urn:adsk.eagle:package:30839/1"/>
 </parts>
 <sheets>
@@
 <attribute name="VALUE" x="8.636" y="11.049" size="1.778" layer="96"/>
 </instance>
+<instance part="CLK_ADC" gate="1" x="40.64" y="2.54" smashed="yes" rot="R180">
+<attribute name="NAME" x="41.783" y="0.6858" size="1.778" layer="95" rot="R180"/>
+<attribute name="VALUE" x="41.783" y="5.842" size="1.778" layer="96" rot="R180"/>
+</instance>
+<instance part="LRCK_ADC" gate="1" x="91.44" y="10.16" smashed="yes" rot="R90">
+<attribute name="NAME" x="89.5858" y="9.017" size="1.778" layer="95" rot="R90"/>
+<attribute name="VALUE" x="94.742" y="9.017" size="1.778" layer="96" rot="R90"/>
+</instance>
+<instance part="BCK_ADC" gate="1" x="111.76" y="12.7" smashed="yes">
+<attribute name="NAME" x="110.617" y="14.5542" size="1.778" layer="95"/>
+<attribute name="VALUE" x="110.617" y="9.398" size="1.778" layer="96"/>
+</instance>
+<instance part="DOUT_ADC" gate="1" x="101.6" y="22.86" smashed="yes" rot="R270">
+<attribute name="NAME" x="103.4542" y="24.003" size="1.778" layer="95"/>
+<attribute name="VALUE" x="98.298" y="24.003" size="1.778" layer="96" rot="R270"/>
+</instance>
 </instances>
 <busses>
@@
 <segment>
 <pinref part="IC1" gate="G$1" pin="SCKI"/>
-<wire x1="38.1" y1="12.7" x2="38.1" y2="5.08" width="0.1524" layer="91"/>
-<label x="38.1" y="5.08" size="1.778" layer="95" xref="yes"/>
+<wire x1="38.1" y1="12.7" x2="38.1" y2="2.54" width="0.1524" layer="91"/>
+<label x="38.1" y="-2.54" size="1.778" layer="95" rot="R270" xref="yes"/>
+<pinref part="CLK_ADC" gate="1" pin="P"/>
+<wire x1="38.1" y1="2.54" x2="38.1" y2="-2.54" width="0.1524" layer="91"/>
+<junction x="38.1" y="2.54"/>
 </segment>
 </net>
@@
 <segment>
 <pinref part="IC1" gate="G$1" pin="DOUT"/>
-<wire x1="88.9" y1="17.78" x2="93.98" y2="17.78" width="0.1524" layer="91"/>
-<label x="93.98" y="17.78" size="1.778" layer="95" xref="yes"/>
+<wire x1="88.9" y1="17.78" x2="101.6" y2="20.32" width="0.1524" layer="91"/>
+<label x="101.6" y="20.32" size="1.778" layer="95" xref="yes"/>
+<pinref part="DOUT_ADC" gate="1" pin="P"/>
 </segment>
 </net>
@@
 <segment>
 <pinref part="IC1" gate="G$1" pin="BCK"/>
-<wire x1="88.9" y1="15.24" x2="111.76" y2="15.24" width="0.1524" layer="91"/>
-<label x="111.76" y="15.24" size="1.778" layer="95" xref="yes"/>
+<wire x1="88.9" y1="15.24" x2="114.3" y2="12.7" width="0.1524" layer="91"/>
+<label x="114.3" y="12.7" size="1.778" layer="95" xref="yes"/>
+<pinref part="BCK_ADC" gate="1" pin="P"/>
 </segment>
 </net>
@@
 <segment>
 <pinref part="IC1" gate="G$1" pin="LRCK"/>
-<wire x1="88.9" y1="12.7" x2="93.98" y2="12.7" width="0.1524" layer="91"/>
-<label x="93.98" y="12.7" size="1.778" layer="95" xref="yes"/>
-</segment>
-</net>
+<wire x1="88.9" y1="12.7" x2="91.44" y2="12.7" width="0.1524" layer="91"/>
+<label x="99.06" y="5.08" size="1.778" layer="95" xref="yes"/>
+<pinref part="LRCK_ADC" gate="1" pin="P"/>
+<wire x1="91.44" y1="12.7" x2="99.06" y2="5.08" width="0.1524" layer="91"/>
+<junction x="91.44" y="12.7"/>
+</segment>
+</net>

Commit message: updates
Connections:
- net VIN1 renamed IN1L_ADC
- net VIN2 renamed IN2L_ADC
- net VIN3 renamed IN3L_ADC
- net VIN4 renamed IN4L_ADC
- new net IN1R_ADC: IC1.VINR2/VIN2M
- new net IN2R_ADC: IC1.VINR1/VIN2P
- new net IN3R_ADC: IC1.VINL3/VIN4P
- new net IN4R_ADC: IC1.VINL4/VIN4M
- net GND: now also IC1.MS/AD
Changed lines of the file:
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@@
 </segment>
 </net>
-<net name="VIN2" class="0">
+<net name="IN2L_ADC" class="0">
 <segment>
 <pinref part="IC1" gate="G$1" pin="VINL1/VIN1P"/>
@@
 </segment>
 </net>
-<net name="VIN1" class="0">
+<net name="IN1L_ADC" class="0">
 <segment>
 <pinref part="IC1" gate="G$1" pin="VINL2/VIN1M"/>
 <wire x1="38.1" y1="48.26" x2="33.02" y2="48.26" width="0.1524" layer="91"/>
+<label x="33.02" y="48.26" size="1.778" layer="95" rot="R180" xref="yes"/>
+<label x="33.02" y="48.26" size="1.778" layer="95" rot="R180" xref="yes"/>
 <label x="33.02" y="48.26" size="1.778" layer="95" rot="R180" xref="yes"/>
 </segment>
@@
 </segment>
 </net>
-<net name="VIN3" class="0">
+<net name="IN3L_ADC" class="0">
 <segment>
 <pinref part="IC1" gate="G$1" pin="VINR3/VIN3P"/>
@@
 </segment>
 </net>
-<net name="VIN4" class="0">
+<net name="IN4L_ADC" class="0">
 <segment>
 <pinref part="IC1" gate="G$1" pin="VINR4/VIN3M"/>
@@
 <label x="139.7" y="50.8" size="1.778" layer="95" rot="R270" xref="yes"/>
 </segment>
+<segment>
+<pinref part="IC1" gate="G$1" pin="MS/AD"/>
+<wire x1="88.9" y1="35.56" x2="93.98" y2="35.56" width="0.1524" layer="91"/>
+<label x="93.98" y="35.56" size="1.778" layer="95" xref="yes"/>
+</segment>
 </net>
 <net name="3V3D" class="0">
@@
 </segment>
 </net>
+<net name="IN1R_ADC" class="0">
+<segment>
+<pinref part="IC1" gate="G$1" pin="VINR2/VIN2M"/>
+<wire x1="38.1" y1="45.72" x2="33.02" y2="45.72" width="0.1524" layer="91"/>
+<label x="33.02" y="45.72" size="1.778" layer="95" rot="R180" xref="yes"/>
+</segment>
+</net>
+<net name="IN2R_ADC" class="0">
+<segment>
+<pinref part="IC1" gate="G$1" pin="VINR1/VIN2P"/>
+<wire x1="38.1" y1="40.64" x2="33.02" y2="40.64" width="0.1524" layer="91"/>
+<label x="33.02" y="40.64" size="1.778" layer="95" rot="R180" xref="yes"/>
+</segment>
+</net>
+<net name="IN3R_ADC" class="0">
+<segment>
+<pinref part="IC1" gate="G$1" pin="VINL3/VIN4P"/>
+<wire x1="38.1" y1="35.56" x2="33.02" y2="35.56" width="0.1524" layer="91"/>
+<label x="33.02" y="35.56" size="1.778" layer="95" rot="R180" xref="yes"/>
+</segment>
+</net>
+<net name="IN4R_ADC" class="0">
+<segment>
+<pinref part="IC1" gate="G$1" pin="VINL4/VIN4M"/>
+<wire x1="38.1" y1="30.48" x2="33.02" y2="30.48" width="0.1524" layer="91"/>
+<label x="33.02" y="30.48" size="1.778" layer="95" rot="R180" xref="yes"/>
+</segment>
+</net>

Commit message: v2 of board finished
Parts:
- added C10, C11, C12, C13, C14, C15, C17, C18: 10uF, rcl:C-USC0402
- added C8, C9: 15pF, rcl:C-USC0402
- added Y1: CM7V-T1A-32.768KHZ-12.5PF-100PPM-TB-QC, CM7V-T1A-32.768KHZ-12.5PF-100PPM-TB-QC:CM7V-T1A-32.768KHZ-12.5PF-100PPM-TB-QC
- C1, C3, C6: value 0.1μF -> 0.1uF
- C2, C4: value 10μF -> 10uF
- C5, C7: value 1μF -> 1uF
Connections:
- removed net IN1L_ADC: IC1.VINL2/VIN1M
- removed net IN1R_ADC: IC1.VINR2/VIN2M
- removed net IN2L_ADC: IC1.VINL1/VIN1P
- removed net IN2R_ADC: IC1.VINR1/VIN2P
- removed net IN3L_ADC: IC1.VINR3/VIN3P
- removed net IN3R_ADC: IC1.VINL3/VIN4P
- removed net IN4L_ADC: IC1.VINR4/VIN3M
- removed net IN4R_ADC: IC1.VINL4/VIN4M
- new net N$1: C8.1, IC1.XO, Y1.2
- new net N$12: C17.2, IC1.VINR4/VIN3M
- new net N$13: C13.2, IC1.VINL4/VIN4M
- new net N$14: C17.1
- new net N$15: C13.1
- new net N$17: C11.1
- new net N$18: C14.1
- new net N$19: C10.1
- new net N$2: C9.1, IC1.XI, Y1.1
- new net N$20: C18.1
- new net N$21: C15.2, IC1.VINR3/VIN3P
- new net N$3: C15.1
- new net N$4: C12.1
- new net N$5: C18.2, IC1.VINL2/VIN1M
- new net N$6: C10.2, IC1.VINR2/VIN2M
- new net N$7: C14.2, IC1.VINL1/VIN1P
- new net N$8: C11.2, IC1.VINR1/VIN2P
- new net N$9: C12.2, IC1.VINL3/VIN4P
- net GND: now also C8.2, C9.2
