File: equalizer.brd (EAGLE design)
At the start: 41.9 x 40.3 mm, 34 parts

Commit message: corrections
Parts:
- removed C86, C89: 10uF, rcl:C0402
- added C1: 10uF, rcl:C0402
- added CE_EQ, CL_EQ, DI_EQ: (no value), wirepad:SMD1,27-2,54
- C60, C61, C64, C65, C66, C67, C70, C71: value 0.047uF -> 0.01uF
- C62, C63, C68, C69: value 0.047uF -> 0.068uF
- C84, C91: value 10uF -> 0.1uF
Connections:
- removed net N$199: C86.1, U$14.53
- removed net N$202: C89.1, U$14.60
- net EIN0: now also U$14.53; no longer C86.2
- net EIN1: now also U$14.60; no longer C89.2
- net EQ1_CE: now also CE_EQ.1
- net EQ1_CL: now also CL_EQ.1
- net EQ1_DI: now also DI_EQ.1
- net GND: now also C1.2
- net N$192: now also C1.1
Routing:
- net N$199: track 4.41 -> 0.00 mm
- net N$202: track 3.34 -> 0.00 mm
- net EIN0: track 5.32 -> 3.07 mm
- net EIN1: track 5.12 -> 3.16 mm
- net VDD: track 3.48 -> 5.16 mm
- net GND: track 17.1 -> 18.4 mm
- net EQ1_CL: track 10.0 -> 10.5 mm, vias 0 -> 1
- net EQ1_DI: track 10.2 -> 9.76 mm, vias 0 -> 1
- net EQ1_CE: track 8.61 -> 8.24 mm, vias 0 -> 1
Other:
- board outline removed

Commit message: updates
Connections:
- net EIN0 renamed IN1_EQ
- net EIN1 renamed IN2_EQ
- net EOUT0 renamed OUT1_EQ
- net EOUT1 renamed OUT2_EQ
Changed lines of the file:
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@@
 <wire x1="10.77158125" y1="15.45" x2="13.4631" y2="15.45" width="0.508" layer="1"/>
 </signal>
-<signal name="EOUT0">
+<signal name="OUT1_EQ">
 <contactref element="C84" pad="2"/>
 <wire x1="7.351" y1="24.511" x2="2.921" y2="24.511" width="0.508" layer="1"/>
 <wire x1="2.921" y1="24.511" x2="2.54" y2="24.13" width="0.508" layer="1"/>
 </signal>
-<signal name="EOUT1">
+<signal name="OUT2_EQ">
 <contactref element="C91" pad="2"/>
 <wire x1="9.256" y1="12.446" x2="4.064" y2="12.446" width="0.508" layer="1"/>
@@
 <wire x1="33.9987" y1="16.51" x2="34.29" y2="16.51" width="0.508" layer="15"/>
 </signal>
-<signal name="EIN1">
+<signal name="IN2_EQ">
 <contactref element="U$14" pad="60"/>
 <wire x1="13.4631" y1="16.25" x2="10.308" y2="16.25" width="0.508" layer="1"/>
 </signal>
-<signal name="EIN0">
+<signal name="IN1_EQ">
 <contactref element="U$14" pad="53"/>
 <wire x1="13.4631" y1="21.85" x2="13.432" y2="21.8189" width="0.508" layer="1"/>

Commit message: v2 of board finished
Parts:
- moved C1 40.2 mm to (38.4, 16.8), turned to 270 degrees
- moved C79 1.83 mm to (36.8, 16.8), turned to 270 degrees
Routing:
- net N$192: track 5.47 -> 9.07 mm
- net GND: track 18.4 -> 19.8 mm
Changed lines of the file:
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@@
 <attribute name="VALUE" x="32.639" y="12.7" size="1.27" layer="27"/>
 </element>
-<element name="C79" library="rcl" library_urn="urn:adsk.eagle:library:334" package="C0402" package3d_urn="urn:adsk.eagle:package:23626/2" value="10uF" x="35.306" y="17.78" smashed="yes">
-<attribute name="NAME" x="34.671" y="18.415" size="1.27" layer="25"/>
-<attribute name="POPULARITY" value="16" x="59.436" y="-26.67" size="1.778" layer="27" display="off"/>
-<attribute name="SPICEPREFIX" value="C" x="59.436" y="-26.67" size="1.778" layer="27" display="off"/>
-<attribute name="VALUE" x="34.671" y="15.875" size="1.27" layer="27"/>
+<element name="C79" library="rcl" library_urn="urn:adsk.eagle:library:334" package="C0402" package3d_urn="urn:adsk.eagle:package:23626/2" value="10uF" x="36.83" y="16.764" smashed="yes" rot="R270">
+<attribute name="NAME" x="37.465" y="17.399" size="1.27" layer="25" rot="R270"/>
+<attribute name="POPULARITY" value="16" x="-7.62" y="-7.366" size="1.778" layer="27" rot="R270" display="off"/>
+<attribute name="SPICEPREFIX" value="C" x="-7.62" y="-7.366" size="1.778" layer="27" rot="R270" display="off"/>
+<attribute name="VALUE" x="34.925" y="17.399" size="1.27" layer="27" rot="R270"/>
 </element>
 <element name="C80" library="rcl" library_urn="urn:adsk.eagle:library:334" package="C0402" package3d_urn="urn:adsk.eagle:package:23626/2" value="10uF" x="33.02" y="23.495" smashed="yes">
@@
 <attribute name="VALUE" x="39.497" y="20.193" size="0.0254" layer="28" rot="MR90"/>
 </element>
-<element name="C1" library="rcl" library_urn="urn:adsk.eagle:library:334" package="C0402" package3d_urn="urn:adsk.eagle:package:23626/2" value="10uF" x="3.81" y="-3.81" smashed="yes">
-<attribute name="NAME" x="3.175" y="-3.175" size="1.27" layer="25"/>
-<attribute name="POPULARITY" value="16" x="3.81" y="-3.81" size="1.778" layer="27" display="off"/>
-<attribute name="SPICEPREFIX" value="C" x="3.81" y="-3.81" size="1.778" layer="27" display="off"/>
-<attribute name="VALUE" x="3.175" y="-5.715" size="1.27" layer="27"/>
+<element name="C1" library="rcl" library_urn="urn:adsk.eagle:library:334" package="C0402" package3d_urn="urn:adsk.eagle:package:23626/2" value="10uF" x="38.354" y="16.764" smashed="yes" rot="R270">
+<attribute name="NAME" x="38.989" y="17.399" size="1.27" layer="25" rot="R270"/>
+<attribute name="POPULARITY" value="16" x="38.354" y="16.764" size="1.778" layer="27" rot="R270" display="off"/>
+<attribute name="SPICEPREFIX" value="C" x="38.354" y="16.764" size="1.778" layer="27" rot="R270" display="off"/>
+<attribute name="VALUE" x="36.449" y="17.399" size="1.27" layer="27" rot="R270"/>
 </element>
 </elements>
@@
 <contactref element="C79" pad="1"/>
 <contactref element="U$14" pad="23"/>
-<wire x1="34.656" y1="17.78" x2="33.9821" y2="18.4539" width="0.508" layer="1"/>
+<wire x1="36.83" y1="17.414" x2="33.9821" y2="18.4539" width="0.508" layer="1"/>
 <wire x1="29.7169" y1="17.85" x2="31.1139" y2="17.85" width="0.508" layer="1"/>
 <wire x1="31.7178" y1="18.4539" x2="31.1139" y2="17.85" width="0.508" layer="1"/>
 <wire x1="33.9821" y1="18.4539" x2="31.7178" y2="18.4539" width="0.508" layer="1"/>
 <contactref element="C1" pad="1"/>
-<wire x1="3.16" y1="-3.81" x2="29.7169" y2="17.85" width="0" layer="19" extent="1-1"/>
+<wire x1="36.83" y1="17.414" x2="38.354" y2="17.414" width="0.508" layer="1"/>
 </signal>
 <signal name="N$193">
@@
 <wire x1="29.7169" y1="16.25" x2="32.6379" y2="16.25" width="0.508" layer="1"/>
 <wire x1="32.7706" y1="16.3827" x2="32.6379" y2="16.25" width="0.508" layer="1"/>
-<wire x1="32.7706" y1="16.3827" x2="35.4327" y2="16.3827" width="0.508" layer="1"/>
-<wire x1="35.956" y1="17.78" x2="35.956" y2="16.906" width="0.508" layer="1"/>
-<wire x1="35.956" y1="16.906" x2="35.4327" y2="16.3827" width="0.508" layer="1"/>
+<wire x1="32.7706" y1="16.3827" x2="36.53348125" y2="16.3827" width="0.508" layer="1"/>
+<wire x1="36.83" y1="16.114" x2="36.53348125" y2="16.3827" width="0.508" layer="1"/>
 <wire x1="27.94" y1="19.05" x2="26.67" y2="19.05" width="0.508" layer="1"/>
 <via x="26.67" y="19.05" extent="1-16" drill="0.508"/>
 <wire x1="26.67" y1="19.05" x2="25.4" y2="19.05" width="0.508" layer="2"/>
 <contactref element="C1" pad="2"/>
-<wire x1="4.46" y1="-3.81" x2="25.4" y2="19.05" width="0" layer="19" extent="1-2"/>
+<wire x1="38.354" y1="16.114" x2="36.83" y2="16.114" width="0.508" layer="1"/>
 </signal>
 <signal name="VDD">
