File: mixer.brd (EAGLE design)
At the start: 20 parts, among them U1 LM4562MAX/NOPB

Commit message: updates
Parts:
- removed AOUT, GND: (no value), wirepad:SMD2,54-5,08
- removed U1: LM4562MAX/NOPB, LM4562MAX_NOPB:SOIC127P599X175-8N
- added C2: 0.1u, rcl:C0402
- added GNDL, GNDR, OUTL_MIX, OUTR_MIX: (no value), wirepad:SMD2,54-5,08
- added OPAMP1_MIX: LM4562MAX/NOPB, LM4562MAX_NOPB:SOIC127P599X175-8N
- added R17, R19, R26, R27: 10k, rcl:R0402
- added R18, R20, R21, R22, R23, R24, R25, R28: 5k, rcl:R0402
- added R29: 50k, rcl:R0402
- added R30: 1k, rcl:R0402
- R11, R12, R2, R4: value 20k -> 10k
- R13, R14: value 20k -> 5k
- R15: value 20k -> 50k
- moved R1 23.3 mm to (16.3, -8.89), turned to 180 degrees
- moved R8 21.0 mm to (15.7, -7.62), turned to 0 degrees
- moved R14 19.4 mm to (-1.27, 0.00), turned to 0 degrees
- moved R7 18.9 mm to (15.7, -6.35), turned to 0 degrees
- moved R12 18.8 mm to (13.2, -7.62), turned to 180 degrees
- moved C1 17.9 mm to (14.5, -9.78), turned to 270 degrees
- moved R3 17.1 mm to (15.7, -5.21), turned to 180 degrees
- moved R11 16.3 mm to (13.3, -6.22), turned to 180 degrees
- moved R16 16.3 mm to (13.1, -9.40)
- moved R10 14.9 mm to (15.7, -3.68), turned to 180 degrees
- moved R6 13.4 mm to (15.7, -2.41), turned to 0 degrees
- moved R15 13.0 mm to (11.8, -9.27), turned to 270 degrees
- moved R5 12.4 mm to (15.9, -1.14), turned to 180 degrees
- moved R13 12.1 mm to (12.4, -4.32), turned to 180 degrees
- moved R9 11.7 mm to (15.9, 0.13), turned to 180 degrees
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Connections:
- net AIN0 renamed IN1L_MIX
- net AIN1 renamed IN2L_MIX
- net AIN2 renamed IN3L_MIX
- net AIN3 renamed IN4L_MIX
- removed net AOUT: AOUT.1, C1.2
- new net IN1R_MIX: R24.1
- new net IN2R_MIX: R25.1
- new net IN3R_MIX: R18.1
- new net IN4R_MIX: R14.1
- new net N$3: R17.1, R20.2, R24.2
- new net N$6: R18.2, R22.1, R26.1
- new net N$7: R19.1, R21.1, R25.2
- new net NEG_A_MIX: OPAMP1_MIX.2, R13.2, R15.1
- new net NEG_B_MIX: OPAMP1_MIX.6, R28.2, R29.1
- new net OUTL_MIX: C1.2, OUTL_MIX.1
- new net OUTR_MIX: C2.2, OUTR_MIX.1
- new net OUT_A_MIX: OPAMP1_MIX.1, R15.2, R16.1
- new net OUT_B_MIX: OPAMP1_MIX.7, R29.2, R30.1
- net GND: now also GNDL.1, GNDR.1, OPAMP1_MIX.4; no longer GND.1, U1.4
- net N$14: no longer U1.6
- net N$2: now also C2.1, R30.2; no longer R14.2, R16.1, U1.1
- net N$4: now also R17.2, R19.2, R26.2, R27.2, R28.1; no longer R13.2, R15.1, U1.7
- net N$5: now also R14.2, R23.1, R27.1; no longer R14.1, R15.2, U1.2
- net VDD: now also OPAMP1_MIX.8; no longer U1.8
- net VREF: now also OPAMP1_MIX.3, OPAMP1_MIX.5, R20.1, R21.2, R22.2, R23.2; no longer U1.3, U1.5
Routing:
- net VREF: track 25.1 -> 44.8 mm, vias 3 -> 5
- net AOUT: track 8.48 -> 0.00 mm
- net NEG_A_MIX: track 0.00 -> 6.37 mm
- net NEG_B_MIX: track 0.00 -> 4.47 mm
- net OUTL_MIX: track 0.00 -> 4.14 mm
- net OUTR_MIX: track 0.00 -> 4.08 mm
- net OUT_B_MIX: track 0.00 -> 3.31 mm
- net IN4R_MIX: track 0.00 -> 3.31 mm
- net IN3R_MIX: track 0.00 -> 3.31 mm
- net IN2R_MIX: track 0.00 -> 3.31 mm
- net IN1R_MIX: track 0.00 -> 3.31 mm
- net OUT_A_MIX: track 0.00 -> 3.28 mm
- net N$5: track 5.90 -> 2.81 mm
- net N$14: track 9.50 -> 6.59 mm
- net N$3: track 0.00 -> 2.81 mm
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
Commit message: v2 of board finished
Changed lines of the file:
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@@
 <contactref element="R16" pad="2"/>
 <contactref element="C1" pad="1"/>
-<wire x1="13.081" y1="-8.748" x2="13.081" y2="-8.898" width="0.508" layer="1"/>
 <wire x1="13.081" y1="-8.898" x2="14.247" y2="-8.898" width="0.508" layer="1"/>
 <wire x1="14.247" y1="-8.898" x2="14.478" y2="-9.129" width="0.508" layer="1"/>
@@
 <wire x1="12.708" y1="-6.35" x2="12.835" y2="-6.223" width="0.508" layer="1"/>
 <wire x1="12.962" y1="-2.413" x2="12.962" y2="-1.143" width="0.508" layer="1"/>
-<wire x1="12.954" y1="-2.421" x2="12.962" y2="-2.413" width="0.508" layer="1"/>
-<wire x1="12.962" y1="-2.413" x2="12.946" y2="-2.429" width="0.508" layer="1"/>
-<wire x1="12.946" y1="-2.429" x2="12.946" y2="-4.318" width="0.508" layer="1"/>
 <wire x1="12.946" y1="-4.318" x2="12.835" y2="-4.429" width="0.508" layer="1"/>
 <wire x1="12.835" y1="-4.429" x2="12.835" y2="-6.223" width="0.508" layer="1"/>
+<wire x1="12.946" y1="-4.318" x2="12.946" y2="-2.429" width="0.508" layer="1"/>
+<wire x1="12.946" y1="-2.429" x2="12.962" y2="-2.413" width="0.508" layer="1"/>
 </signal>
 <signal name="N$15">
@@
 <contactref element="R13" pad="2"/>
 <contactref element="OPAMP1_MIX" pad="2"/>
-<wire x1="9.971" y1="-8.771" x2="9.963" y2="-8.763" width="0.508" layer="1"/>
 <wire x1="11.946" y1="-4.318" x2="11.946" y2="-8.636" width="0.508" layer="1"/>
-<wire x1="11.946" y1="-8.636" x2="11.811" y2="-8.771" width="0.508" layer="1"/>
-<wire x1="9.963" y1="-8.763" x2="11.803" y2="-8.763" width="0.508" layer="1"/>
+<wire x1="11.819" y1="-8.763" x2="11.811" y2="-8.771" width="0.508" layer="1"/>
 <wire x1="11.803" y1="-8.763" x2="11.811" y2="-8.771" width="0.508" layer="1"/>
+<wire x1="9.963" y1="-8.763" x2="11.819" y2="-8.763" width="0.508" layer="1"/>
+<wire x1="11.819" y1="-8.763" x2="11.946" y2="-8.636" width="0.508" layer="1"/>
 </signal>
 <signal name="OUT_A_MIX">
