File: nopi.brd (EAGLE design)
At the start: 15 parts, among them U6 TMUX1204DGSR, U7 TMUX1204DGSR, U8 TMUX1204DGSR, U9 TCA9546ADR

Commit message: updates
Parts:
- added CS: (no value), wirepad:SMD1,27-2,54
- added U1: TMUX1204DGSR, TMUX1204DGSR:SOP50P490X110-10N
Connections:
- net CS0_0 renamed CS0_COMP1
- net CS0_1 renamed CS0_COMP2
- net CS0_2 renamed CS0_COMP3
- net CS0_3 renamed CS0_COMP4
- net CS1_0 renamed CS1_COMP1
- net CS1_1 renamed CS1_COMP2
- net CS1_2 renamed CS1_COMP3
- net CS1_3 renamed CS1_COMP4
- net CS2_0 renamed CS2_COMP1
- net CS2_1 renamed CS2_COMP2
- net CS2_2 renamed CS2_COMP3
- net CS2_3 renamed CS2_COMP4
- new net CS: CS.1, U1.8
- new net CS0_PAN4: U1.7
- new net CS_PAN1: U1.2
- new net CS_PAN2: U1.9
- new net CS_PAN3: U1.4
- net +3V3: now also U1.5, U1.6
- net DGND: now also U1.3
- net MUX0: now also U1.1
- net MUX1: now also U1.10
Changed lines of the file:
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@@
 <attribute name="VALUE" x="19.05" y="5.01" size="0.0254" layer="28" rot="MR0"/>
+</element>
+<element name="U1" library="TMUX1204DGSR" package="SOP50P490X110-10N" value="TMUX1204DGSR" x="3.81" y="-3.81" smashed="yes">
+<attribute name="AVAILABILITY" value="In Stock" x="3.81" y="-3.81" size="1.778" layer="27" display="off"/>
+<attribute name="CHECK_PRICES" value="https://www.snapeda.com/parts/TMUX1204DGSR/Texas+Instruments/view-part/?ref=eda" x="3.81" y="-3.81" size="1.778" layer="27" display="off"/>
+<attribute name="DESCRIPTION" value=" 5-V, 4:1, 1-channel, general-purpose analog multiplexer " x="3.81" y="-3.81" size="1.778" layer="27" display="off"/>
+<attribute name="MF" value="Texas Instruments" x="3.81" y="-3.81" size="1.778" layer="27" display="off"/>
+<attribute name="MP" value="TMUX1204DGSR" x="3.81" y="-3.81" size="1.778" layer="27" display="off"/>
+<attribute name="NAME" x="0.81" y="-1.81" size="1.016" layer="25"/>
+<attribute name="PACKAGE" value="VSSOP-10 Texas Instruments" x="3.81" y="-3.81" size="1.778" layer="27" display="off"/>
+<attribute name="PRICE" value="None" x="3.81" y="-3.81" size="1.778" layer="27" display="off"/>
+<attribute name="PURCHASE-URL" value="https://www.snapeda.com/api/url_track_click_mouser/?unipart_id=3657556&amp;manufacturer=Texas Instruments&amp;part_name=TMUX1204DGSR&amp;search_term=tmux1204" x="3.81" y="-3.81" size="1.778" layer="27" display="off"/>
+<attribute name="SNAPEDA_LINK" value="https://www.snapeda.com/parts/TMUX1204DGSR/Texas+Instruments/view-part/?ref=snap" x="3.81" y="-3.81" size="1.778" layer="27" display="off"/>
+<attribute name="VALUE" x="0.81" y="-5.81" size="1.016" layer="27" align="top-left"/>
+</element>
+<element name="CS" library="wirepad" library_urn="urn:adsk.eagle:library:412" package="SMD1,27-2,54" package3d_urn="urn:adsk.eagle:package:30839/1" value="" x="-1.27" y="-3.81" smashed="yes">
+<attribute name="NAME" x="-2.07" y="-6.21" size="1.27" layer="25" rot="R90"/>
+<attribute name="POPULARITY" value="15" x="-1.27" y="-3.81" size="1.778" layer="27" display="off"/>
+<attribute name="VALUE" x="-1.27" y="-3.81" size="0.0254" layer="27"/>
 </element>
 </elements>
@@
 <wire x1="13.2334" y1="21.41973125" x2="9.25313125" y2="25.4" width="0.508" layer="2"/>
 <wire x1="9.25313125" y1="25.4" x2="5.08" y2="25.4" width="0.508" layer="2"/>
+<contactref element="U1" pad="3"/>
+<wire x1="1.66" y1="-3.81" x2="12.437" y2="3.683" width="0" layer="19" extent="1-16"/>
 </signal>
 <signal name="+3V3">
@@
 <wire x1="11.557" y1="23.622" x2="11.049" y2="23.114" width="0.254" layer="16"/>
 <wire x1="11.049" y1="23.114" x2="11.049" y2="19.32" width="0.254" layer="16"/>
-</signal>
-<signal name="CS0_0">
+<contactref element="U1" pad="6"/>
+<contactref element="U1" pad="5"/>
+<wire x1="5.96" y1="-4.81" x2="8.137" y2="2.683" width="0" layer="19" extent="1-16"/>
+<wire x1="1.66" y1="-4.81" x2="5.96" y2="-4.81" width="0" layer="19" extent="1-1"/>
+</signal>
+<signal name="CS0_COMP1">
 <contactref element="U6" pad="2"/>
 <wire x1="12.31" y1="20.82" x2="14.097" y2="20.82" width="0.254" layer="16"/>
@@
 <via x="14.097" y="21.59" extent="1-16" drill="0.508"/>
 </signal>
-<signal name="CS1_0">
+<signal name="CS1_COMP1">
 <contactref element="U8" pad="2"/>
 <wire x1="12.437" y1="4.183" x2="13.454" y2="4.183" width="0.254" layer="16"/>
@@
 <via x="14.859" y="5.588" extent="1-16" drill="0.508"/>
 </signal>
-<signal name="CS2_0">
+<signal name="CS2_COMP1">
 <contactref element="U7" pad="2"/>
 <wire x1="12.31" y1="11.93" x2="14.47" y2="11.93" width="0.254" layer="16"/>
@@
 <contactref element="U9" pad="7"/>
 </signal>
-<signal name="CS0_1">
+<signal name="CS0_COMP2">
 <contactref element="U6" pad="9"/>
 <wire x1="8.01" y1="20.82" x2="6.088" y2="20.82" width="0.254" layer="16"/>
@@
 <via x="5.842" y="20.574" extent="1-16" drill="0.508"/>
 </signal>
-<signal name="CS1_1">
+<signal name="CS1_COMP2">
 <contactref element="U8" pad="9"/>
 <wire x1="8.137" y1="4.183" x2="6.215" y2="4.183" width="0.254" layer="16"/>
@@
 <via x="6.096" y="4.064" extent="1-16" drill="0.508"/>
 </signal>
-<signal name="CS2_1">
+<signal name="CS2_COMP2">
 <contactref element="U7" pad="9"/>
 <wire x1="8.01" y1="11.93" x2="5.58" y2="11.93" width="0.254" layer="16"/>
@@
 <wire x1="12.31" y1="12.43" x2="12.31" y2="13.335" width="0.254" layer="16"/>
 <wire x1="12.31" y1="13.335" x2="12.437" y2="13.462" width="0.254" layer="16"/>
+<contactref element="U1" pad="1"/>
+<wire x1="1.66" y1="-2.81" x2="12.437" y2="4.683" width="0" layer="19" extent="1-16"/>
 </signal>
 <signal name="MUX1">
@@
 <wire x1="3.699" y1="21.701" x2="3.588" y2="21.59" width="0.254" layer="16"/>
 <wire x1="3.588" y1="21.59" x2="3.556" y2="21.59" width="0.254" layer="16"/>
-</signal>
-<signal name="CS0_2">
+<contactref element="U1" pad="10"/>
+<wire x1="5.96" y1="-2.81" x2="8.137" y2="4.683" width="0" layer="19" extent="1-16"/>
+</signal>
+<signal name="CS0_COMP3">
 <contactref element="U6" pad="4"/>
 <wire x1="12.31" y1="19.82" x2="13.327" y2="19.82" width="0.254" layer="16"/>
@@
 <wire x1="13.327" y1="19.82" x2="14.224" y2="18.923" width="0.254" layer="16"/>
 </signal>
-<signal name="CS1_2">
+<signal name="CS1_COMP3">
 <contactref element="U8" pad="4"/>
 <wire x1="12.437" y1="3.183" x2="13.835" y2="3.183" width="0.254" layer="16"/>
@@
 <wire x1="8.763" y1="15.621" x2="10.16" y2="14.224" width="0.254" layer="16"/>
 </signal>
-<signal name="CS2_2">
+<signal name="CS2_COMP3">
 <contactref element="U7" pad="4"/>
 <wire x1="12.31" y1="10.93" x2="13.962" y2="10.93" width="0.254" layer="16"/>
@@
 <contactref element="U9" pad="11"/>
 </signal>
-<signal name="CS0_3">
+<signal name="CS0_COMP4">
 <contactref element="U6" pad="7"/>
 <wire x1="8.01" y1="19.82" x2="6.612" y2="19.82" width="0.254" layer="16"/>
@@
 <via x="6.223" y="19.431" extent="1-16" drill="0.508"/>
 </signal>
-<signal name="CS1_3">
+<signal name="CS1_COMP4">
 <contactref element="U8" pad="7"/>
 <wire x1="8.137" y1="3.183" x2="8.129" y2="3.175" width="0.254" layer="16"/>
@@
 <wire x1="8.129" y1="3.175" x2="6.223" y2="3.175" width="0.254" layer="16"/>
 </signal>
-<signal name="CS2_3">
+<signal name="CS2_COMP4">
 <contactref element="U7" pad="7"/>
 <wire x1="8.01" y1="10.93" x2="6.104" y2="10.93" width="0.254" layer="16"/>
@@
 <contactref element="SCK" pad="1"/>
 </signal>
+<signal name="CS_PAN1">
+<contactref element="U1" pad="2"/>
+</signal>
+<signal name="CS_PAN2">
+<contactref element="U1" pad="9"/>
+</signal>
+<signal name="CS_PAN3">
+<contactref element="U1" pad="4"/>
+</signal>
+<signal name="CS0_PAN4">
+<contactref element="U1" pad="7"/>
+</signal>
+<signal name="CS">
+<contactref element="U1" pad="8"/>
+<contactref element="CS" pad="1"/>
+<wire x1="-1.27" y1="-3.81" x2="5.96" y2="-3.81" width="0" layer="19" extent="1-1"/>
+</signal>
 </signals>

Commit message: v2 of board finished
Parts:
- moved CS 10.9 mm to (8.89, 0.00), flipped to the bottom, turned to 270 degrees
- moved GND 6.35 mm to (14.0, 0.00), turned to 270 degrees
- moved U1 6.35 mm to (10.2, -3.81), flipped to the bottom
Routing:
- net MUX1: track 28.8 -> 43.3 mm
- net MUX0: track 30.5 -> 44.4 mm
- net +3V3: track 39.1 -> 51.2 mm
- net CS: track 0.00 -> 4.68 mm
- net CS_PAN3: track 0.00 -> 3.32 mm, vias 0 -> 1
- net CS_PAN1: track 0.00 -> 2.58 mm, vias 0 -> 1
- net DGND: track 68.8 -> 71.0 mm
- net CS_PAN2: track 0.00 -> 2.10 mm, vias 0 -> 1
- net CS0_PAN4: track 0.00 -> 2.10 mm, vias 0 -> 1
