File: combined-v2.sch (EAGLE design)
At the start: 0 parts

Commit message: v2 of board finished
Parts:
- added 100POT1_COMP1, 100POT1_COMP2, 100POT1_COMP3, 100POT1_COMP5: MCP42100-I/P, MCP42100-I_P:MCP42100-I/P
- added 10KPOT1_PAN1, 10KPOT1_PAN2, 10KPOT1_PAN3, 10KPOT1_PAN4, 10POT1_COMP1, 10POT1_COMP2, 10POT1_COMP3, 10POT1_COMP5, 10POT2_COMP1, 10POT2_COMP2, 10POT2_COMP3, 10POT2_COMP5: MCP4131-503E/SN, MCP4131-503E_SN:MCP4131-503E/SN
- added 200POT1_COMP1, 200POT1_COMP2, 200POT1_COMP3, 200POT1_COMP5, 200POT2_COMP1, 200POT2_COMP2, 200POT2_COMP3, 200POT2_COMP5: MAX5419LETA+, MAX5419LETA_:MAX5419LETA+
- added 3V3_D1, 9VDD1, BCK_ADC1, CE_EQ1, CE_EQ2, CLK_ADC1, CS3, CS4, CS5, CS6, DOUT_ADC1, GND4, GND6, LRCK_ADC1, MUX2, MUX3, PAD1, PAD10, PAD11, PAD12, PAD13, PAD14, PAD15, PAD16, PAD2, PAD3, PAD4, PAD5, PAD6, PAD7, PAD8, PAD9, SCK1, SCL1, SCL2, SDA1, SDA2, SDI/O1: (no value), wirepad:SMD2
- added C10, C105, C106, C109, C11, C110, C111, C112, C115, C116, C14, C15, C16, C17, C20, C21: 0.01uF, rcl:C-USC0402
- added C103, C104, C117, C118, C22, C23, C7, C9: 0.047uF, rcl:C-USC0402
- added C107, C108, C113, C114, C12, C13, C18, C19: 0.068uF, rcl:C-USC0402
- added C119, C120, C121, C122, C123, C124, C125, C126, C127, C129, C130, C131, C132, C134, C2, C24, C25, C26, C27, C28, C29, C30, C31, C32, C34, C35, C36, C37, C39, C5, C6, C69, C71, C77, C78, C79, C8, C80, C81, C82, C83, C84: 10uF, rcl:C-USC0402
- added C128, C133, C33, C38, C68, C70, C73: 0.1uF, rcl:C-USC0402
- added C3, C4: 0.1u, rcl:C-USC0402
- added C42, C45, C48, C54: 680p, rcl:C-USC0402
- added C43, C46, C49, C55: 10u, rcl:C-USC0402
- added C44, C47, C50, C56: 1.5u, rcl:C-USC0402
- added C72, C74: 1uF, rcl:C-USC0402
- added C75, C76: 15pF, rcl:C-USC0402
- added D16, D17, D18, D19, D20, D21, D22, D23, D24, D25, D26, D27, D28, D29, D30, D31, D32, D33, D34, D35, D36, D37, D38, D39, D40, D41, D42, D43, D44, D45, D46, D47, D48, D60, D61, D62, D63, D64, D65, D66, D67, D68, D69, D70: 1N4148W-TP, 1N4148W-TP:1N4148W-TP
- added D2, D3, D4, D5: 1N4148W-TPSOD123-L, 1N4148W-TP:1N4148W-TPSOD123-L
- added GND1, GND2, GND3, GND5, GNDL1, GNDR1, IN_COMP1, IN_COMP2, IN_COMP3, IN_COMP5, OUTL_MIX1, OUTR_MIX1: (no value), wirepad:SMD5
- added IC2: PCM1865DBT, PCM1865DBT:PCM1865DBT
- added OPAMP1_COMP1, OPAMP1_COMP2, OPAMP1_COMP3, OPAMP1_COMP5, OPAMP1_MIX1, OPAMP1_PAN1, OPAMP1_PAN2, OPAMP1_PAN3, OPAMP1_PAN4, OPAMP2_COMP1, OPAMP2_COMP2, OPAMP2_COMP3, OPAMP2_COMP5, OPAMP3_COMP1, OPAMP3_COMP2, OPAMP3_COMP3, OPAMP3_COMP5, OPAMP4_COMP1, OPAMP4_COMP2, OPAMP4_COMP3, OPAMP4_COMP5, U2: LM4562MAX/NOPB, LM4562MAX_NOPB:LM4562MAX/NOPB
- added R10, R11, R13, R16, R17, R18, R20, R31, R33, R35, R36, R37, R38, R39, R40, R43, R46, R48, R50, R51, R52, R53, R54, R55, R58, R69, R7, R70, R71, R73, R83, R84, R85, R87: 5k, rcl:R-US_R0402
- added R100, R102, R103, R104, R107, R108, R109, R111, R112, R113, R117, R118, R120, R121, R122, R125, R126, R127, R129, R130, R149, R153, R154, R156, R157, R158, R161, R162, R163, R165, R166, R63, R67, R75, R77, R78, R79, R89, R90, R91, R93, R94, R95, R99: 100k, rcl:R-US_R0402
- added R101, R105, R110, R119, R12, R123, R128, R14, R155, R159, R164, R19, R21, R32, R34, R41, R42, R47, R49, R56, R57, R72, R74, R76, R80, R86, R88, R92: 10k, rcl:R-US_R0402
- added R106, R124, R160, R81: 20k, rcl:R-US_R0402
- added R114, R116, R150, R152, R64, R66, R96, R98: 470k, rcl:R-US_R0402
- added R115, R151, R45, R5, R60, R65, R8, R9, R97: 1k, rcl:R-US_R0402
- added R15, R6, R68, R82: 1M, rcl:R-US_R0402
- added R22: 1.7k, rcl:R-US_R0402
- added R44, R59: 50k, rcl:R-US_R0402
- added U$1, U$3: LC75281E, LC75281E:LC75281E
- added U11, U3, U4, U5: TMUX1204DGSR, TMUX1204DGSR:TMUX1204DGSR
- added Y2: CM7V-T1A-32.768KHZ-12.5PF-100PPM-TB-QC, CM7V-T1A-32.768KHZ-12.5PF-100PPM-TB-QC:CM7V-T1A-32.768KHZ-12.5PF-100PPM-TB-QC
Connections:
- new net +3V3: 3V3_D1.P, U11.EN, U11.VDD, U3.EN, U3.VDD, U4.EN, U4.VDD, U5.EN, U5.VDD
- new net 3V3A: C70.1, C71.1, IC2.AVDD, U2.NEG_A, U2.OUT_A
- new net 3V3D: C68.1, C69.1, IC2.DVDD, IC2.IOVDD
- new net BCK_ADC: BCK_ADC1.P, IC2.BCK
- new net CLK_ADC: CLK_ADC1.P, IC2.SCKI
- new net CS: CS6.P, U11.D
- new net CS0: CS3.P, U3.D
- new net CS0_COMP1: 100POT1_COMP1.~CS, U3.S1
- new net CS0_COMP2: 100POT1_COMP3.~CS, U3.S2
- new net CS0_COMP3: 100POT1_COMP2.~CS, U3.S3
- new net CS0_COMP4: 100POT1_COMP5.~CS, U3.S4
- new net CS1: CS4.P, U5.D
- new net CS1_COMP1: 10POT1_COMP1.!CS, U5.S1
- new net CS1_COMP2: 10POT1_COMP3.!CS, U5.S2
- new net CS1_COMP3: 10POT1_COMP2.!CS, U5.S3
- new net CS1_COMP4: 10POT1_COMP5.!CS, U5.S4
- new net CS2: CS5.P, U4.D
- new net CS2_COMP1: 10POT2_COMP1.!CS, U4.S1
- new net CS2_COMP2: 10POT2_COMP3.!CS, U4.S2
- new net CS2_COMP3: 10POT2_COMP2.!CS, U4.S3
- new net CS2_COMP4: 10POT2_COMP5.!CS, U4.S4
- new net CS_PAN1: 10KPOT1_PAN1.!CS, U11.S1
- new net CS_PAN2: 10KPOT1_PAN3.!CS, U11.S2
- new net CS_PAN3: 10KPOT1_PAN2.!CS, U11.S3
- new net CS_PAN4: 10KPOT1_PAN4.!CS, U11.S4
- new net DOUT_ADC: DOUT_ADC1.P, IC2.DOUT
- new net EQ1_CE1: CE_EQ1.P, U$1.CE
- new net EQ2_CE3: CE_EQ2.P, U$3.CE
- new net GND: 100POT1_COMP1.VSS, 100POT1_COMP2.VSS, 100POT1_COMP3.VSS, 100POT1_COMP5.VSS, 10KPOT1_PAN1.VSS, 10KPOT1_PAN2.VSS, 10KPOT1_PAN3.VSS, 10KPOT1_PAN4.VSS, 10POT1_COMP1.VSS, 10POT1_COMP2.VSS, 10POT1_COMP3.VSS, 10POT1_COMP5.VSS, 10POT2_COMP1.VSS, 10POT2_COMP2.VSS, 10POT2_COMP3.VSS, 10POT2_COMP5.VSS, 200POT1_COMP1.EPAD, 200POT1_COMP1.GND, 200POT1_COMP2.EPAD, 200POT1_COMP2.GND, 200POT1_COMP3.EPAD, 200POT1_COMP3.GND, 200POT1_COMP5.EPAD, 200POT1_COMP5.GND, 200POT2_COMP1.A0, 200POT2_COMP1.EPAD, 200POT2_COMP1.GND, 200POT2_COMP2.A0, 200POT2_COMP2.EPAD, 200POT2_COMP2.GND, 200POT2_COMP3.A0, 200POT2_COMP3.EPAD, 200POT2_COMP3.GND, 200POT2_COMP5.A0, 200POT2_COMP5.EPAD, 200POT2_COMP5.GND, C123.2, C134.2, C28.2, C39.2, C68.2, C69.2, C70.2, C71.2, C72.2, C73.2, C74.2, C75.2, C76.2, GND1.P, GND2.P, GND3.P, GND4.P, GND5.P, GND6.P, GNDL1.P, GNDR1.P, IC2.AGND, IC2.DGND, IC2.MS/AD, OPAMP1_COMP1.V-, OPAMP1_COMP2.V-, OPAMP1_COMP3.V-, OPAMP1_COMP5.V-, OPAMP1_MIX1.V-, OPAMP1_PAN1.V-, OPAMP1_PAN2.V-, OPAMP1_PAN3.V-, OPAMP1_PAN4.V-, OPAMP2_COMP1.V-, OPAMP2_COMP2.V-, OPAMP2_COMP3.V-, OPAMP2_COMP5.V-, OPAMP3_COMP1.V-, OPAMP3_COMP2.V-, OPAMP3_COMP3.V-, OPAMP3_COMP5.V-, OPAMP4_COMP1.V-, OPAMP4_COMP2.V-, OPAMP4_COMP3.V-, OPAMP4_COMP5.V-, R5.1, R9.1, U$1.TEST, U$1.V_SS, U$3.TEST, U$3.V_SS, U11.GND, U2.V-, U3.GND, U4.GND, U5.GND
- new net H1_COMP1: 200POT1_COMP1.H, 200POT2_COMP1.H, C44.1, OPAMP1_COMP1.NEG_B, R66.1
- new net H1_COMP2: 200POT1_COMP3.H, 200POT2_COMP3.H, C50.1, OPAMP1_COMP3.NEG_B, R116.1
- new net H1_COMP3: 200POT1_COMP2.H, 200POT2_COMP2.H, C47.1, OPAMP1_COMP2.NEG_B, R98.1
- new net H1_COMP4: 200POT1_COMP5.H, 200POT2_COMP5.H, C56.1, OPAMP1_COMP5.NEG_B, R152.1
- new net IN_COMP1: C43.2, IN_COMP1.P
- new net IN_COMP2: C49.2, IN_COMP3.P
- new net IN_COMP3: C46.2, IN_COMP2.P
- new net IN_COMP4: C55.2, IN_COMP5.P
- new net L1_COMP1: 200POT1_COMP1.L, 200POT1_COMP1.W, D19.C
- new net L1_COMP2: 200POT1_COMP3.L, 200POT1_COMP3.W, D41.C
- new net L1_COMP3: 200POT1_COMP2.L, 200POT1_COMP2.W, D30.C
- new net L1_COMP4: 200POT1_COMP5.L, 200POT1_COMP5.W, D63.C
- new net L2_COMP1: 200POT2_COMP1.L, 200POT2_COMP1.W, R94.2
- new net L2_COMP2: 200POT2_COMP3.L, 200POT2_COMP3.W, R130.2
- new net L2_COMP3: 200POT2_COMP2.L, 200POT2_COMP2.W, R112.2
- new net L2_COMP4: 200POT2_COMP5.L, 200POT2_COMP5.W, R166.2
- new net LRCK_ADC: IC2.LRCK, LRCK_ADC1.P
- new net MUX0: MUX2.P, U11.A0, U3.A0, U4.A0, U5.A0
- new net MUX1: MUX3.P, U11.A1, U3.A1, U4.A1, U5.A1
- new net N$10: R32.2, R34.2, R41.2, R42.2, R43.1
- new net N$100: D64.A, D65.C
- new net N$101: C55.1, R163.2
- new net N$102: D68.A, D69.C
- new net N$103: D67.A, D68.C
- new net N$11: R31.2, R38.1, R42.1
- new net N$114: C72.1, IC2.VREF
- new net N$115: C73.1, C74.1, IC2.LDO
- new net N$116: C75.1, IC2.XO, Y2.2
- new net N$117: C76.1, IC2.XI, Y2.1
- new net N$118: C84.2, IC2.VINL2/VIN1M
- new net N$119: C77.2, IC2.VINR2/VIN2M
- new net N$12: R33.2, R37.1, R41.1
- new net N$120: C103.1, U$3.LLC1
- new net N$121: C105.1, U$3.LLMC1
- new net N$122: C106.1, U$3.LLMC4
- new net N$123: C81.2, IC2.VINL1/VIN1P
- new net N$124: C107.1, U$3.LHMC1
- new net N$125: C78.2, IC2.VINR1/VIN2P
- new net N$126: C79.2, IC2.VINL3/VIN4P
- new net N$127: C83.2, IC2.VINR4/VIN3M
- new net N$128: C80.2, IC2.VINL4/VIN4M
- new net N$13: C13.1, U$1.LHMC4
- new net N$131: C108.1, U$3.LHMC4
- new net N$132: C109.1, U$3.LHC1
- new net N$135: C110.1, U$3.LHC4
- new net N$136: C111.1, U$3.RHC4
- new net N$137: C112.1, U$3.RHC1
- new net N$138: C113.1, U$3.RHMC4
- new net N$139: C114.1, U$3.RHMC1
- new net N$14: C14.1, U$1.LHC1
- new net N$140: C115.1, U$3.RLMC4
- new net N$141: C116.1, U$3.RLMC1
- new net N$142: C117.1, U$3.RLC4
- new net N$143: C118.1, U$3.RLC1
- new net N$144: C103.2, U$3.LLC2
- new net N$145: C104.2, C119.2, U$3.LLC3
- new net N$146: C119.1, U$3.LLC5
- new net N$147: C120.1, U$3.LLMC5
- new net N$148: C121.1, U$3.LHMC5
- new net N$149: C122.1, U$3.LHC5
- new net N$15: C15.1, U$1.LHC4
- new net N$150: C123.1, C134.1, U$3.V_REF
- new net N$151: C124.1, U$3.RHC5
- new net N$152: C125.1, U$3.RHMC5
- new net N$153: C126.1, U$3.RLMC5
- new net N$154: C127.1, U$3.RLC5
- new net N$155: C128.1, U$3.ROUT
- new net N$156: C129.1, U$3.RBOOS2
- new net N$157: C130.1, U$3.RCUT2
- new net N$158: C131.1, U$3.LCUT1
- new net N$159: C132.1, U$3.LBOOS1
- new net N$16: C16.1, U$1.RHC4
- new net N$160: C133.1, U$3.LOUT
- new net N$161: C105.2, U$3.LLMC2
- new net N$162: C106.2, C120.2, U$3.LLMC3
- new net N$163: C107.2, U$3.LHMC2
- new net N$164: C108.2, C121.2, U$3.LHMC3
- new net N$165: C109.2, U$3.LHC2
- new net N$166: C110.2, C122.2, U$3.LHC3
- new net N$167: C111.2, C124.2, U$3.RHC3
- new net N$168: C112.2, U$3.RHC2
- new net N$169: C113.2, C125.2, U$3.RHMC3
- new net N$17: C17.1, U$1.RHC1
- new net N$170: C114.2, U$3.RHMC2
- new net N$171: C115.2, C126.2, U$3.RLMC3
- new net N$172: C116.2, U$3.RLMC2
- new net N$173: C117.2, C127.2, U$3.RLC3
- new net N$174: C118.2, U$3.RLC2
- new net N$175: C129.2, U$3.RBOOS1
- new net N$176: C130.2, U$3.RCUT1
- new net N$177: C131.2, U$3.LCUT2
- new net N$178: C132.2, U$3.LBOOS2
- new net N$179: C104.1, U$3.LLC4
- new net N$18: R34.1, R36.1, R40.2
- new net N$183: C82.2, IC2.VINR3/VIN3P
- new net N$19: C4.1, R60.2
- new net N$2: C2.2, R10.2, R6.2, R7.2
- new net N$20: R47.1, R50.2, R54.2
- new net N$21: R47.2, R49.2, R56.2, R57.2, R58.1
- new net N$211: C42.1, D17.A, D18.C, D25.A, R65.1, R89.2
- new net N$212: C48.1, D39.A, D40.C, D47.A, R115.1, R125.2
- new net N$213: C45.1, D28.A, D29.C, D36.A, R107.2, R97.1
- new net N$214: C54.1, D61.A, D62.C, D69.A, R151.1, R161.2
- new net N$22: R46.2, R53.1, R57.1
- new net N$23: R48.2, R52.1, R56.1
- new net N$24: R49.1, R51.1, R55.2
- new net N$25: C18.1, U$1.RHMC4
- new net N$26: C6.2, R68.2, R69.2, R70.2
- new net N$27: C19.1, U$1.RHMC1
- new net N$28: C8.2, R82.2, R83.2, R84.2
- new net N$29: C20.1, U$1.RLMC4
- new net N$3: C5.2, R15.2, R16.2, R17.2
- new net N$30: C21.1, U$1.RLMC1
- new net N$31: C22.1, U$1.RLC4
- new net N$32: C23.1, U$1.RLC1
- new net N$33: C7.2, U$1.LLC2
- new net N$34: C24.2, C9.2, U$1.LLC3
- new net N$35: C24.1, U$1.LLC5
- new net N$36: C25.1, U$1.LLMC5
- new net N$37: C26.1, U$1.LHMC5
- new net N$38: C27.1, U$1.LHC5
- new net N$39: C28.1, C39.1, U$1.V_REF
- new net N$4: C7.1, U$1.LLC1
- new net N$40: C29.1, U$1.RHC5
- new net N$41: C30.1, U$1.RHMC5
- new net N$42: C31.1, U$1.RLMC5
- new net N$43: C32.1, U$1.RLC5
- new net N$44: C33.1, U$1.ROUT
- new net N$45: C34.1, U$1.RBOOS2
- new net N$46: C35.1, U$1.RCUT2
- new net N$47: C36.1, U$1.LCUT1
- new net N$48: C37.1, U$1.LBOOS1
- new net N$49: C38.1, U$1.LOUT
- new net N$5: C10.1, U$1.LLMC1
- new net N$50: C10.2, U$1.LLMC2
- new net N$51: C11.2, C25.2, U$1.LLMC3
- new net N$52: C12.2, U$1.LHMC2
- new net N$53: C13.2, C26.2, U$1.LHMC3
- new net N$54: C14.2, U$1.LHC2
- new net N$55: C15.2, C27.2, U$1.LHC3
- new net N$56: C16.2, C29.2, U$1.RHC3
- new net N$57: C17.2, U$1.RHC2
- new net N$58: C18.2, C30.2, U$1.RHMC3
- new net N$59: C19.2, U$1.RHMC2
- new net N$6: C11.1, U$1.LLMC4
- new net N$60: C20.2, C31.2, U$1.RLMC3
- new net N$61: C21.2, U$1.RLMC2
- new net N$62: C22.2, C32.2, U$1.RLC3
- new net N$63: C23.2, U$1.RLC2
- new net N$64: C34.2, U$1.RBOOS1
- new net N$65: C35.2, U$1.RCUT1
- new net N$66: C36.2, U$1.LCUT2
- new net N$67: C37.2, U$1.LBOOS2
- new net N$68: C9.1, U$1.LLC4
- new net N$7: C12.1, U$1.LHMC1
- new net N$70: R22.2, R9.2, U2.POS_A
- new net N$71: R5.2, R8.2, U2.POS_B
- new net N$74: D16.A, D17.C
- new net N$75: D21.A, D22.C
- new net N$76: D20.A, D21.C
- new net N$77: C43.1, R91.2
- new net N$78: D24.A, D25.C
- new net N$79: D23.A, D24.C
- new net N$8: C3.1, R45.2
- new net N$80: D27.A, D28.C
- new net N$81: D32.A, D33.C
- new net N$82: D31.A, D32.C
- new net N$83: C46.1, R109.2
- new net N$84: D35.A, D36.C
- new net N$85: D34.A, D35.C
- new net N$86: D38.A, D39.C
- new net N$87: D43.A, D44.C
- new net N$88: D42.A, D43.C
- new net N$89: C49.1, R127.2
- new net N$9: R32.1, R35.2, R39.2
- new net N$90: D46.A, D47.C
- new net N$91: D45.A, D46.C
- new net N$98: D60.A, D61.C
- new net N$99: D65.A, D66.C
- new net NEG_A1_COMP1: C42.2, D16.C, D18.A, OPAMP1_COMP1.NEG_A, R63.2
- new net NEG_A1_COMP2: C48.2, D38.C, D40.A, OPAMP1_COMP3.NEG_A, R113.2
- new net NEG_A1_COMP3: C45.2, D27.C, D29.A, OPAMP1_COMP2.NEG_A, R95.2
- new net NEG_A1_COMP4: C54.2, D60.C, D62.A, OPAMP1_COMP5.NEG_A, R149.2
- new net NEG_A2_COMP1: OPAMP2_COMP1.NEG_A, R67.2, R75.1
- new net NEG_A2_COMP2: OPAMP2_COMP3.NEG_A, R117.2, R118.1
- new net NEG_A2_COMP3: OPAMP2_COMP2.NEG_A, R100.1, R99.2
- new net NEG_A2_COMP4: OPAMP2_COMP5.NEG_A, R153.2, R154.1
- new net NEG_A3_COMP1: OPAMP3_COMP1.NEG_A, R77.1, R78.2
- new net NEG_A3_COMP2: OPAMP3_COMP3.NEG_A, R120.1, R121.2
- new net NEG_A3_COMP3: OPAMP3_COMP2.NEG_A, R102.1, R103.2
- new net NEG_A3_COMP4: OPAMP3_COMP5.NEG_A, R156.1, R157.2
- new net NEG_A4_COMP1: OPAMP4_COMP1.NEG_A, R79.2, R80.2
- new net NEG_A4_COMP2: OPAMP4_COMP3.NEG_A, R122.2, R123.2
- new net NEG_A4_COMP3: OPAMP4_COMP2.NEG_A, R104.2, R105.2
- new net NEG_A4_COMP4: OPAMP4_COMP5.NEG_A, R158.2, R159.2
- new net NEG_A_MIX: OPAMP1_MIX1.NEG_A, R43.2, R44.1
- new net NEG_A_PAN1: OPAMP1_PAN1.NEG_A, R71.1, R74.1
- new net NEG_A_PAN2: OPAMP1_PAN3.NEG_A, R85.1, R88.1
- new net NEG_A_PAN3: OPAMP1_PAN2.NEG_A, R11.1, R14.1
- new net NEG_A_PAN4: OPAMP1_PAN4.NEG_A, R18.1, R21.1
- new net NEG_B2_COMP1: OPAMP2_COMP1.NEG_B, OPAMP2_COMP1.OUT_B, R93.2
- new net NEG_B2_COMP2: OPAMP2_COMP3.NEG_B, OPAMP2_COMP3.OUT_B, R129.2
- new net NEG_B2_COMP3: OPAMP2_COMP2.NEG_B, OPAMP2_COMP2.OUT_B, R111.2
- new net NEG_B2_COMP4: OPAMP2_COMP5.NEG_B, OPAMP2_COMP5.OUT_B, R165.2
- new net NEG_B3_COMP1: OPAMP3_COMP1.NEG_B, R89.1, R90.2
- new net NEG_B3_COMP2: OPAMP3_COMP3.NEG_B, R125.1, R126.2
- new net NEG_B3_COMP3: OPAMP3_COMP2.NEG_B, R107.1, R108.2
- new net NEG_B3_COMP4: OPAMP3_COMP5.NEG_B, R161.1, R162.2
- new net NEG_B4_COMP1: 100POT1_COMP1.PB1, OPAMP4_COMP1.NEG_B, R81.2
- new net NEG_B4_COMP2: 100POT1_COMP3.PB1, OPAMP4_COMP3.NEG_B, R124.2
- new net NEG_B4_COMP3: 100POT1_COMP2.PB1, OPAMP4_COMP2.NEG_B, R106.2
- new net NEG_B4_COMP4: 100POT1_COMP5.PB1, OPAMP4_COMP5.NEG_B, R160.2
- new net NEG_B_MIX: OPAMP1_MIX1.NEG_B, R58.2, R59.1
- new net NEG_B_PAN1: OPAMP1_PAN1.NEG_B, R72.2, R73.2
- new net NEG_B_PAN2: OPAMP1_PAN3.NEG_B, R86.2, R87.2
- new net NEG_B_PAN3: OPAMP1_PAN2.NEG_B, R12.2, R13.2
- new net NEG_B_PAN4: OPAMP1_PAN4.NEG_B, R19.2, R20.2
- new net OUT1_EQ1: C33.2, C6.1, PAD16.P
- new net OUT1_EQ2: C128.2, C5.1, PAD14.P
- new net OUT2_EQ1: C38.2, C8.1, PAD15.P
- new net OUT2_EQ2: C133.2, C2.1, PAD13.P
- new net OUTL_MIX1: C3.2, OUTL_MIX1.P
- new net OUTL_PAN1: C79.1, OPAMP1_PAN1.OUT_A, PAD3.P, R55.1, R74.2
- new net OUTL_PAN2: C80.1, OPAMP1_PAN3.OUT_A, PAD5.P, R31.1, R88.2
- new net OUTL_PAN3: C78.1, OPAMP1_PAN2.OUT_A, PAD1.P, R14.2, R46.1
- new net OUTL_PAN4: C84.1, OPAMP1_PAN4.OUT_A, PAD7.P, R21.2, R40.1
- new net OUTR_MIX1: C4.2, OUTR_MIX1.P
- new net OUTR_PAN1: C82.1, OPAMP1_PAN1.OUT_B, PAD6.P, R33.1, R72.1
- new net OUTR_PAN2: C83.1, OPAMP1_PAN3.OUT_B, PAD4.P, R54.1, R86.1
- new net OUTR_PAN3: C81.1, OPAMP1_PAN2.OUT_B, PAD8.P, R12.1, R39.1
- new net OUTR_PAN4: C77.1, OPAMP1_PAN4.OUT_B, PAD2.P, R19.1, R48.1
- new net OUT_A1_COMP1: OPAMP1_COMP1.OUT_A, R65.2
- new net OUT_A1_COMP2: OPAMP1_COMP3.OUT_A, R115.2
- new net OUT_A1_COMP3: OPAMP1_COMP2.OUT_A, R97.2
- new net OUT_A1_COMP4: OPAMP1_COMP5.OUT_A, R151.2
- new net OUT_A2_COMP1: 100POT1_COMP1.PB0, OPAMP2_COMP1.OUT_A, R75.2
- new net OUT_A2_COMP2: 100POT1_COMP3.PB0, OPAMP2_COMP3.OUT_A, R118.2
- new net OUT_A2_COMP3: 100POT1_COMP2.PB0, OPAMP2_COMP2.OUT_A, R100.2
- new net OUT_A2_COMP4: 100POT1_COMP5.PB0, OPAMP2_COMP5.OUT_A, R154.2
- new net OUT_A3_COMP1: D26.A, OPAMP3_COMP1.OUT_A
- new net OUT_A3_COMP2: D48.A, OPAMP3_COMP3.OUT_A
- new net OUT_A3_COMP3: D37.A, OPAMP3_COMP2.OUT_A
- new net OUT_A3_COMP4: D70.A, OPAMP3_COMP5.OUT_A
- new net OUT_A4_COMP1: OPAMP4_COMP1.OUT_A, OPAMP4_COMP1.POS_B, R78.1, R79.1
- new net OUT_A4_COMP2: OPAMP4_COMP3.OUT_A, OPAMP4_COMP3.POS_B, R121.1, R122.1
- new net OUT_A4_COMP3: OPAMP4_COMP2.OUT_A, OPAMP4_COMP2.POS_B, R103.1, R104.1
- new net OUT_A4_COMP4: OPAMP4_COMP5.OUT_A, OPAMP4_COMP5.POS_B, R157.1, R158.1
- new net OUT_A_MIX: OPAMP1_MIX1.OUT_A, R44.2, R45.1
- new net OUT_B1_COMP1: D19.A, OPAMP1_COMP1.OUT_B
- new net OUT_B1_COMP2: D41.A, OPAMP1_COMP3.OUT_B
- new net OUT_B1_COMP3: D30.A, OPAMP1_COMP2.OUT_B
- new net OUT_B1_COMP4: D63.A, OPAMP1_COMP5.OUT_B
- new net OUT_B3_COMP1: D20.C, OPAMP3_COMP1.OUT_B, R90.1
- new net OUT_B3_COMP2: D42.C, OPAMP3_COMP3.OUT_B, R126.1
- new net OUT_B3_COMP3: D31.C, OPAMP3_COMP2.OUT_B, R108.1
- new net OUT_B3_COMP4: D64.C, OPAMP3_COMP5.OUT_B, R162.1
- new net OUT_B_MIX: OPAMP1_MIX1.OUT_B, R59.2, R60.1
- new net OUT_COMP1: 100POT1_COMP1.PA1, 100POT1_COMP1.PW1, OPAMP4_COMP1.OUT_B, PAD10.P, U$1.LIN
- new net OUT_COMP2: 100POT1_COMP3.PA1, 100POT1_COMP3.PW1, OPAMP4_COMP3.OUT_B, PAD9.P, U$1.RIN
- new net OUT_COMP3: 100POT1_COMP2.PA1, 100POT1_COMP2.PW1, OPAMP4_COMP2.OUT_B, PAD12.P, U$3.LIN
- new net OUT_COMP4: 100POT1_COMP5.PA1, 100POT1_COMP5.PW1, OPAMP4_COMP5.OUT_B, PAD11.P, U$3.RIN
- new net P0A1_COMP1: 10POT1_COMP1.P0A, R76.2
- new net P0A1_COMP2: 10POT1_COMP3.P0A, R119.2
- new net P0A1_COMP3: 10POT1_COMP2.P0A, R101.2
- new net P0A1_COMP4: 10POT1_COMP5.P0A, R155.2
- new net P0A2_COMP1: 10POT2_COMP1.P0A, R92.1
- new net P0A2_COMP2: 10POT2_COMP3.P0A, R128.1
- new net P0A2_COMP3: 10POT2_COMP2.P0A, R110.1
- new net P0A2_COMP4: 10POT2_COMP5.P0A, R164.1
- new net P0A_PAN1: 10KPOT1_PAN1.P0A, R70.1, R71.2
- new net P0A_PAN2: 10KPOT1_PAN3.P0A, R84.1, R85.2
- new net P0A_PAN3: 10KPOT1_PAN2.P0A, R10.1, R11.2
- new net P0A_PAN4: 10KPOT1_PAN4.P0A, R17.1, R18.2
- new net P0B_PAN1: 10KPOT1_PAN1.P0B, R69.1, R73.1
- new net P0B_PAN2: 10KPOT1_PAN3.P0B, R83.1, R87.1
- new net P0B_PAN3: 10KPOT1_PAN2.P0B, R13.1, R7.1
- new net P0B_PAN4: 10KPOT1_PAN4.P0B, R16.1, R20.1
- new net P0W1_COMP1: 10POT1_COMP1.P0W, R67.1
- new net P0W1_COMP2: 10POT1_COMP3.P0W, R117.1
- new net P0W1_COMP3: 10POT1_COMP2.P0W, R99.1
- new net P0W1_COMP4: 10POT1_COMP5.P0W, R153.1
- new net P0W_PAN1: 10KPOT1_PAN1.P0W, D2.C
- new net P0W_PAN2: 10KPOT1_PAN3.P0W, D4.C
- new net P0W_PAN3: 10KPOT1_PAN2.P0W, D3.C
- new net P0W_PAN4: 10KPOT1_PAN4.P0W, D5.C
- new net POS_A1_COMP1: 100POT1_COMP1.PW0, OPAMP1_COMP1.POS_A
- new net POS_A1_COMP2: 100POT1_COMP3.PW0, OPAMP1_COMP3.POS_A
- new net POS_A1_COMP3: 100POT1_COMP2.PW0, OPAMP1_COMP2.POS_A
- new net POS_A1_COMP4: 100POT1_COMP5.PW0, OPAMP1_COMP5.POS_A
- new net POS_A2_COMP1: OPAMP2_COMP1.POS_A, R64.2, R66.2
- new net POS_A2_COMP2: OPAMP2_COMP3.POS_A, R114.2, R116.2
- new net POS_A2_COMP3: OPAMP2_COMP2.POS_A, R96.2, R98.2
- new net POS_A2_COMP4: OPAMP2_COMP5.POS_A, R150.2, R152.2
- new net POS_A4_COMP1: D22.A, D23.C, OPAMP4_COMP1.POS_A, R93.1
- new net POS_A4_COMP2: D44.A, D45.C, OPAMP4_COMP3.POS_A, R129.1
- new net POS_A4_COMP3: D33.A, D34.C, OPAMP4_COMP2.POS_A, R111.1
- new net POS_A4_COMP4: D66.A, D67.C, OPAMP4_COMP5.POS_A, R165.1
- new net POS_B1_COMP1: D26.C, OPAMP1_COMP1.POS_B, R77.2
- new net POS_B1_COMP2: D48.C, OPAMP1_COMP3.POS_B, R120.2
- new net POS_B1_COMP3: D37.C, OPAMP1_COMP2.POS_B, R102.2
- new net POS_B1_COMP4: D70.C, OPAMP1_COMP5.POS_B, R156.2
- new net POS_B2_COMP1: 10POT2_COMP1.P0B, 10POT2_COMP1.P0W, OPAMP2_COMP1.POS_B, R91.1
- new net POS_B2_COMP2: 10POT2_COMP3.P0B, 10POT2_COMP3.P0W, OPAMP2_COMP3.POS_B, R127.1
- new net POS_B2_COMP3: 10POT2_COMP2.P0B, 10POT2_COMP2.P0W, OPAMP2_COMP2.POS_B, R109.1
- new net POS_B2_COMP4: 10POT2_COMP5.P0B, 10POT2_COMP5.P0W, OPAMP2_COMP5.POS_B, R163.1
- new net SCK: 100POT1_COMP1.SCK, 100POT1_COMP2.SCK, 100POT1_COMP3.SCK, 100POT1_COMP5.SCK, 10KPOT1_PAN1.SCK, 10KPOT1_PAN2.SCK, 10KPOT1_PAN3.SCK, 10KPOT1_PAN4.SCK, 10POT1_COMP1.SCK, 10POT1_COMP2.SCK, 10POT1_COMP3.SCK, 10POT1_COMP5.SCK, 10POT2_COMP1.SCK, 10POT2_COMP2.SCK, 10POT2_COMP3.SCK, 10POT2_COMP5.SCK, SCK1.P, U$1.CL, U$3.CL
- new net SCL: 200POT1_COMP1.SCL, 200POT1_COMP2.SCL, 200POT1_COMP3.SCL, 200POT1_COMP5.SCL, 200POT2_COMP1.SCL, 200POT2_COMP2.SCL, 200POT2_COMP3.SCL, 200POT2_COMP5.SCL, SCL1.P
- new net SCL1: IC2.MC/SCL, SCL2.P
- new net SDA: 200POT1_COMP1.SDA, 200POT1_COMP2.SDA, 200POT1_COMP3.SDA, 200POT1_COMP5.SDA, 200POT2_COMP1.SDA, 200POT2_COMP2.SDA, 200POT2_COMP3.SDA, 200POT2_COMP5.SDA, SDA1.P
- new net SDA1: IC2.MOSI/SDA, SDA2.P
- new net SDI/O: 100POT1_COMP1.SI, 100POT1_COMP2.SI, 100POT1_COMP3.SI, 100POT1_COMP5.SI, 10KPOT1_PAN1.SDI/SDO, 10KPOT1_PAN2.SDI/SDO, 10KPOT1_PAN3.SDI/SDO, 10KPOT1_PAN4.SDI/SDO, 10POT1_COMP1.SDI/SDO, 10POT1_COMP2.SDI/SDO, 10POT1_COMP3.SDI/SDO, 10POT1_COMP5.SDI/SDO, 10POT2_COMP1.SDI/SDO, 10POT2_COMP2.SDI/SDO, 10POT2_COMP3.SDI/SDO, 10POT2_COMP5.SDI/SDO, SDI/O1.P, U$1.DI, U$3.DI
- new net VDD: 9VDD1.P, OPAMP1_COMP1.V+, OPAMP1_COMP2.V+, OPAMP1_COMP3.V+, OPAMP1_COMP5.V+, OPAMP1_MIX1.V+, OPAMP1_PAN1.V+, OPAMP1_PAN2.V+, OPAMP1_PAN3.V+, OPAMP1_PAN4.V+, OPAMP2_COMP1.V+, OPAMP2_COMP2.V+, OPAMP2_COMP3.V+, OPAMP2_COMP5.V+, OPAMP3_COMP1.V+, OPAMP3_COMP2.V+, OPAMP3_COMP3.V+, OPAMP3_COMP5.V+, OPAMP4_COMP1.V+, OPAMP4_COMP2.V+, OPAMP4_COMP3.V+, OPAMP4_COMP5.V+, R101.1, R119.1, R155.1, R22.1, R76.1, R8.1, U$1.V_DD, U$3.V_DD, U2.V+
- new net VREF: 100POT1_COMP1.PA0, 100POT1_COMP1.VDD, 100POT1_COMP1.~RS, 100POT1_COMP1.~SHDN, 100POT1_COMP2.PA0, 100POT1_COMP2.VDD, 100POT1_COMP2.~RS, 100POT1_COMP2.~SHDN, 100POT1_COMP3.PA0, 100POT1_COMP3.VDD, 100POT1_COMP3.~RS, 100POT1_COMP3.~SHDN, 100POT1_COMP5.PA0, 100POT1_COMP5.VDD, 100POT1_COMP5.~RS, 100POT1_COMP5.~SHDN, 10KPOT1_PAN1.VDD, 10KPOT1_PAN2.VDD, 10KPOT1_PAN3.VDD, 10KPOT1_PAN4.VDD, 10POT1_COMP1.P0B, 10POT1_COMP1.VDD, 10POT1_COMP2.P0B, 10POT1_COMP2.VDD, 10POT1_COMP3.P0B, 10POT1_COMP3.VDD, 10POT1_COMP5.P0B, 10POT1_COMP5.VDD, 10POT2_COMP1.VDD, 10POT2_COMP2.VDD, 10POT2_COMP3.VDD, 10POT2_COMP5.VDD, 200POT1_COMP1.A0, 200POT1_COMP1.VDD, 200POT1_COMP2.A0, 200POT1_COMP2.VDD, 200POT1_COMP3.A0, 200POT1_COMP3.VDD, 200POT1_COMP5.A0, 200POT1_COMP5.VDD, 200POT2_COMP1.VDD, 200POT2_COMP2.VDD, 200POT2_COMP3.VDD, 200POT2_COMP5.VDD, C44.2, C47.2, C50.2, C56.2, D2.A, D3.A, D4.A, D5.A, OPAMP1_MIX1.POS_A, OPAMP1_MIX1.POS_B, OPAMP1_PAN1.POS_A, OPAMP1_PAN1.POS_B, OPAMP1_PAN2.POS_A, OPAMP1_PAN2.POS_B, OPAMP1_PAN3.POS_A, OPAMP1_PAN3.POS_B, OPAMP1_PAN4.POS_A, OPAMP1_PAN4.POS_B, OPAMP3_COMP1.POS_A, OPAMP3_COMP1.POS_B, OPAMP3_COMP2.POS_A, OPAMP3_COMP2.POS_B, OPAMP3_COMP3.POS_A, OPAMP3_COMP3.POS_B, OPAMP3_COMP5.POS_A, OPAMP3_COMP5.POS_B, R105.1, R106.1, R110.2, R112.1, R113.1, R114.1, R123.1, R124.1, R128.2, R130.1, R149.1, R15.1, R150.1, R159.1, R160.1, R164.2, R166.1, R35.1, R36.2, R37.2, R38.2, R50.1, R51.2, R52.2, R53.2, R6.1, R63.1, R64.1, R68.1, R80.1, R81.1, R82.1, R92.2, R94.1, R95.1, R96.1, U2.NEG_B, U2.OUT_B

Commit message: update footprint names of MAX5419 for LMNP variants
Parts:
- 200POT1_COMP1, 200POT2_COMP1: value MAX5419LETA+ -> MAX5419NETA+; device MAX5419LETA_:MAX5419LETA+ -> MAX5419NETA_:MAX5419NETA+
- 200POT1_COMP2, 200POT2_COMP2: value MAX5419LETA+ -> MAX5419META+; device MAX5419LETA_:MAX5419LETA+ -> MAX5419LETA_:MAX5419META+
- 200POT1_COMP3, 200POT2_COMP3: value MAX5419LETA+ -> MAX5419PETAT; device MAX5419LETA_:MAX5419LETA+ -> MAX5419PETAT:MAX5419PETAT
Other:
- moved on the sheet: C80
Changed lines of the file:
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@@
 <part name="10POT1_COMP1" library="MCP4131-503E_SN" deviceset="MCP4131-503E/SN" device=""/>
 <part name="10POT2_COMP1" library="MCP4131-503E_SN" deviceset="MCP4131-503E/SN" device=""/>
-<part name="200POT2_COMP1" library="MAX5419LETA_" deviceset="MAX5419LETA+" device=""/>
-<part name="200POT1_COMP1" library="MAX5419LETA_" deviceset="MAX5419LETA+" device=""/>
+<part name="200POT2_COMP1" library="MAX5419NETA_" deviceset="MAX5419NETA+" device=""/>
+<part name="200POT1_COMP1" library="MAX5419NETA_" deviceset="MAX5419NETA+" device=""/>
 <part name="C44" library="rcl" library_urn="urn:adsk.eagle:library:334" deviceset="C-US" device="C0402" package3d_urn="urn:adsk.eagle:package:23626/2" value="1.5u"/>
 <part name="OPAMP1_COMP1" library="LM4562MAX_NOPB" deviceset="LM4562MAX/NOPB" device=""/>
@@
 <part name="10POT1_COMP3" library="MCP4131-503E_SN" deviceset="MCP4131-503E/SN" device=""/>
 <part name="10POT2_COMP3" library="MCP4131-503E_SN" deviceset="MCP4131-503E/SN" device=""/>
-<part name="200POT2_COMP3" library="MAX5419LETA_" deviceset="MAX5419LETA+" device=""/>
-<part name="200POT1_COMP3" library="MAX5419LETA_" deviceset="MAX5419LETA+" device=""/>
+<part name="200POT2_COMP3" library="MAX5419PETAT" deviceset="MAX5419PETAT" device=""/>
+<part name="200POT1_COMP3" library="MAX5419PETAT" deviceset="MAX5419PETAT" device=""/>
 <part name="C50" library="rcl" library_urn="urn:adsk.eagle:library:334" deviceset="C-US" device="C0402" package3d_urn="urn:adsk.eagle:package:23626/2" value="1.5u"/>
 <part name="OPAMP1_COMP3" library="LM4562MAX_NOPB" deviceset="LM4562MAX/NOPB" device=""/>
@@
 <part name="10POT1_COMP2" library="MCP4131-503E_SN" deviceset="MCP4131-503E/SN" device=""/>
 <part name="10POT2_COMP2" library="MCP4131-503E_SN" deviceset="MCP4131-503E/SN" device=""/>
-<part name="200POT2_COMP2" library="MAX5419LETA_" deviceset="MAX5419LETA+" device=""/>
-<part name="200POT1_COMP2" library="MAX5419LETA_" deviceset="MAX5419LETA+" device=""/>
+<part name="200POT2_COMP2" library="MAX5419LETA_" deviceset="MAX5419META+" device=""/>
+<part name="200POT1_COMP2" library="MAX5419LETA_" deviceset="MAX5419META+" device=""/>
 <part name="C47" library="rcl" library_urn="urn:adsk.eagle:library:334" deviceset="C-US" device="C0402" package3d_urn="urn:adsk.eagle:package:23626/2" value="1.5u"/>
 <part name="OPAMP1_COMP2" library="LM4562MAX_NOPB" deviceset="LM4562MAX/NOPB" device=""/>
@@
 <attribute name="VALUE" x="293.116" y="719.709" size="1.778" layer="96"/>
 </instance>
-<instance part="C80" gate="G$1" x="302.26" y="723.9" smashed="yes">
-<attribute name="NAME" x="303.276" y="724.535" size="1.778" layer="95"/>
-<attribute name="VALUE" x="303.276" y="719.709" size="1.778" layer="96"/>
+<instance part="C80" gate="G$1" x="279.4" y="690.88" smashed="yes">
+<attribute name="NAME" x="280.416" y="691.515" size="1.778" layer="95"/>
+<attribute name="VALUE" x="280.416" y="686.689" size="1.778" layer="96"/>
 </instance>
 <instance part="C81" gate="G$1" x="276.86" y="734.06" smashed="yes">
@@
 <segment>
 <pinref part="C80" gate="G$1" pin="1"/>
-<wire x1="302.26" y1="726.44" x2="302.26" y2="734.06" width="0.1524" layer="91"/>
+<wire x1="279.4" y1="693.42" x2="302.26" y2="734.06" width="0.1524" layer="91"/>
 <label x="302.26" y="734.06" size="1.778" layer="95" xref="yes"/>
 </segment>
@@
 <pinref part="C80" gate="G$1" pin="2"/>
 <pinref part="IC2" gate="G$1" pin="VINL4/VIN4M"/>
-<wire x1="302.26" y1="718.82" x2="302.26" y2="685.8" width="0.1524" layer="91"/>
+<wire x1="279.4" y1="685.8" x2="302.26" y2="685.8" width="0.1524" layer="91"/>
 </segment>
 </net>

Commit message: update CAM
Parts:
- Y2: value CM7V-T1A-32.768KHZ-12.5PF-100PPM-TB-QC -> ECS-245.7-20-3X-EN-TR; device CM7V-T1A-32.768KHZ-12.5PF-100PPM-TB-QC:CM7V-T1A-32.768KHZ-12.5PF-100PPM-TB-QC -> ECS-245.7-20-3X-EN-TR:ECS-245.7-20-3X-EN-TR
Changed lines of the file:
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@@
 <part name="BCK_ADC1" library="wirepad" library_urn="urn:adsk.eagle:library:412" deviceset="SMD2" device="" package3d_urn="urn:adsk.eagle:package:30839/1"/>
 <part name="DOUT_ADC1" library="wirepad" library_urn="urn:adsk.eagle:library:412" deviceset="SMD2" device="" package3d_urn="urn:adsk.eagle:package:30839/1"/>
-<part name="Y2" library="CM7V-T1A-32.768KHZ-12.5PF-100PPM-TB-QC" deviceset="CM7V-T1A-32.768KHZ-12.5PF-100PPM-TB-QC" device=""/>
+<part name="Y2" library="ECS-245.7-20-3X-EN-TR" deviceset="ECS-245.7-20-3X-EN-TR" device=""/>
 <part name="C75" library="rcl" library_urn="urn:adsk.eagle:library:334" deviceset="C-US" device="C0402" package3d_urn="urn:adsk.eagle:package:23626/2" value="15pF"/>
 <part name="C76" library="rcl" library_urn="urn:adsk.eagle:library:334" deviceset="C-US" device="C0402" package3d_urn="urn:adsk.eagle:package:23626/2" value="15pF"/>

Commit message: fixes and export using jlcpcb ulp
Parts:
- C3, C4: value 0.1u -> 0.1uF
- C43, C46, C49, C55: value 10u -> 10uF
- D2, D3, D4, D5: value 1N4148W-TPSOD123-L -> 1N4148W-TP; device 1N4148W-TP:1N4148W-TPSOD123-L -> 1N4148W-TP:1N4148W-TP
Changed lines of the file:
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@@
 <part name="R44" library="rcl" library_urn="urn:adsk.eagle:library:334" deviceset="R-US_" device="R0402" package3d_urn="urn:adsk.eagle:package:23547/3" value="50k"/>
 <part name="R45" library="rcl" library_urn="urn:adsk.eagle:library:334" deviceset="R-US_" device="R0402" package3d_urn="urn:adsk.eagle:package:23547/3" value="1k"/>
-<part name="C3" library="rcl" library_urn="urn:adsk.eagle:library:334" deviceset="C-US" device="C0402" package3d_urn="urn:adsk.eagle:package:23626/2" value="0.1u"/>
+<part name="C3" library="rcl" library_urn="urn:adsk.eagle:library:334" deviceset="C-US" device="C0402" package3d_urn="urn:adsk.eagle:package:23626/2" value="0.1uF"/>
 <part name="OPAMP1_MIX1" library="LM4562MAX_NOPB" deviceset="LM4562MAX/NOPB" device=""/>
 <part name="GNDL1" library="wirepad" library_urn="urn:adsk.eagle:library:412" deviceset="SMD5" device="" package3d_urn="urn:adsk.eagle:package:30841/1"/>
@@
 <part name="R59" library="rcl" library_urn="urn:adsk.eagle:library:334" deviceset="R-US_" device="R0402" package3d_urn="urn:adsk.eagle:package:23547/3" value="50k"/>
 <part name="R60" library="rcl" library_urn="urn:adsk.eagle:library:334" deviceset="R-US_" device="R0402" package3d_urn="urn:adsk.eagle:package:23547/3" value="1k"/>
-<part name="C4" library="rcl" library_urn="urn:adsk.eagle:library:334" deviceset="C-US" device="C0402" package3d_urn="urn:adsk.eagle:package:23626/2" value="0.1u"/>
+<part name="C4" library="rcl" library_urn="urn:adsk.eagle:library:334" deviceset="C-US" device="C0402" package3d_urn="urn:adsk.eagle:package:23626/2" value="0.1uF"/>
 <part name="GNDR1" library="wirepad" library_urn="urn:adsk.eagle:library:412" deviceset="SMD5" device="" package3d_urn="urn:adsk.eagle:package:30841/1"/>
 <part name="OUTR_MIX1" library="wirepad" library_urn="urn:adsk.eagle:library:412" deviceset="SMD5" device="" package3d_urn="urn:adsk.eagle:package:30841/1"/>
@@
 </part>
 <part name="OPAMP1_PAN1" library="LM4562MAX_NOPB" deviceset="LM4562MAX/NOPB" device=""/>
-<part name="D2" library="1N4148W-TP" deviceset="1N4148W-TP" device="SOD123-L" value="1N4148W-TPSOD123-L"/>
+<part name="D2" library="1N4148W-TP" deviceset="1N4148W-TP" device="" value="1N4148W-TP"/>
 <part name="C6" library="rcl" library_urn="urn:adsk.eagle:library:334" deviceset="C-US" device="C0402" package3d_urn="urn:adsk.eagle:package:23626/2" value="10uF"/>
 <part name="R82" library="rcl" library_urn="urn:adsk.eagle:library:334" deviceset="R-US_" device="R0402" package3d_urn="urn:adsk.eagle:package:23547/3" value="1M"/>
@@
 </part>
 <part name="OPAMP1_PAN3" library="LM4562MAX_NOPB" deviceset="LM4562MAX/NOPB" device=""/>
-<part name="D4" library="1N4148W-TP" deviceset="1N4148W-TP" device="SOD123-L" value="1N4148W-TPSOD123-L"/>
+<part name="D4" library="1N4148W-TP" deviceset="1N4148W-TP" device="" value="1N4148W-TP"/>
 <part name="C8" library="rcl" library_urn="urn:adsk.eagle:library:334" deviceset="C-US" device="C0402" package3d_urn="urn:adsk.eagle:package:23626/2" value="10uF"/>
 <part name="R6" library="rcl" library_urn="urn:adsk.eagle:library:334" deviceset="R-US_" device="R0402" package3d_urn="urn:adsk.eagle:package:23547/3" value="1M"/>
@@
 </part>
 <part name="OPAMP1_PAN2" library="LM4562MAX_NOPB" deviceset="LM4562MAX/NOPB" device=""/>
-<part name="D3" library="1N4148W-TP" deviceset="1N4148W-TP" device="SOD123-L" value="1N4148W-TPSOD123-L"/>
+<part name="D3" library="1N4148W-TP" deviceset="1N4148W-TP" device="" value="1N4148W-TP"/>
 <part name="C2" library="rcl" library_urn="urn:adsk.eagle:library:334" deviceset="C-US" device="C0402" package3d_urn="urn:adsk.eagle:package:23626/2" value="10uF"/>
 <part name="R15" library="rcl" library_urn="urn:adsk.eagle:library:334" deviceset="R-US_" device="R0402" package3d_urn="urn:adsk.eagle:package:23547/3" value="1M"/>
@@
 </part>
 <part name="OPAMP1_PAN4" library="LM4562MAX_NOPB" deviceset="LM4562MAX/NOPB" device=""/>
-<part name="D5" library="1N4148W-TP" deviceset="1N4148W-TP" device="SOD123-L" value="1N4148W-TPSOD123-L"/>
+<part name="D5" library="1N4148W-TP" deviceset="1N4148W-TP" device="" value="1N4148W-TP"/>
 <part name="C5" library="rcl" library_urn="urn:adsk.eagle:library:334" deviceset="C-US" device="C0402" package3d_urn="urn:adsk.eagle:package:23626/2" value="10uF"/>
 <part name="U$1" library="LC75281E" deviceset="LC75281E" device="" package3d_urn="urn:adsk.eagle:package:41897184/1"/>
@@
 <part name="D24" library="1N4148W-TP" deviceset="1N4148W-TP" device=""/>
 <part name="D25" library="1N4148W-TP" deviceset="1N4148W-TP" device=""/>
-<part name="C43" library="rcl" library_urn="urn:adsk.eagle:library:334" deviceset="C-US" device="C0402" package3d_urn="urn:adsk.eagle:package:23626/2" value="10u"/>
+<part name="C43" library="rcl" library_urn="urn:adsk.eagle:library:334" deviceset="C-US" device="C0402" package3d_urn="urn:adsk.eagle:package:23626/2" value="10uF"/>
 <part name="D26" library="1N4148W-TP" deviceset="1N4148W-TP" device=""/>
 <part name="100POT1_COMP1" library="MCP42100-I_P" deviceset="MCP42100-I/P" device=""/>
@@
 <part name="D46" library="1N4148W-TP" deviceset="1N4148W-TP" device=""/>
 <part name="D47" library="1N4148W-TP" deviceset="1N4148W-TP" device=""/>
-<part name="C49" library="rcl" library_urn="urn:adsk.eagle:library:334" deviceset="C-US" device="C0402" package3d_urn="urn:adsk.eagle:package:23626/2" value="10u"/>
+<part name="C49" library="rcl" library_urn="urn:adsk.eagle:library:334" deviceset="C-US" device="C0402" package3d_urn="urn:adsk.eagle:package:23626/2" value="10uF"/>
 <part name="D48" library="1N4148W-TP" deviceset="1N4148W-TP" device=""/>
 <part name="100POT1_COMP3" library="MCP42100-I_P" deviceset="MCP42100-I/P" device=""/>
@@
 <part name="D35" library="1N4148W-TP" deviceset="1N4148W-TP" device=""/>
 <part name="D36" library="1N4148W-TP" deviceset="1N4148W-TP" device=""/>
-<part name="C46" library="rcl" library_urn="urn:adsk.eagle:library:334" deviceset="C-US" device="C0402" package3d_urn="urn:adsk.eagle:package:23626/2" value="10u"/>
+<part name="C46" library="rcl" library_urn="urn:adsk.eagle:library:334" deviceset="C-US" device="C0402" package3d_urn="urn:adsk.eagle:package:23626/2" value="10uF"/>
 <part name="D37" library="1N4148W-TP" deviceset="1N4148W-TP" device=""/>
 <part name="100POT1_COMP2" library="MCP42100-I_P" deviceset="MCP42100-I/P" device=""/>
@@
 <part name="D68" library="1N4148W-TP" deviceset="1N4148W-TP" device=""/>
 <part name="D69" library="1N4148W-TP" deviceset="1N4148W-TP" device=""/>
-<part name="C55" library="rcl" library_urn="urn:adsk.eagle:library:334" deviceset="C-US" device="C0402" package3d_urn="urn:adsk.eagle:package:23626/2" value="10u"/>
+<part name="C55" library="rcl" library_urn="urn:adsk.eagle:library:334" deviceset="C-US" device="C0402" package3d_urn="urn:adsk.eagle:package:23626/2" value="10uF"/>
 <part name="D70" library="1N4148W-TP" deviceset="1N4148W-TP" device=""/>
 <part name="100POT1_COMP5" library="MCP42100-I_P" deviceset="MCP42100-I/P" device=""/>
